File: SPCoast/GilroyCalTrain/GilroyCalTrain.kicad_sch (KiCad schematic)
At the start: 38 parts, among them SW771 771, SW773 773, SW775 775

Commit message: fix(kicad): approach circuits end in T; desk tokens follow
Plants: Christopher 1NA/2NA/1SA/2SA, GilroyCalTrain 1NA/1SA, GilroyInterchange
1SA, Sargent 1NA/1SA/2SA gain the final T (ADR 0003 D4). Sargent's reference
Corporal:2NA becomes Corporal:2NAT, the circuit Corporal draws.

Desk (South-cTc sheets): IndicationToken follows the plants for Christopher,
GilroyCalTrain, GilroyInterchange; Corporal 1SA becomes 1SAT (the plant already
had it); Christopher 815T2 becomes 815AT1 (the OS circuit of switch 815A).

Not changed, awaiting decisions in the dry-run report: 0<n>T renames (IND,
TK<n>, Interchange, 2NAAT, 2SAT), section 2 of an approach, unnamed circuits,
Watsonville, CP_Watsonville: references, 1TK.

Verified: netlists rebuilt for all affected projects; of 33 desk circuit tokens,
5 now match no plant circuit (was 11): 1TK, CP_Watsonville:SA1,
CP_Watsonville:837T1, Watsonville 1NAK and 2NAK. KiCad closed, no ~*.lck.

Co-Authored-By: Claude Sonnet 5.5 <noreply@anthropic.com>
Parts:
- TC1: value 1SA -> 1SAT
- TC5: value 1NA -> 1NAT
Changed lines of the file:
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@@
 			)
 		)
-		(property "Value" "1NA"
+		(property "Value" "1NAT"
 			(at 192.28 56.9 0)
 			(show_name no)
@@
 			)
 		)
-		(property "Value" "1SA"
+		(property "Value" "1SAT"
 			(at 56.39 56.9 0)
 			(show_name no)

Commit message: SPCoast: owner's edits: NextCP values (Sargent, Watsonville), yard crew names (GilroyCalTrain)
Baseline of the working tree as saved by KiCad, before the next fix. Saving in
KiCad wrote Luchessa's stale root UUID back into the instance paths of
GilroyCalTrain, Sargent and Watsonville (the .kicad_pro files still record it
under "sheets"); the following commit corrects both.

Co-Authored-By: Claude Sonnet 5.5 <noreply@anthropic.com>
Parts:
- DOT4: value YARD -> Track 3
- DOT5: value YARD -> Track 2
- DOT6: value YARD -> Track 1
Changed lines of the file:
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@@
 		(instances
 			(project "GilroyCalTrain"
-				(path "/2483c39b-4890-45a3-8f90-421e08f2026a"
+				(path "/87b90fc6-5e27-4e06-8416-fb28e674fdea"
 					(reference "B5")
 					(unit 1)
@@
 		(instances
 			(project "GilroyCalTrain"
-				(path "/2483c39b-4890-45a3-8f90-421e08f2026a"
+				(path "/87b90fc6-5e27-4e06-8416-fb28e674fdea"
 					(reference "B1")
 					(unit 1)
@@
 		(instances
 			(project "GilroyCalTrain"
-				(path "/2483c39b-4890-45a3-8f90-421e08f2026a"
+				(path "/87b90fc6-5e27-4e06-8416-fb28e674fdea"
 					(reference "H7")
 					(unit 1)
@@
 		(instances
 			(project "GilroyCalTrain"
-				(path "/2483c39b-4890-45a3-8f90-421e08f2026a"
+				(path "/87b90fc6-5e27-4e06-8416-fb28e674fdea"
 					(reference "SW773")
 					(unit 1)
@@
 		(instances
 			(project "GilroyCalTrain"
-				(path "/2483c39b-4890-45a3-8f90-421e08f2026a"
+				(path "/87b90fc6-5e27-4e06-8416-fb28e674fdea"
 					(reference "B4")
 					(unit 1)
@@
 		(instances
 			(project "GilroyCalTrain"
-				(path "/2483c39b-4890-45a3-8f90-421e08f2026a"
+				(path "/87b90fc6-5e27-4e06-8416-fb28e674fdea"
 					(reference "S1")
 					(unit 1)
@@
 			)
 		)
-		(property "Value" "YARD"
-			(at 193.802 110.49 0)
+		(property "Value" "Track 1"
+			(at 201.168 111.252 0)
 			(show_name no)
 			(do_not_autoplace yes)
@@
 		(instances
 			(project "GilroyCalTrain"
-				(path "/2483c39b-4890-45a3-8f90-421e08f2026a"
+				(path "/87b90fc6-5e27-4e06-8416-fb28e674fdea"
 					(reference "DOT6")
 					(unit 1)
@@
 		(instances
 			(project "GilroyCalTrain"
-				(path "/2483c39b-4890-45a3-8f90-421e08f2026a"
+				(path "/87b90fc6-5e27-4e06-8416-fb28e674fdea"
 					(reference "H4")
 					(unit 1)
@@
 		(instances
 			(project "GilroyCalTrain"
-				(path "/2483c39b-4890-45a3-8f90-421e08f2026a"
+				(path "/87b90fc6-5e27-4e06-8416-fb28e674fdea"
 					(reference "TC5")
 					(unit 1)
@@
 		(instances
 			(project "GilroyCalTrain"
-				(path "/2483c39b-4890-45a3-8f90-421e08f2026a"
+				(path "/87b90fc6-5e27-4e06-8416-fb28e674fdea"
 					(reference "CP1")
 					(unit 1)
@@
 		(instances
 			(project "GilroyCalTrain"
-				(path "/2483c39b-4890-45a3-8f90-421e08f2026a"
+				(path "/87b90fc6-5e27-4e06-8416-fb28e674fdea"
 					(reference "H1")
 					(unit 1)
@@
 			)
 		)
-		(property "Value" "YARD"
-			(at 195.072 93.98 0)
+		(property "Value" "Track 2"
+			(at 200.66 94.996 0)
 			(show_name no)
 			(do_not_autoplace yes)
@@
 		(instances
 			(project "GilroyCalTrain"
-				(path "/2483c39b-4890-45a3-8f90-421e08f2026a"
+				(path "/87b90fc6-5e27-4e06-8416-fb28e674fdea"
 					(reference "DOT5")
 					(unit 1)
@@
 		(instances
 			(project "GilroyCalTrain"
-				(path "/2483c39b-4890-45a3-8f90-421e08f2026a"
+				(path "/87b90fc6-5e27-4e06-8416-fb28e674fdea"
 					(reference "B3")
 					(unit 1)
@@
 		(instances
 			(project "GilroyCalTrain"
-				(path "/2483c39b-4890-45a3-8f90-421e08f2026a"
+				(path "/87b90fc6-5e27-4e06-8416-fb28e674fdea"
 					(reference "SW775")
 					(unit 1)
@@
 		(instances
 			(project "GilroyCalTrain"
-				(path "/2483c39b-4890-45a3-8f90-421e08f2026a"
+				(path "/87b90fc6-5e27-4e06-8416-fb28e674fdea"
 					(reference "CP2")
 					(unit 1)
@@
 		(instances
 			(project "GilroyCalTrain"
-				(path "/2483c39b-4890-45a3-8f90-421e08f2026a"
+				(path "/87b90fc6-5e27-4e06-8416-fb28e674fdea"
 					(reference "B2")
 					(unit 1)
@@
 		(instances
 			(project "GilroyCalTrain"
-				(path "/2483c39b-4890-45a3-8f90-421e08f2026a"
+				(path "/87b90fc6-5e27-4e06-8416-fb28e674fdea"
 					(reference "B8")
 					(unit 1)
@@
 		(instances
 			(project "GilroyCalTrain"
-				(path "/2483c39b-4890-45a3-8f90-421e08f2026a"
+				(path "/87b90fc6-5e27-4e06-8416-fb28e674fdea"
 					(reference "B10")
 					(unit 1)
@@
 		(instances
 			(project "GilroyCalTrain"
-				(path "/2483c39b-4890-45a3-8f90-421e08f2026a"
+				(path "/87b90fc6-5e27-4e06-8416-fb28e674fdea"
 					(reference "S3")
 					(unit 1)
@@
 		(instances
 			(project "GilroyCalTrain"
-				(path "/2483c39b-4890-45a3-8f90-421e08f2026a"
+				(path "/87b90fc6-5e27-4e06-8416-fb28e674fdea"
 					(reference "H5")
 					(unit 1)
@@
 		(instances
 			(project "GilroyCalTrain"
-				(path "/2483c39b-4890-45a3-8f90-421e08f2026a"
+				(path "/87b90fc6-5e27-4e06-8416-fb28e674fdea"
 					(reference "H3")
 					(unit 1)
@@
 			)
 		)
-		(property "Value" "YARD"
-			(at 195.072 77.47 0)
+		(property "Value" "Track 3"
+			(at 201.168 78.486 0)
 			(show_name no)
 			(do_not_autoplace yes)
@@
 		(instances
 			(project "GilroyCalTrain"
-				(path "/2483c39b-4890-45a3-8f90-421e08f2026a"
+				(path "/87b90fc6-5e27-4e06-8416-fb28e674fdea"
 					(reference "DOT4")
 					(unit 1)
@@
 		(instances
 			(project "GilroyCalTrain"
-				(path "/2483c39b-4890-45a3-8f90-421e08f2026a"
+				(path "/87b90fc6-5e27-4e06-8416-fb28e674fdea"
 					(reference "H6")
 					(unit 1)
@@
 		(instances
 			(project "GilroyCalTrain"
-				(path "/2483c39b-4890-45a3-8f90-421e08f2026a"
+				(path "/87b90fc6-5e27-4e06-8416-fb28e674fdea"
 					(reference "TC2")
 					(unit 1)
@@
 		(instances
 			(project "GilroyCalTrain"
-				(path "/2483c39b-4890-45a3-8f90-421e08f2026a"
+				(path "/87b90fc6-5e27-4e06-8416-fb28e674fdea"
 					(reference "B6")
 					(unit 1)
@@
 		(instances
 			(project "GilroyCalTrain"
-				(path "/2483c39b-4890-45a3-8f90-421e08f2026a"
+				(path "/87b90fc6-5e27-4e06-8416-fb28e674fdea"
 					(reference "DOT2")
 					(unit 1)
@@
 		(instances
 			(project "GilroyCalTrain"
-				(path "/2483c39b-4890-45a3-8f90-421e08f2026a"
+				(path "/87b90fc6-5e27-4e06-8416-fb28e674fdea"
 					(reference "S5")
 					(unit 1)
@@
 		(instances
 			(project "GilroyCalTrain"
-				(path "/2483c39b-4890-45a3-8f90-421e08f2026a"
+				(path "/87b90fc6-5e27-4e06-8416-fb28e674fdea"
 					(reference "S2")
 					(unit 1)
@@
 		(instances
 			(project "GilroyCalTrain"
-				(path "/2483c39b-4890-45a3-8f90-421e08f2026a"
+				(path "/87b90fc6-5e27-4e06-8416-fb28e674fdea"
 					(reference "HOUSE1")
 					(unit 1)
@@
 		(instances
 			(project "GilroyCalTrain"
-				(path "/2483c39b-4890-45a3-8f90-421e08f2026a"
+				(path "/87b90fc6-5e27-4e06-8416-fb28e674fdea"
 					(reference "B7")
 					(unit 1)
@@
 		(instances
 			(project "GilroyCalTrain"
-				(path "/2483c39b-4890-45a3-8f90-421e08f2026a"
+				(path "/87b90fc6-5e27-4e06-8416-fb28e674fdea"
 					(reference "SW771")
 					(unit 1)
@@
 		(instances
 			(project "GilroyCalTrain"
-				(path "/2483c39b-4890-45a3-8f90-421e08f2026a"
+				(path "/87b90fc6-5e27-4e06-8416-fb28e674fdea"
 					(reference "TC3")
 					(unit 1)
@@
 		(instances
 			(project "GilroyCalTrain"
-				(path "/2483c39b-4890-45a3-8f90-421e08f2026a"
+				(path "/87b90fc6-5e27-4e06-8416-fb28e674fdea"
 					(reference "H2")
 					(unit 1)
@@
 		(instances
 			(project "GilroyCalTrain"
-				(path "/2483c39b-4890-45a3-8f90-421e08f2026a"
+				(path "/87b90fc6-5e27-4e06-8416-fb28e674fdea"
 					(reference "B9")
 					(unit 1)
@@
 		(instances
 			(project "GilroyCalTrain"
-				(path "/2483c39b-4890-45a3-8f90-421e08f2026a"
+				(path "/87b90fc6-5e27-4e06-8416-fb28e674fdea"
 					(reference "TC1")
 					(unit 1)
@@
 		(instances
 			(project "GilroyCalTrain"
-				(path "/2483c39b-4890-45a3-8f90-421e08f2026a"
+				(path "/87b90fc6-5e27-4e06-8416-fb28e674fdea"
 					(reference "DOT1")
 					(unit 1)
@@
 		(instances
 			(project "GilroyCalTrain"
-				(path "/2483c39b-4890-45a3-8f90-421e08f2026a"
+				(path "/87b90fc6-5e27-4e06-8416-fb28e674fdea"
 					(reference "TC4")
 					(unit 1)
@@
 		(instances
 			(project "GilroyCalTrain"
-				(path "/2483c39b-4890-45a3-8f90-421e08f2026a"
+				(path "/87b90fc6-5e27-4e06-8416-fb28e674fdea"
 					(reference "S4")
 					(unit 1)
