File: SPCoast/Watsonville/Watsonville.kicad_sch (KiCad schematic)
At the start: 125 parts, among them SW11 11, SW13 13, SW15 15, SW17 17, SW19 19, SW21 21, SW23 23, SW25 25, SW3 3, SW5 5, SW7 7, SW837 837, SW9 9

Commit message: SPCoast: owner's edits: NextCP values (Sargent, Watsonville), yard crew names (GilroyCalTrain)
Baseline of the working tree as saved by KiCad, before the next fix. Saving in
KiCad wrote Luchessa's stale root UUID back into the instance paths of
GilroyCalTrain, Sargent and Watsonville (the .kicad_pro files still record it
under "sheets"); the following commit corrects both.

Co-Authored-By: Claude Sonnet 5.5 <noreply@anthropic.com>
Parts:
- added CP1: Sargent, symbol Railroad:NextCP
Connections:
- net at SW837.1 (C): now also CP1.1 (To)
