File: SPCoast/Luchessa/Luchessa.kicad_sch (KiCad schematic)
At the start: 47 parts, among them SW783 783, SW795 795, SW799 799

Commit message: SPCoast: Address field and Kind on PanelColumn-MAX7313; encoding Values; HBA; Watsonville update
Owner's drawing changes of 2026-10-02..03 (FieldUnit-Subdivision ADR 0002 D18
and the owner's responses):

- PanelColumn-MAX7313: the expander address moves from the Value to an
  Address field (Value is ${Address}); BusKind renamed Kind (I2C-MAX7313)
- Luchessa encoding symbols: Value "US&S 506 time-coded DC pulses"
- Sargent: HBD renamed HBA; traffic indications [NSEW]FLK
- Watsonville schematic brought to a usable state
- Luchessa plant: track circuits end in T; MC1 at CP Gilroy's house

Co-Authored-By: Claude Fable 5.1 <noreply@anthropic.com>
Parts:
- added FLK1: NFLK, symbol Railroad:AUXILIARY
- added FLK2: SFLK, symbol Railroad:AUXILIARY
Other:
- note added: "TRAFFIC"

Commit message: fix(kicad): Luchessa circuit 2NAAT becomes 01T
Owner-approved. The circuit lies between the OS circuits of switches 795 and
799 and contains neither, so it takes the zero-prefixed local form 0<n>T. The
desk OS lamp token follows.

Verified: the plant compiles with 01T in the home-clear lists of the same
routes as before; desk lamp tokens read 795T1, 01T, 799T1. FieldUnit-Subdivision
tests, the smoke script and generated JSON still cite 2NAAT; they change in
their own step.

Co-Authored-By: Claude Sonnet 5.5 <noreply@anthropic.com>
Parts:
- TC4: value 2NAAT -> 01T
Changed lines of the file:
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@@
 			)
 		)
-		(property "Value" "2NAAT"
+		(property "Value" "01T"
 			(at 135.128 83.566 0)
 			(show_name no)

Commit message: fix(kicad): remaining class I circuits take the 0<n>T form
Owner-approved numbers: Luchessa 2SAT -> 02T; Christopher IND -> 01T;
Corporal IND -> 01T; GilroyInterchange Interchange -> 01T and TK1 -> 02T
(passing-track main and siding merged into class I). Desk lamp 1TK on
GilroyInterchange column 4 becomes 02T.

Verified: netlists rebuilt for the five projects; every 0<n>T is unique within
its plant; desk circuit tokens that match no plant circuit are down to four
(CP_Watsonville:SA1, CP_Watsonville:837T1, Watsonville 1NAK and 2NAK).

Co-Authored-By: Claude Sonnet 5.5 <noreply@anthropic.com>
Parts:
- TC5: value 2SAT -> 02T
Changed lines of the file:
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@@
 			)
 		)
-		(property "Value" "2SAT"
+		(property "Value" "02T"
 			(at 70.358 67.056 0)
 			(show_name no)

Commit message: SPCoast: owner's edits: schematics synced with the revised symbol libraries (baseline)
Update Symbols from Library on all plant and desk sheets; CP values for
Christopher, GilroyInterchange and Luchessa; Restricted Speed markers
consolidated in Corporal, Luchessa and Sargent.

Observed in the diff, not changed by the sweep that follows: CP changed on 23
symbols (Christopher: prefix removed, 815/815A/IND now Christopher North) and
added on 12 (GilroyInterchange); two lamps' Color reset to their symbol variant
(Christopher LMP93 red -> yellow, Sargent LMP133 yellow -> red).

Verified: netlists keep their net counts (Christopher 33, Corporal 26,
GilroyCalTrain 27, GilroyInterchange 22, Luchessa 34, Sargent 18, Watsonville
96, South-cTc 341); desk compiles to 75 appliances, 137 bindings, 14 columns;
no root-UUID regression.

Co-Authored-By: Claude Sonnet 5.5 <noreply@anthropic.com>
Parts:
- removed DOT5: Restricted Speed, symbol Railroad:Rule105-RestrictedSpeed
- added DOT6: Restricted Speed, symbol Railroad:Rule105-RestrictedSpeed
- FLK1, FLK2, S784E1: CP (none) -> CP Luchessa
- MC1, S784E2, S784W1: CP (none) -> CP Gilroy
- S784W2, S784W3: CP (none) -> CP Carnadero
Connections:
- net at B10.2 (B), B4.2 (B), TC5.1 (TC): now also DOT6.1 (To)

Commit message: chore(kicad): sweep instance Role/Kind and stale fields to the library vocabulary
Scripted, one pass over every sheet except Watsonville (open in KiCad, locked):
- Role/Kind of placed symbols refreshed from the library by lib_id: 10 Role
  (MAIN HOUSE CONTROLLED_POINT -> CONTROL_POINT, Rule251-DoT empty) and 17 Kind
  (IRJ-Signal IRJ -> IRJ_SIGNAL x7, Mast_Single/Double swaps, HandThrow
  -> SWITCH_MANUAL, Derail, PanelLock -> LOCK_LEVER, NextCP).
- Stale instance fields dropped where the library no longer has them: 39 Name,
  28 Direction (all empty or retired), 5 CP on Bumper and IRJ symbols.
- Orphan embedded copies of the retired symbol Rule6.28-OtherThanMain removed
  from two sheets (unused).

Not done: Watsonville (locked); CMRInet -> CMRI (library Kind still CMRInet);
fields new to the library (MAIN HOUSE Kind, switch Indications) are not copied
onto instances, the compiler will read library defaults by lib_id; Rulebook
fields stay until the compiler stops requiring them.

Verified: per-symbol before/after comparison shows only these changes, same
symbol sets, positions and lib_ids; netlists keep their net counts (Christopher
33, Corporal 26, GilroyCalTrain 27, GilroyInterchange 22, Luchessa 34, Sargent
18, South-cTc 341); desk still 75 appliances, 137 bindings, 14 columns.

Co-Authored-By: Claude Sonnet 5.5 <noreply@anthropic.com>
Parts:
- DOT1: Name Track Signaled in One Direction -> (none)
- HOUSE1, HOUSE2, HOUSE3: Role CONTROLLED_POINT -> CONTROL_POINT
Changed lines of the file:
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@@
 			)
 		)
-		(property "Name" "Track Signaled in One Direction"
-			(at 230.505 79.375 0)
-			(hide yes)
-			(show_name no)
-			(do_not_autoplace no)
-			(effects
-				(font
-					(size 1.27 1.27)
-				)
-			)
-		)
 		(property "Role" "POLICY"
 			(at 229.87 83.82 0)
@@
 			)
 		)
-		(property "Role" "CONTROLLED_POINT"
+		(property "Role" "CONTROL_POINT"
 			(at 109.22 30.48 0)
 			(hide yes)
@@
 			)
 		)
-		(property "Role" "CONTROLLED_POINT"
+		(property "Role" "CONTROL_POINT"
 			(at 172.72 30.48 0)
 			(hide yes)
@@
 			)
 		)
-		(property "Role" "CONTROLLED_POINT"
+		(property "Role" "CONTROL_POINT"
 			(at 71.12 30.48 0)
 			(hide yes)

Commit message: chore(kicad): masts and maintainer calls carry no CP; IRJ-Signals do; CMRInet Kind is CMRI
Owner decision: an IRJ-Signal is the single source of a signal's control point
(a mast attaches to exactly one IRJ-Signal through its SIGNAL pin); a
maintainer call is tied to its house by the netlist.
- CP dropped from 23 masts and 5 maintainer calls.
- 7 empty IRJ-Signal CPs filled with the plant's only house (Corporal, Sargent).
- 43 empty Name fields that KiCad re-added to Christopher dropped again.
- Codeline-Transport Kind CMRInet -> CMRI on the placed instance and the
  embedded library copy (South-cTc root sheet).

Verified: per-symbol before/after comparison shows only these changes; every
IRJ-Signal in all seven plants has a CP naming one of its plant's houses; net
counts unchanged (Christopher 33, Corporal 26, GilroyCalTrain 27,
GilroyInterchange 22, Luchessa 34, Sargent 18, Watsonville 96, South-cTc 341);
desk compiles to 75 appliances, 137 bindings, 14 columns. Remaining CP
diagnostic: Sargent's Corporal:2NAT placeholder (cross-plant reference).

Co-Authored-By: Claude Sonnet 5.5 <noreply@anthropic.com>
Parts:
- MC1, S784E2, S784W1: CP CP Gilroy -> (none)
- S784E1: CP CP Luchessa -> (none)
- S784W2, S784W3: CP CP Carnadero -> (none)
Changed lines of the file:
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@@
 			)
 		)
-		(property "CP" "CP Gilroy"
-			(at 121.92 99.06 0)
-			(hide yes)
-			(show_name no)
-			(do_not_autoplace no)
-			(effects
-				(font
-					(size 1.27 1.27)
-				)
-			)
-		)
 		(pin "1"
 		)
@@
 			)
 		)
-		(property "CP" "CP Carnadero"
-			(at 204.47 82.55 0)
-			(hide yes)
-			(show_name no)
-			(do_not_autoplace no)
-			(effects
-				(font
-					(size 1.27 1.27)
-				)
-			)
-		)
 		(pin "1"
 		)
@@
 			)
 		)
-		(property "CP" "CP Gilroy"
-			(at 77.47 73.66 0)
-			(hide yes)
-			(show_name no)
-			(do_not_autoplace no)
-			(effects
-				(font
-					(size 1.27 1.27)
-				)
-			)
-		)
 		(pin "1"
 		)
@@
 			)
 		)
-		(property "CP" "CP Gilroy"
-			(at 109.22 30.48 0)
-			(hide yes)
-			(show_name no)
-			(do_not_autoplace no)
-			(effects
-				(font
-					(size 1.27 1.27)
-				)
-			)
-		)
 		(pin "1"
 		)
@@
 			)
 		)
-		(property "CP" "CP Luchessa"
-			(at 58.42 90.17 0)
-			(hide yes)
-			(show_name no)
-			(do_not_autoplace no)
-			(effects
-				(font
-					(size 1.27 1.27)
-				)
-			)
-		)
 		(pin "2"
 		)
@@
 			(at 204.47 66.04 0)
 			(hide yes)
-			(show_name no)
-			(do_not_autoplace no)
-			(effects
-				(font
-					(size 1.27 1.27)
-				)
-			)
-		)
-		(property "CP" "CP Carnadero"
-			(at 204.47 66.04 0)
-			(hide yes)

Commit message: SPCoast: owner's edits: Interlocking symbol on every Trackplan; MAIN HOUSE is STRUCTURE/CONTROL_POINT (baseline)
Each plant has one Interlocking symbol (Value is the authoritative name) and
every MAIN HOUSE's Interlocking pin is wired to it. Library Role/Kind:
Interlocking is STRUCTURE/INTERLOCKING, MAIN HOUSE is STRUCTURE/CONTROL_POINT
(refreshed on all instances by the owner).

Verified: one Interlocking symbol per plant; every house shares a net with it;
net counts are one higher than before in each plant (Christopher 34, Corporal
27, GilroyCalTrain 28, GilroyInterchange 23, Luchessa 35, Sargent 19,
Watsonville 97); no root-UUID regression; no symbol moved or removed.

Co-Authored-By: Claude Sonnet 5.5 <noreply@anthropic.com>
Parts:
- added Plant1: ${TITLE}, symbol Railroad:Interlocking
- HOUSE1, HOUSE2, HOUSE3: Kind (none) -> CONTROL_POINT; Role CONTROL_POINT -> STRUCTURE
Connections:
- new net: HOUSE1.2 (Interlocking), HOUSE2.2 (Interlocking), HOUSE3.2 (Interlocking), Plant1.1 (Interlocking)
Changed lines of the file:
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@@
 	)
 	(junction
+		(at 109.22 25.4)
+		(diameter 0)
+		(color 0 0 0 0)
+	)
+	(junction
 		(at 137.16 86.36)
 		(diameter 0)
@@
 	(wire
 		(pts
+			(xy 71.12 25.4) (xy 109.22 25.4)
+		)
+		(stroke
+			(width 0)
+			(type default)
+		)
+	)
+	(wire
+		(pts
 			(xy 214.63 69.85) (xy 229.87 69.85)
 		)
@@
 	(wire
 		(pts
+			(xy 109.22 25.4) (xy 172.72 25.4)
+		)
+		(stroke
+			(width 0)
+			(type default)
+		)
+	)
+	(wire
+		(pts
 			(xy 214.63 86.36) (xy 229.87 86.36)
 		)
@@
 			)
 		)
-		(property "Description" "Rrepresents the Control Point Maintainer Bungalow (plus optional Maintainer Call)"
+		(property "Description" "The Control Point Maintainer Bungalow (plus optional Maintainer Call)"
 			(at 109.22 36.195 0)
 			(hide yes)
@@
 			)
 		)
-		(property "Role" "CONTROL_POINT"
-			(at 109.22 30.48 0)
+		(property "Role" "STRUCTURE"
+			(at 93.98 27.94 0)
+			(hide yes)
+			(show_name no)
+			(do_not_autoplace no)
+			(effects
+				(font
+					(size 1.27 1.27)
+				)
+			)
+		)
+		(property "Kind" "CONTROL_POINT"
+			(at 95.885 29.972 0)
 			(hide yes)
 			(show_name no)
@@
 		(pin "1"
 		)
+		(pin "2"
+		)
 		(instances
 			(project "Luchessa"
@@
 	)
 	(symbol
+		(lib_id "Railroad:Interlocking")
+		(at 109.22 25.4 0)
+		(unit 1)
+		(body_style 1)
+		(exclude_from_sim no)
+		(in_bom yes)
+		(on_board yes)
+		(in_pos_files yes)
+		(dnp no)
+		(fields_autoplaced yes)
+		(property "Reference" "Plant1"
+			(at 94.996 19.558 0)
+			(hide yes)
+			(show_name no)
+			(do_not_autoplace no)
+			(effects
+				(font
+					(size 1.27 1.27)
+				)
+			)
+		)
+		(property "Value" "${TITLE}"
+			(at 106.172 22.352 0)
+			(show_name no)
+			(do_not_autoplace yes)
+			(effects
+				(font
+					(size 1.27 1.27)
+				)
+				(justify left)
+			)
+		)
+		(property "Footprint" ""
+			(at 109.22 25.4 0)
+			(hide yes)
+			(show_name no)
+			(do_not_autoplace no)
+			(effects
+				(font
+					(size 1.27 1.27)
+				)
+			)
+		)
+		(property "Datasheet" ""
+			(at 109.22 25.4 0)
+			(hide yes)
+			(show_name no)
+			(do_not_autoplace no)
+			(effects
+				(font
+					(size 1.27 1.27)
+				)
+			)
+		)
+		(property "Description" ""
+			(at 109.22 25.4 0)
+			(hide yes)
+			(show_name no)
+			(do_not_autoplace no)
+			(effects
+				(font
+					(size 1.27 1.27)
+				)
+			)
+		)
+		(property "Role" "STRUCTURE"
+			(at 97.917 15.748 0)
+			(hide yes)
+			(show_name no)
+			(do_not_autoplace no)
+			(effects
+				(font
+					(size 1.27 1.27)
+				)
+			)
+		)
+		(property "Kind" "INTERLOCKING"
+			(at 99.314 17.399 0)
+			(hide yes)
+			(show_name no)
+			(do_not_autoplace no)
+			(effects
+				(font
+					(size 1.27 1.27)
+				)
+			)
+		)
+		(pin "1"
+		)
+		(instances
+			(project "Luchessa"
+				(path "/87b90fc6-5e27-4e06-8416-fb28e674fdea"
+					(reference "Plant1")
+					(unit 1)
+				)
+			)
+		)
+	)
+	(symbol
 		(lib_id "Railroad:NextCP")
 		(at 245.11 102.87 180)
@@
 			)
 		)
-		(property "Description" "Rrepresents the Control Point Maintainer Bungalow (plus optional Maintainer Call)"
+		(property "Description" "The Control Point Maintainer Bungalow (plus optional Maintainer Call)"
 			(at 172.72 36.195 0)
 			(hide yes)
@@
 			)
 		)
-		(property "Role" "CONTROL_POINT"
-			(at 172.72 30.48 0)
+		(property "Role" "STRUCTURE"
+			(at 157.48 27.94 0)
+			(hide yes)
+			(show_name no)
+			(do_not_autoplace no)
+			(effects
+				(font
+					(size 1.27 1.27)
+				)
+			)
+		)
+		(property "Kind" "CONTROL_POINT"
+			(at 159.385 29.972 0)
 			(hide yes)
 			(show_name no)
@@
 		(pin "1"
 		)
+		(pin "2"
+		)
 		(instances
 			(project "Luchessa"
@@
 			)
 		)
-		(property "Description" "Rrepresents the Control Point Maintainer Bungalow (plus optional Maintainer Call)"
+		(property "Description" "The Control Point Maintainer Bungalow (plus optional Maintainer Call)"
 			(at 71.12 36.195 0)
 			(hide yes)
@@
 			)
 		)
-		(property "Role" "CONTROL_POINT"
-			(at 71.12 30.48 0)
+		(property "Role" "STRUCTURE"
+			(at 55.88 27.94 0)
+			(hide yes)
+			(show_name no)
+			(do_not_autoplace no)
+			(effects
+				(font
+					(size 1.27 1.27)
+				)
+			)
+		)
+		(property "Kind" "CONTROL_POINT"
+			(at 57.785 29.972 0)
 			(hide yes)
 			(show_name no)
@@
 		(pin "1"
 		)
+		(pin "2"
+		)
 		(instances

Commit message: SPCoast: owner's edits: NextCP names, Christopher heads and masts, Sargent milepost, Watsonville circuits and desk tokens (baseline)
- NextCP values name interlockings: GilroyCalTrain CP2 -> Gilroy Interchange;
  Luchessa CP1 -> Gilroy Interchange, CP2 -> Hollister, CP3 and CP4 ->
  Christopher.
- Christopher: the two unnamed dwarf masts, their IRJ-Signals (now plain IRJs)
  and heads removed; remaining heads lettered A, B, C.
- Sargent MAIN HOUSE Milepost 83.5.
- Watsonville circuits SDT -> 0DT and SAT -> 0AT; desk tokens 0DT, 0AT, AT and
  Watsonville:837T1 follow.

Verified: netlists rebuild (Christopher 30, Corporal 27, GilroyCalTrain 28,
GilroyInterchange 23, Luchessa 35, Sargent 19, Watsonville 97, South-cTc 341);
Christopher has no mast or head diagnostics left; desk compiles to 75
appliances, 137 bindings, 14 columns; no root-UUID regression.

Co-Authored-By: Claude Sonnet 5.5 <noreply@anthropic.com>
Parts:
- CP1: value CP Lick -> Gilroy Interchange
- CP2: value CP Hollister -> Hollister
- CP3, CP4: value CP Christopher -> Christopher
Changed lines of the file:
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@@
 			)
 		)
-		(property "Value" "CP Christopher"
+		(property "Value" "Christopher"
 			(at 248.158 102.87 0)
 			(show_name no)
@@
 			)
 		)
-		(property "Value" "CP Christopher"
+		(property "Value" "Christopher"
 			(at 248.158 86.36 0)
 			(show_name no)
@@
 			)
 		)
-		(property "Value" "CP Hollister"
+		(property "Value" "Hollister"
 			(at 248.158 69.85 0)
 			(show_name no)
@@
 			)
 		)
-		(property "Value" "CP Lick"
-			(at 22.098 86.36 0)
-			(show_name no)
-			(do_not_autoplace no)
+		(property "Value" "Gilroy Interchange"
+			(at 23.368 88.9 0)
+			(show_name no)
+			(do_not_autoplace no)
