File: SPCoast/Christopher/Christopher.kicad_sch (KiCad schematic)
At the start: 42 parts, among them SW813 813, SW815 815, SW817 817, SW900 815A

Commit message: chore(kicad): refresh instances to the ADR 0003 libraries (InterlockingPlant 95f53e2)
- Desk sheets (South-cTc/*) and the Sargent sandbox: embedded PanelSwitch, PanelLock,
  PanelSignal, PanelMCall, PanelCode, PanelLamp-*, PanelColumn-MAX7313 definitions refreshed
  from the library (refresh_embedded.py, checked against the pre-pass library: only Description
  text had drifted). Instance Role APPLIANCE -> PANEL (77).
- Plant sheets: powered-switch instance Kind SWITCH_POWERED -> SWITCH_REMOTE (21), matching the
  library (sweep_role_kind_fields.py).

Verified:
- verify_symbol_diff.py: same symbols, lib_ids and positions; only Role/Kind changed.
- Nets unchanged: Christopher 30, Corporal 27, GilroyCalTrain 28, GilroyInterchange 23,
  Luchessa 35, Sargent 61, Watsonville 99, South-cTc 341.
- parse_kicad_plant.py --format text identical before/after for all seven plants.
- Desk compile 75/137/14, diagnostics identical; the 7 desk locks bind WLS/~{WLS}/~{WLK}/WLK
  to the bits that were NWS/RWS/RWK/NWK.
- No sheet or project outside Luchessa carries the copied root UUID.

Co-Authored-By: Claude Opus 5.5 <noreply@anthropic.com>
Parts:
- SW815, SW900: Kind SWITCH_POWERED -> SWITCH_REMOTE
Changed lines of the file:
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@@
 			)
 		)
-		(property "Kind" "SWITCH_POWERED"
+		(property "Kind" "SWITCH_REMOTE"
 			(at 132.08 100.33 0)
 			(hide yes)
@@
 			)
 		)
-		(property "Kind" "SWITCH_POWERED"
+		(property "Kind" "SWITCH_REMOTE"
 			(at 170.18 67.31 0)
 			(hide yes)
