File: SPCoast/South-cTc/GilroyCaltrain.kicad_sch (KiCad schematic)
At the start: 14 parts, among them U21 ${ADDRESS}, U22 ${ADDRESS}

Commit message: chore(kicad): refresh instances to the ADR 0003 libraries (InterlockingPlant 95f53e2)
- Desk sheets (South-cTc/*) and the Sargent sandbox: embedded PanelSwitch, PanelLock,
  PanelSignal, PanelMCall, PanelCode, PanelLamp-*, PanelColumn-MAX7313 definitions refreshed
  from the library (refresh_embedded.py, checked against the pre-pass library: only Description
  text had drifted). Instance Role APPLIANCE -> PANEL (77).
- Plant sheets: powered-switch instance Kind SWITCH_POWERED -> SWITCH_REMOTE (21), matching the
  library (sweep_role_kind_fields.py).

Verified:
- verify_symbol_diff.py: same symbols, lib_ids and positions; only Role/Kind changed.
- Nets unchanged: Christopher 30, Corporal 27, GilroyCalTrain 28, GilroyInterchange 23,
  Luchessa 35, Sargent 61, Watsonville 99, South-cTc 341.
- parse_kicad_plant.py --format text identical before/after for all seven plants.
- Desk compile 75/137/14, diagnostics identical; the 7 desk locks bind WLS/~{WLS}/~{WLK}/WLK
  to the bits that were NWS/RWS/RWK/NWK.
- No sheet or project outside Luchessa carries the copied root UUID.

Co-Authored-By: Claude Opus 5.5 <noreply@anthropic.com>
Parts:
- CDE2, LMP11, LMP12, LMP21, LMP22, LMP23, MCK1, MCL1, SWL1, SWL2: Role APPLIANCE -> PANEL
Changed lines of the file:
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@@
 			)
 		)
-		(property "Role" "APPLIANCE"
+		(property "Role" "PANEL"
 			(at 80.01 29.21 0)
 			(hide yes)
@@
 			)
 		)
-		(property "Role" "APPLIANCE"
+		(property "Role" "PANEL"
 			(at 131.445 76.2 0)
 			(hide yes)
@@
 			)
 		)
-		(property "Role" "APPLIANCE"
+		(property "Role" "PANEL"
 			(at 130.81 90.17 0)
 			(hide yes)
@@
 			)
 		)
-		(property "Role" "APPLIANCE"
+		(property "Role" "PANEL"
 			(at 80.645 76.2 0)
 			(hide yes)
@@
 			)
 		)
-		(property "Role" "APPLIANCE"
+		(property "Role" "PANEL"
 			(at 130.81 24.13 0)
 			(hide yes)
@@
 			)
 		)
-		(property "Role" "APPLIANCE"
+		(property "Role" "PANEL"
 			(at 86.36 44.45 0)
 			(hide yes)
@@
 			)
 		)
-		(property "Role" "APPLIANCE"
+		(property "Role" "PANEL"
 			(at 130.81 29.21 0)
 			(hide yes)
@@
 			)
 		)
-		(property "Role" "APPLIANCE"
+		(property "Role" "PANEL"
 			(at 130.81 34.29 0)
 			(hide yes)
@@
 			)
 		)
-		(property "Role" "APPLIANCE"
+		(property "Role" "PANEL"
 			(at 80.01 101.6 0)
 			(hide yes)
@@
 			)
 		)
-		(property "Role" "APPLIANCE"
+		(property "Role" "PANEL"
 			(at 80.01 29.21 0)
 			(hide yes)

Commit message: chore(kicad): desk sheets to Driver-I2C-MAX7313 and the PanelLock Kind (InterlockingPlant owner review)
- 14 desk expanders: lib_id RailroadPanel:PanelColumn-MAX7313 -> Driver-I2C-MAX7313, embedded
  definition refreshed (pins A1..B8, same numbers and positions).
- 8 PanelLock instances: Kind LOCK_LEVER -> LOCK_LEVER_2LAMP_2CONTACT (7 desk, 1 Sargent sandbox).

Verified:
- verify_symbol_diff.py: only those lib_id and Kind changes.
- South-cTc 341 nets, Sargent 61; desk compile 75/137/14 with bindings identical to e2c1093.

Co-Authored-By: Claude Opus 5.5 <noreply@anthropic.com>
Parts:
- U21, U22: symbol RailroadPanel:PanelColumn-MAX7313 -> RailroadPanel:Driver-I2C-MAX7313
Changed lines of the file:
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@@
 	)
 	(symbol
-		(lib_id "RailroadPanel:PanelColumn-MAX7313")
+		(lib_id "RailroadPanel:Driver-I2C-MAX7313")
 		(at 99.06 72.39 0)
 		(unit 1)
@@
 	)
 	(symbol
-		(lib_id "RailroadPanel:PanelColumn-MAX7313")
+		(lib_id "RailroadPanel:Driver-I2C-MAX7313")
 		(at 149.86 72.39 0)
 		(unit 1)
