File: SPCoast/SPCoast.kicad_sch (KiCad schematic)
At the start: 0 parts

Commit message: feat(kicad): unified SPCoast title blocks (owner's specification)
Regenerated by build_spcoast.py: every sheet carries the same title block (US Letter landscape,
2026.10, rev 0.2, SPCoast Railroad, comments 1-9) except the title: South cTc on the root and
machine sheets, the interlocking name on each plant sheet and its Panel.

Verified: diff is title-block lines only; build check still 650 nets with all eight archived
projects identical, ERC unchanged (85), no root-UUID copies.

Co-Authored-By: Claude Opus 5.5 <noreply@anthropic.com>
Other:
- title: SPCoast -> South cTc
Changed lines of the file:
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@@
 	(paper "USLetter")
 	(title_block
-		(title "SPCoast")
+		(title "South cTc")
+		(date "2026.10")
+		(rev "0.2")
 		(company "SPCoast Railroad")
-		(comment 1 "Generated by FieldUnit-Subdivision tools/unify/build_spcoast.py until cutover")
+		(comment 1 "JPlocher")
+		(comment 2 "Layout Maintenance Drawing")
+		(comment 3 "South cTc")
+		(comment 4 "Southern Pacific Railroad")
+		(comment 5 "Coast Division")
+		(comment 6 "Era: 1985")
+		(comment 7 "As Planned")
+		(comment 8 "Layout Plan Drawings")
+		(comment 9 "active")
 	)
 	(sheet
