File: SPCoast/Sargent-Panel.kicad_sch (KiCad schematic)
At the start: 9 parts, among them U1 0x2C

Commit message: feat(kicad): deployment cases: Caltrain on a CMRInet node, Gilroy Interchange JMRI turnouts over MQTT
Gilroy Caltrain: field I/O drawn as per-bit CMRInet drivers (Driver-CMRI-IB/OB,
UA 30, 14 in / 20 out) with named devices for 3 switches, 5 track circuits and
7 heads (four encoder-wired, three lamp-wired). No processor is named: every
chip is on the hosted CMRInet bus, so the field unit runs on that bus's host.

Gilroy Interchange: proof of concept for JMRI turnouts and sensors over MQTT
(Driver-JMRI-Turnout, -Turnout-Feedback, -Sensor-Feedback) on switches 777
and 781. Known: the 777 drivers carry Address 771 (typo, fixed by the
follow-up rewrite); the JMRI symbols fail lint_symbol_fields (Pin.D names no
pin, Topic/States casing), also fixed by the rewrite.

Libraries: Railroad-HardwareIO gains Driver-CMRI-IB/OB and the four JMRI
drivers; Railroad-Field's Device-Head-CPL pins renumbered top down (G, Y, R).
Nine other sheets were re-saved by KiCad with property placements only.

Verified:
- kicad-cli ERC: 0 violations, whole project
- every Caltrain and Gilroy Interchange device binds; no duplicate CMRI bits
- netlist_diff vs post-sync.net: only additions on the two sheets (49 parts,
  34 nets, 68 nodes), nothing lost or changed elsewhere
- library-owned field drift on the new instances: 0

Co-Authored-By: Claude Fable 5.1 <noreply@anthropic.com>
Parts:
- COL1: Interlocking Sargent -> Luchessa
- LMP1: IndicationToken HBAK -> S
- LMP2: IndicationToken 835T1 -> S
- LMP3: IndicationToken Watsonville:837T1 -> S
- MCK1: IndicationToken MC1K -> S
Changed lines of the file:
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@@
 			)
 		)
-		(property "IndicationToken" "MC1K"
+		(property "IndicationToken" "S"
 			(at 78.105 104.14 0)
 			(show_name no)
@@
 			)
 		)
-		(property "IndicationToken" "Watsonville:837T1"
+		(property "IndicationToken" "S"
 			(at 78.105 36.83 0)
 			(show_name no)
@@
 			)
 		)
-		(property "IndicationToken" "835T1"
+		(property "IndicationToken" "S"
 			(at 78.105 31.75 0)
 			(show_name no)
@@
 			)
 		)
-		(property "ki_locked" ""
-			(at 80.01 63.5 0)
-			(hide yes)
-			(show_name no)
-			(do_not_autoplace no)
-			(effects
-				(font
-					(size 1.27 1.27)
-				)
-			)
-		)
 		(pin "4"
 		)
@@
 			)
 		)
-		(property "IndicationToken" "HBAK"
+		(property "IndicationToken" "S"
 			(at 78.105 26.67 0)
 			(show_name no)
@@
 			)
 		)
-		(property "Interlocking" "Sargent"
+		(property "Interlocking" "Luchessa"
 			(at 80.01 129.54 0)
 			(show_name yes)
@@
 			(hide yes)
 			(show_name no)
-			(do_not_autoplace no)
-			(effects
-				(font
-					(size 1.27 1.27)
-				)
-			)
-		)
-		(property "ki_locked" ""
-			(at 80.01 63.5 0)
-			(hide yes)
-			(show_name no)

Commit message: refactor(kicad): mast anchors with explicit indication-to-aspect casts; restore fields KiCad reset
Second pass after the cast chains (b4c58d3), decided 2026-10-17: the per-head
anchors Head-CPL/CL/Semaphore were the mast's indication table collapsed into
a symbol. The chain is now

    [Mast 774NAB] -indication- [Cast-Aspect-CPL unit B] -aspect- [Cast-Encoder-CPL] -bits- [chip]

Cast-Aspect-CPL/CL/Semaphore are multi-unit casts, one unit per head letter
(A..E), so placing unit B beside mast 774N is head 774NB with nothing typed;
the reader derives every head name from mast plus unit. Style's home is the
aspect cast. The project ERC now ignores missing_unit and missing_input_pin,
since an aspect cast places only the units its mast has.

CMRI bits: Address is the node (the chip every bit folds into, as for every
other driver), Bit is the bit, UA = ${Address} is a display echo, Value =
UA${Address}.IN.${Bit}.

Restore (SPCoast/edits/2026-10-17-restore-reset-fields.py): the owner's last
KiCad save before 857cae2 ran "update symbols from library" with field reset,
putting library defaults into per-instance fields on nine sheets: every
PanelLamp IndicationToken ("S"), PanelColumn Interlocking ("Luchessa"),
Luchessa encoding Station ("Panel"), Sargent Exp2 PCA9685-PWM 0x27 -> 0x20
(colliding with Exp3), and the 34 Caltrain bit numbers. All 98 values are
restored from the last good netlist export, embedded in the script.

Scripts: SPCoast/edits/2026-10-17-mast-chain.py (second pass; reuses the
first pass's helpers), 2026-10-17-restore-reset-fields.py. __pycache__/
added to .gitignore.

Verified:
- post-restore netlist vs the last good export: no field differs except on
  the anchors the first pass replaced and the intended JMRI blanks
- lint_symbol_fields: 93 symbols, 0 errors (per-unit cast rule)
- kicad-cli ERC: 0 violations; netlist export without warnings
- gate vs post-restore: nets not touching an anchor identical; all 11 aspect
  nets re-sourced from a Cast-Aspect un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
Parts:
- COL1: Interlocking Luchessa -> Sargent
- LMP1: IndicationToken S -> HBAK
- LMP2: IndicationToken S -> 835T1
- LMP3: IndicationToken S -> Watsonville:837T1
- MCK1: IndicationToken S -> MC1K
Changed lines of the file:
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@@
 			)
 		)
-		(property "IndicationToken" "S"
+		(property "IndicationToken" "MC1K"
 			(at 78.105 104.14 0)
 			(show_name no)
@@
 			)
 		)
-		(property "IndicationToken" "S"
+		(property "IndicationToken" "Watsonville:837T1"
 			(at 78.105 36.83 0)
 			(show_name no)
@@
 			)
 		)
-		(property "IndicationToken" "S"
+		(property "IndicationToken" "835T1"
 			(at 78.105 31.75 0)
 			(show_name no)
@@
 			)
 		)
-		(property "IndicationToken" "S"
+		(property "IndicationToken" "HBAK"
 			(at 78.105 26.67 0)
 			(show_name no)
@@
 			)
 		)
-		(property "Interlocking" "Luchessa"
+		(property "Interlocking" "Sargent"
 			(at 80.01 129.54 0)
 			(show_name yes)
