File: SPCoast/Sargent-Panel.kicad_sch (KiCad schematic)
At the start: 9 parts, among them U1 0x2C

Commit message: refactor(kicad): seam vocabulary after the naming audit: Processor, IOBus, PanelIOBus, House, Style, TimeCode, LocoNet, NodeType, MQTT-JMRI
SPCoast/edits/2026-10-22-vocabulary.py, the owner's rulings on
FieldUnit-Subdivision docs/review/naming-audit-2026-10-22.md:
- Host stays only on the transport symbols; the Interlocking, OfficeUnit and Processor pins, the unit
  sheets' port and labels are Processor.
- IOBus on the Processor pin; the office side is PanelIOBus on the unit ports, the Panel boxes' pins,
  the panel labels and the root sheet pins.
- MAIN HOUSE is House; its H pin is MC and hidden, as asked.
- OfficeUnit Type -> Style = US&S; TimeCode and LocoNet spellings, the LocoNet transport's pin is
  Transport; the one input Codeline sheet pin is bidirectional.
- The CMRInet node's Board -> NodeType (body text follows); JMRI drivers' IC = MQTT-JMRI.

Verified: --check on production/vocab-before.net vs vocab-after.net: identical connectivity under the
pin map, same parts (MAIN HOUSE -> House), only the ruled fields changed; field-io --check passes;
ERC 0 violations.

Co-Authored-By: Claude Fable 5.1 <noreply@anthropic.com>
Connections:
- net IOBus renamed PanelIOBus
Changed lines of the file:
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@@
 		(at 87.63 74.93)
 	)
-	(hierarchical_label "IOBus"
+	(hierarchical_label "PanelIOBus"
 		(shape bidirectional)
 		(at 111.76 111.76 0)

Commit message: refactor(kicad): model board lamps leave the columns; stale instance fields follow the libraries; PanelLamp-* retired
The owner's ruling (2026-10-23): the PanelColumn is the logical column, tied to a control point; the panel
I/O hardware is not. Every PanelLamp was a model board lamp except the maintainer-call lamp on the column's
pin 8. 34 lamps are now ModelLamp-<color> (no Column pin, Style board); 8 MC lamps are PanelMCall-Lamp.
Wires untouched: ~{LAMP} keeps its pin and the Column wire of a model lamp ends on nothing. Instance fields
the libraries dropped in c1d446b are gone from the sheets: Address on 7 processors, Interlocking and Machine
on 14 columns, Host on 2 transports. Railroad stays on the AAR encoding because its Topic template reads
${Railroad}; where Railroad lives is pending. Cached definitions refreshed for Processor, PanelColumn,
Transport-MQTT and Encoding-AAR. Scripted: SPCoast/edits/2026-10-23-model-lamps.py (edit, --check, --retire).

Verified: the script's gate on production/fields-after.net vs model-lamps-after.net: same 743 parts, lib ids
change only on the 42 lamps to the expected targets, fields change only as listed (Style indication->board
x34, the 37 drops), connectivity after == before minus the model lamps' pin 1, ERC 0 violations (the two
lib_symbol_mismatch warnings gone). lint_symbol_fields: 97 symbols, 0 errors (PanelLamp-BLUE, -GREEN, -RED, -YELLOW retired; there was no AMBER). Subdivision tests: 157 OK.

Co-Authored-By: Claude Fable 5.1 <noreply@anthropic.com>
Parts:
- COL1: Interlocking Sargent -> (none); Machine SPCoast South -> (none)
- LMP1, LMP2, LMP3: symbol Railroad-Office:PanelLamp-RED -> Railroad-Office:ModelLamp-RED; Style indication -> board
- MCK1: symbol Railroad-Office:PanelLamp-YELLOW -> Railroad-Office:PanelMCall-Lamp
Connections:
- net at COL1.3 (Column): no longer LMP3.1 (Column)
- net at COL1.2 (Column): no longer LMP2.1 (Column)
- net at COL1.1 (Column): no longer LMP1.1 (Column)
Changed lines of the file:
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@@
 	)
 	(symbol
-		(lib_id "Railroad-Office:PanelLamp-YELLOW")
+		(lib_id "Railroad-Office:PanelMCall-Lamp")
 		(at 80.01 104.14 0)
 		(unit 1)
@@
 			)
 		)
-		(property "Description" "One physical model board lamp. Value is a free descriptive label (e.g. OS, TRACK, MC) and is not used elsewhere. IndicationToken is a comma-separated list of indication names (track circuits such as 795T1,2NAA,799T1, or tokens such as MC1K) OR'd to drive this one lamp. All listed indications are still individually on the CodeLine wire"
+		(property "Description" "One physical Maintainer Call lamp.  IndicationToken is a comma-separated list of indication names (tokens such as MC1K)"
 			(at 80.01 111.76 0)
 			(hide yes)
@@
 	)
 	(symbol
-		(lib_id "Railroad-Office:PanelLamp-RED")
+		(lib_id "Railroad-Office:ModelLamp-RED")
 		(at 80.01 36.83 0)
 		(unit 1)
@@
 			)
 		)
-		(property "Description" "One physical model board lamp. Value is a free descriptive label (e.g. OS, TRACK, MC) and is not used elsewhere. IndicationToken is a comma-separated list of indication names (track circuits such as 795T1,2NAA,799T1, or tokens such as MC1K) OR'd to drive this one lamp. All listed indications are still individually on the CodeLine wire"
+		(property "Description" "One physical model board lamp. Value is a free descriptive label (e.g. OS, TRACK ...) and is not used elsewhere. IndicationToken is a comma-separated list of indication names (tokens from the CodeLine) OR'd to drive this one lamp."
 			(at 79.375 46.355 0)
 			(hide yes)
@@
 			)
 		)
-		(property "Style" "indication"
+		(property "Style" "board"
 			(at 80.01 39.37 0)
 			(hide yes)
@@
 				)
 			)
-		)
-		(pin "1"
 		)
 		(pin "2"
@@
 	)
 	(symbol
-		(lib_id "Railroad-Office:PanelLamp-RED")
+		(lib_id "Railroad-Office:ModelLamp-RED")
 		(at 80.01 31.75 0)
 		(unit 1)
@@
 			)
 		)
-		(property "Description" "One physical model board lamp. Value is a free descriptive label (e.g. OS, TRACK, MC) and is not used elsewhere. IndicationToken is a comma-separated list of indication names (track circuits such as 795T1,2NAA,799T1, or tokens such as MC1K) OR'd to drive this one lamp. All listed indications are still individually on the CodeLine wire"
+		(property "Description" "One physical model board lamp. Value is a free descriptive label (e.g. OS, TRACK ...) and is not used elsewhere. IndicationToken is a comma-separated list of indication names (tokens from the CodeLine) OR'd to drive this one lamp."
 			(at 79.375 41.275 0)
 			(hide yes)
@@
 			)
 		)
-		(property "Style" "indication"
+		(property "Style" "board"
 			(at 80.01 34.29 0)
 			(hide yes)
@@
 				)
 			)
-		)
-		(pin "1"
 		)
 		(pin "2"
@@
 	)
 	(symbol
-		(lib_id "Railroad-Office:PanelLamp-RED")
+		(lib_id "Railroad-Office:ModelLamp-RED")
 		(at 80.01 26.67 0)
 		(unit 1)
@@
 			)
 		)
-		(property "Description" "One physical model board lamp. Value is a free descriptive label (e.g. OS, TRACK, MC) and is not used elsewhere. IndicationToken is a comma-separated list of indication names (track circuits such as 795T1,2NAA,799T1, or tokens such as MC1K) OR'd to drive this one lamp. All listed indications are still individually on the CodeLine wire"
+		(property "Description" "One physical model board lamp. Value is a free descriptive label (e.g. OS, TRACK ...) and is not used elsewhere. IndicationToken is a comma-separated list of indication names (tokens from the CodeLine) OR'd to drive this one lamp."
 			(at 79.375 36.195 0)
 			(hide yes)
@@
 			)
 		)
-		(property "Style" "indication"
+		(property "Style" "board"
 			(at 80.01 29.21 0)
 			(hide yes)
@@
 				)
 			)
-		)
-		(pin "1"
 		)
 		(pin "2"
@@
 				)
 			)
-		)
-		(property "Interlocking" "Sargent"
-			(at 80.01 129.54 0)
-			(show_name yes)
-			(do_not_autoplace yes)
-			(effects
-				(font
-					(size 1.27 1.27)
-				)
-			)
-		)
-		(property "Machine" "SPCoast South"
-			(at 80.645 125.73 0)
-			(show_name no)
-			(do_not_autoplace yes)
-			(effects
-				(font
-					(size 1.905 1.905)
-				)
-			)
