File: SPCoast/Sargent.kicad_sch (KiCad schematic)
At the start: 43 parts, among them SW2 835, SW3 1, SW4 835

Commit message: feat(kicad): deployment cases: Caltrain on a CMRInet node, Gilroy Interchange JMRI turnouts over MQTT
Gilroy Caltrain: field I/O drawn as per-bit CMRInet drivers (Driver-CMRI-IB/OB,
UA 30, 14 in / 20 out) with named devices for 3 switches, 5 track circuits and
7 heads (four encoder-wired, three lamp-wired). No processor is named: every
chip is on the hosted CMRInet bus, so the field unit runs on that bus's host.

Gilroy Interchange: proof of concept for JMRI turnouts and sensors over MQTT
(Driver-JMRI-Turnout, -Turnout-Feedback, -Sensor-Feedback) on switches 777
and 781. Known: the 777 drivers carry Address 771 (typo, fixed by the
follow-up rewrite); the JMRI symbols fail lint_symbol_fields (Pin.D names no
pin, Topic/States casing), also fixed by the rewrite.

Libraries: Railroad-HardwareIO gains Driver-CMRI-IB/OB and the four JMRI
drivers; Railroad-Field's Device-Head-CPL pins renumbered top down (G, Y, R).
Nine other sheets were re-saved by KiCad with property placements only.

Verified:
- kicad-cli ERC: 0 violations, whole project
- every Caltrain and Gilroy Interchange device binds; no duplicate CMRI bits
- netlist_diff vs post-sync.net: only additions on the two sheets (49 parts,
  34 nets, 68 nodes), nothing lost or changed elsewhere
- library-owned field drift on the new instances: 0

Co-Authored-By: Claude Fable 5.1 <noreply@anthropic.com>
Parts:
- Exp2: Address 0x27 -> 0x20
Changed lines of the file:
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@@
 			)
 		)
-		(property "ki_locked" ""
-			(at 83.82 106.68 0)
-			(hide yes)
-			(show_name no)
-			(do_not_autoplace no)
-			(effects
-				(font
-					(size 1.27 1.27)
-				)
-			)
-		)
 		(pin "1"
 		)
@@
 			)
 		)
-		(property "Address" "0x27"
+		(property "Address" "0x20"
 			(at 176.911 106.807 0)
 			(hide yes)
@@
 			)
 		)
-		(property "ki_locked" ""
-			(at 91.44 118.11 0)
-			(hide yes)
-			(show_name no)
-			(do_not_autoplace no)
-			(effects
-				(font
-					(size 1.27 1.27)
-				)
-			)
-		)
 		(pin "1"
 		)
@@
 		)
 		(property "Pin.B" "binary"
-			(at 160.02 96.52 0)
+			(at 155.956 91.694 0)
 			(hide yes)
 			(show_name no)
-			(do_not_autoplace no)
+			(do_not_autoplace yes)
 			(effects
 				(font
-					(size 1.27 1.27)
+					(size 0.635 0.635)
 				)
 			)
@@
 			)
 		)
-		(property "ki_locked" ""
-			(at 91.44 118.11 0)
-			(hide yes)
-			(show_name no)
-			(do_not_autoplace no)
-			(effects
-				(font
-					(size 1.27 1.27)
-				)
-			)
-		)
 		(pin "1"
 		)
@@
 			)
 		)
-		(property "ki_locked" ""
-			(at 83.82 96.52 0)
-			(hide yes)
-			(show_name no)
-			(do_not_autoplace no)
-			(effects
-				(font
-					(size 1.27 1.27)
-				)
-			)
-		)
 		(pin "3"
 		)
@@
 			)
 		)
-		(property "ki_locked" ""
-			(at 83.82 106.68 0)
-			(hide yes)
-			(show_name no)
-			(do_not_autoplace no)
-			(effects
-				(font
-					(size 1.27 1.27)
-				)
-			)
-		)
 		(pin "4"
 		)
@@
 			)
 		)
-		(property "ki_locked" ""
-			(at 91.44 118.11 0)
-			(hide yes)
-			(show_name no)
-			(do_not_autoplace no)
-			(effects
-				(font
-					(size 1.27 1.27)
-				)
-			)
-		)
 		(pin "1"
 		)
@@
 			)
 		)
-		(property "Address" "0x27"
+		(property "Address" "0x20"
 			(at 176.911 96.647 0)
 			(hide yes)
@@
 			)
 		)
-		(property "Address" "0x27"
+		(property "Address" "0x20"
 			(at 176.911 116.967 0)
 			(hide yes)
@@
 			)
 		)
-		(property "Address" "0x27"
+		(property "Address" "0x20"
 			(at 176.911 127.127 0)
 			(hide yes)
@@
 		)
 		(property "Pin.B" "binary"
-			(at 200.66 95.25 0)
+			(at 190.881 90.932 0)
 			(hide yes)
 			(show_name no)
-			(do_not_autoplace no)
+			(do_not_autoplace yes)
 			(effects
 				(font
-					(size 1.27 1.27)
+					(size 0.635 0.635)
 				)
 			)
 		)
 		(property "Pin.G" "binary"
-			(at 200.66 95.25 0)
+			(at 190.881 90.932 0)
 			(hide yes)
 			(show_name no)
-			(do_not_autoplace no)
+			(do_not_autoplace yes)
 			(effects
 				(font
-					(size 1.27 1.27)
+					(size 0.635 0.635)
 				)
 			)
 		)
 		(property "Pin.R" "binary"
-			(at 200.66 95.25 0)
-			(hide yes)
-			(show_name no)
-			(do_not_autoplace no)
-			(effects
-				(font
-					(size 1.27 1.27)
-				)
-			)
-		)
-		(property "ki_locked" ""
-			(at 200.66 95.25 0)
+			(at 190.881 90.932 0)
 			(hide yes)
 			(show_name no)
-			(do_not_autoplace no)
+			(do_not_autoplace yes)
 			(effects
 				(font
-					(size 1.27 1.27)
+					(size 0.635 0.635)
 				)
 			)
@@
 		)
 		(property "Pin.B" "binary"
-			(at 160.02 115.57 0)
+			(at 150.241 111.252 0)
 			(hide yes)
 			(show_name no)
-			(do_not_autoplace no)
+			(do_not_autoplace yes)
 			(effects
 				(font
-					(size 1.27 1.27)
+					(size 0.635 0.635)
 				)
 			)
 		)
 		(property "Pin.G" "binary"
-			(at 160.02 115.57 0)
+			(at 150.241 111.252 0)
 			(hide yes)
 			(show_name no)
-			(do_not_autoplace no)
+			(do_not_autoplace yes)
 			(effects
 				(font
-					(size 1.27 1.27)
+					(size 0.635 0.635)
 				)
 			)
 		)
 		(property "Pin.R" "binary"
-			(at 160.02 115.57 0)
-			(hide yes)
-			(show_name no)
-			(do_not_autoplace no)
-			(effects
-				(font
-					(size 1.27 1.27)
-				)
-			)
-		)
-		(property "ki_locked" ""
-			(at 160.02 115.57 0)
+			(at 150.241 111.252 0)
 			(hide yes)
 			(show_name no)
-			(do_not_autoplace no)
+			(do_not_autoplace yes)
 			(effects
 				(font
-					(size 1.27 1.27)
+					(size 0.635 0.635)
 				)
 			)
@@
 			)
 		)
-		(property "ki_locked" ""
-			(at 83.82 96.52 0)
-			(hide yes)
-			(show_name no)
-			(do_not_autoplace no)
-			(effects
-				(font
-					(size 1.27 1.27)
-				)
-			)
-		)
 		(pin "1"
 		)
@@
 		)
 		(property "Pin.B" "binary"
-			(at 160.02 115.57 0)
+			(at 150.241 111.252 0)
 			(hide yes)
 			(show_name no)
-			(do_not_autoplace no)
+			(do_not_autoplace yes)
 			(effects
 				(font
-					(size 1.27 1.27)
+					(size 0.635 0.635)
 				)
 			)
 		)
 		(property "Pin.G" "binary"
-			(at 160.02 115.57 0)
+			(at 150.241 111.252 0)
 			(hide yes)
 			(show_name no)
-			(do_not_autoplace no)
+			(do_not_autoplace yes)
 			(effects
 				(font
-					(size 1.27 1.27)
+					(size 0.635 0.635)
 				)
 			)
 		)
 		(property "Pin.R" "binary"
-			(at 160.02 115.57 0)
-			(hide yes)
-			(show_name no)
-			(do_not_autoplace no)
-			(effects
-				(font
-					(size 1.27 1.27)
-				)
-			)
-		)
-		(property "ki_locked" ""
-			(at 160.02 115.57 0)
+			(at 150.241 111.252 0)
 			(hide yes)
 			(show_name no)
-			(do_not_autoplace no)
+			(do_not_autoplace yes)
 			(effects
 				(font
-					(size 1.27 1.27)
+					(size 0.635 0.635)
 				)
 			)
@@
 		)
 		(property "Pin.B" "binary"
-			(at 160.02 115.57 0)
+			(at 150.241 111.252 0)
 			(hide yes)
 			(show_name no)
-			(do_not_autoplace no)
+			(do_not_autoplace yes)
 			(effects
 				(font
-					(size 1.27 1.27)
+					(size 0.635 0.635)
 				)
 			)
 		)
 		(property "Pin.G" "binary"
-			(at 160.02 115.57 0)
+			(at 150.241 111.252 0)
 			(hide yes)
 			(show_name no)
-			(do_not_autoplace no)
+			(do_not_autoplace yes)
 			(effects
 				(font
-					(size 1.27 1.27)
+					(size 0.635 0.635)
 				)
 			)
 		)
 		(property "Pin.R" "binary"
-			(at 160.02 115.57 0)
-			(hide yes)
-			(show_name no)
-			(do_not_autoplace no)
-			(effects
-				(font
-					(size 1.27 1.27)
-				)
-			)
-		)
-		(property "ki_locked" ""
-			(at 160.02 115.57 0)
+			(at 150.241 111.252 0)
 			(hide yes)
 			(show_name no)
-			(do_not_autoplace no)
+			(do_not_autoplace yes)
 			(effects
 				(font
-					(size 1.27 1.27)
+					(size 0.635 0.635)
 				)
 			)

Commit message: refactor(kicad): explicit cast chains for heads; generic JMRI drivers
Decided 2026-10-17: no magic casts. A head device is an anchor (Head-CPL,
Head-CL, Head-Semaphore: Role DEVICE, Value = the head, one ASPECT output)
wired to explicit cast symbols (Role CAST: Cast-Lamps-RYG, Cast-Encoder-CPL,
Cast-Lamps-RGB, Cast-Color, Cast-Arm), each one aspect input to one output
kind. Drivers are generic sinks; a JMRI driver's Address is derived from the
served appliance unless written. New: Mast (indication output) and
Driver-JMRI-SignalMast (indication input). Pin kinds are value types:
binary, level, position, color, aspect, indication; pixel -> color.

Mechanical rewrite by SPCoast/edits/2026-10-17-cast-chain.py:
- Railroad-Field: six Device-Head-* symbols retired, nine symbols added.
- Railroad-HardwareIO: the four Driver-JMRI-* symbols lose topic/States and
  the Address template and gain Pin.* per pin; Driver-GPIO-Pixel kind color.
- Sargent, GilroyCalTrain: 11 head devices -> 11 anchors + 12 casts. Casts
  keep the old pin geometry so the chip pins stay touched; 836SB (4 units)
  gets Cast-Arm + Cast-Lamps-RGB joined by label 836SB_ASPECT and three wires.
- GilroyInterchange: six JMRI instances cleared of copied Value/Address/
  topic/States; the unannotated sensor driver annotated JMRI_MQTT5.
Placement is mechanical; tidy in KiCad as wanted.

Verified:
- lint_symbol_fields (with CAST role and the new vocabulary): 93 symbols, 0 errors
- kicad-cli ERC: 0 violations, whole project; netlist export without warnings
- gate vs pre-cast.net: every net not touching a head identical; all 28
  chip-side head nets reach the same chip pins through a cast pin of the same
  function; 11 aspect nets, each anchor + cast(s)
- kicad-cli sym export svg renders every symbol

Co-Authored-By: Claude Fable 5.1 <noreply@anthropic.com>
Parts:
- removed DevHead1: 836SA, symbol Railroad-Field:Device-Head-CL
- removed DevHead2: 836NA, symbol Railroad-Field:Device-Head-CPL-Encoder
- removed DevHead3: 836NB, symbol Railroad-Field:Device-Head-CPL-Encoder
- removed DevHead4: 836SB, symbol Railroad-Field:Device-Head-Semaphore-RGB
- added Cast1, Cast4: (no value), symbol Railroad-Field:Cast-Lamps-RGB
- added Cast2, Cast3: (no value), symbol Railroad-Field:Cast-Encoder-CPL
- added Cast5: (no value), symbol Railroad-Field:Cast-Arm
- added DevHead1: 836SA, symbol Railroad-Field:Head-CL
- added DevHead2: 836NA, symbol Railroad-Field:Head-CPL
- added DevHead3: 836NB, symbol Railroad-Field:Head-CPL
- added DevHead4: 836SB, symbol Railroad-Field:Head-Semaphore
Connections:
- net at Exp2.5 (A5): now also Cast2.2 (S1)
- net at Exp2.6 (A6): now also Cast3.1 (S0)
- net at Exp2.7 (A7): now also Cast3.2 (S1)
- net at Exp3.1 (A1): now also Cast5.1 (ARM)
- net at Exp2.3 (A3): now also Cast1.1 (~{R})
- net at Exp2.2 (A2): now also Cast1.2 (~{G})
- net at Exp2.1 (A1): now also Cast1.3 (~{B})
- net at Exp2.4 (A4): now also Cast2.1 (S0)
- net at Exp2.10 (B2): now also Cast4.2 (~{G})
- net at Exp2.11 (B3): now also Cast4.3 (~{B})
- net at Exp2.12 (B4): now also Cast4.1 (~{R})
- new net: Cast3.3 (ASPECT), DevHead3.1 (ASPECT)
- new net: Cast2.3 (ASPECT), DevHead2.1 (ASPECT)
- new net: Cast1.4 (ASPECT), DevHead1.1 (ASPECT)
- new net 836SB_ASPECT: Cast4.4 (ASPECT), Cast5.2 (ASPECT), DevHead4.1 (ASPECT)

Commit message: refactor(kicad): mast anchors with explicit indication-to-aspect casts; restore fields KiCad reset
Second pass after the cast chains (b4c58d3), decided 2026-10-17: the per-head
anchors Head-CPL/CL/Semaphore were the mast's indication table collapsed into
a symbol. The chain is now

    [Mast 774NAB] -indication- [Cast-Aspect-CPL unit B] -aspect- [Cast-Encoder-CPL] -bits- [chip]

Cast-Aspect-CPL/CL/Semaphore are multi-unit casts, one unit per head letter
(A..E), so placing unit B beside mast 774N is head 774NB with nothing typed;
the reader derives every head name from mast plus unit. Style's home is the
aspect cast. The project ERC now ignores missing_unit and missing_input_pin,
since an aspect cast places only the units its mast has.

CMRI bits: Address is the node (the chip every bit folds into, as for every
other driver), Bit is the bit, UA = ${Address} is a display echo, Value =
UA${Address}.IN.${Bit}.

Restore (SPCoast/edits/2026-10-17-restore-reset-fields.py): the owner's last
KiCad save before 857cae2 ran "update symbols from library" with field reset,
putting library defaults into per-instance fields on nine sheets: every
PanelLamp IndicationToken ("S"), PanelColumn Interlocking ("Luchessa"),
Luchessa encoding Station ("Panel"), Sargent Exp2 PCA9685-PWM 0x27 -> 0x20
(colliding with Exp3), and the 34 Caltrain bit numbers. All 98 values are
restored from the last good netlist export, embedded in the script.

Scripts: SPCoast/edits/2026-10-17-mast-chain.py (second pass; reuses the
first pass's helpers), 2026-10-17-restore-reset-fields.py. __pycache__/
added to .gitignore.

Verified:
- post-restore netlist vs the last good export: no field differs except on
  the anchors the first pass replaced and the intended JMRI blanks
- lint_symbol_fields: 93 symbols, 0 errors (per-unit cast rule)
- kicad-cli ERC: 0 violations; netlist export without warnings
- gate vs post-restore: nets not touching an anchor identical; all 11 aspect
  nets re-sourced from a Cast-Aspect un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
Parts:
- removed DevHead1: 836SA, symbol Railroad-Field:Head-CL
- removed DevHead2: 836NA, symbol Railroad-Field:Head-CPL
- removed DevHead3: 836NB, symbol Railroad-Field:Head-CPL
- removed DevHead4: 836SB, symbol Railroad-Field:Head-Semaphore
- added Cast13: (no value), symbol Railroad-Field:Cast-Aspect-CPL
- added Cast14: (no value), symbol Railroad-Field:Cast-Aspect-CL
- added Cast15: (no value), symbol Railroad-Field:Cast-Aspect-Semaphore
- added DevMast1: 836N, symbol Railroad-Field:Mast
- added DevMast2: 836S, symbol Railroad-Field:Mast
- Exp2: value ${ADDRESS} -> 0x27; Address 0x20 -> 0x27
Connections:
- net 836SB_ASPECT: now also Cast15.4 (ASPECT)
- net at Cast3.3 (ASPECT): now also Cast13.4 (ASPECT)
- net at Cast2.3 (ASPECT): now also Cast13.2 (ASPECT)
- net at Cast1.4 (ASPECT): now also Cast14.2 (ASPECT)
- new net: Cast13.1 (IND), Cast13.3 (IND), DevMast1.1 (IND)
- new net: Cast14.1 (IND), Cast15.3 (IND), DevMast2.1 (IND)

Commit message: refactor(kicad): one-step head casts with an explicit Head letter
The multi-unit aspect casts hid the head assignment in a KiCad unit number
and said the head style twice. One cast per head rendering now takes the
mast's indication and drives the lamps, select code, LED, color point or
arm directly: Cast-Head-CPL, Cast-Head-CPL-Encoded, Cast-Head-RGB,
Cast-Head-Color, Cast-Head-Semaphore (Role CAST, IND input, shown Head and
Style fields). The aspect is derived from style and indication, never
drawn; the aspect pin kind is retired. Cast-Aspect-*, Cast-Lamps-*,
Cast-Encoder-CPL, Cast-Color and Cast-Arm are retired. Bodies follow the
owner's tidy: one width, visible text inside, Pin.* beside their pins, the
encoder's select-code table kept. Two renderings of one head (836SB: arm
and RGB LED) are two casts with the same Head on the mast's IND net.

Sargent and GilroyCalTrain: every unit and its downstream casts collapse
onto the downstream positions by 2026-10-18-head-cast.py, pairing by the
baseline netlist; the ERC severities set to ignore for partial multi-unit
placement go back to warning.

Verified: 2026-10-18-head-cast-gate.py on production/pre-head.net vs
post-head.net: 535 nets not touching a unit or a head input identical;
eleven head names derived from mast Value + Head equal the old unit
letters (774NA-E, 774SA-B, 836NA-B, 836SA-B); only the 12 head casts
re-symbolled; no field change outside their own fields; ERC 0;
lint_symbol_fields 90 symbols 0 errors; sync-library-fields changed 0.

Co-Authored-By: Claude Fable 5.1 <noreply@anthropic.com>
Parts:
- removed Cast1, Cast4: (no value), symbol Railroad-Field:Cast-Lamps-RGB
- removed Cast13: (no value), symbol Railroad-Field:Cast-Aspect-CPL
- removed Cast14: (no value), symbol Railroad-Field:Cast-Aspect-CL
- removed Cast15: (no value), symbol Railroad-Field:Cast-Aspect-Semaphore
- removed Cast2, Cast3: (no value), symbol Railroad-Field:Cast-Encoder-CPL
- removed Cast5: (no value), symbol Railroad-Field:Cast-Arm
- added Cast1, Cast4: (no value), symbol Railroad-Field:Cast-Head-RGB
- added Cast2, Cast3: (no value), symbol Railroad-Field:Cast-Head-CPL-Encoded
- added Cast5: (no value), symbol Railroad-Field:Cast-Head-Semaphore
Connections:
- net at Exp2.6 (A6): now also Cast3.1 (S0)
- net at Exp2.7 (A7): now also Cast3.2 (S1)
- net at DevMast1.1 (IND): now also Cast2.3 (IND), Cast3.3 (IND)
- net at Exp2.5 (A5): now also Cast2.2 (S1)
- net at Exp3.1 (A1): now also Cast5.1 (ARM)
- net at Exp2.12 (B4): now also Cast4.1 (~{R})
- net at Exp2.10 (B2): now also Cast4.2 (~{G})
- net at Exp2.11 (B3): now also Cast4.3 (~{B})
- net 836S_IND: now reaches DevMast2.1 (IND)
- net 836S_IND: now also Cast1.4 (IND), Cast4.4 (IND), Cast5.2 (IND)
- net at Exp2.4 (A4): now also Cast2.1 (S0)
- net at Exp2.3 (A3): now also Cast1.1 (~{R})
- net at Exp2.2 (A2): now also Cast1.2 (~{G})
- net at Exp2.1 (A1): now also Cast1.3 (~{B})
