File: SPCoast/Sargent.kicad_sch (KiCad schematic)
At the start: 50 parts, among them SW2 835, SW3 1, SW4 835

Commit message: refactor(kicad): head devices are DEVICE with Appliance head; the OfficeUnit's Role is OFFICE_UNIT; stale instance Roles follow the libraries
SPCoast/edits/2026-10-23-roles.py, ADR 0009 §3.10 as approved: CAST and MACHINE were implementation
words. The seven Device-Head-* symbols and their 57 placed instances carry Role DEVICE and Appliance head;
the OfficeUnit carries OFFICE_UNIT; the four transport instances still saying CODELINE_TRANSPORT say
TRANSPORT. Descriptions: Device-Switch loses "cast", the JMRI drivers say FieldUnit, the OfficeUnit says
what it is. Every cached definition that differed from its library copy refreshed.

Verified: netlist connectivity and parts identical; no field changed beyond Role, Appliance and
Description; no CAST, MACHINE or CODELINE_TRANSPORT remains on any instance; ERC 0.

Co-Authored-By: Claude Fable 5.1 <noreply@anthropic.com>
Parts:
- Cast1, Cast2, Cast3, Cast4, Cast5: Appliance (none) -> head; Role CAST -> DEVICE
Changed lines of the file:
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@@
 			)
 		)
-		(property "Role" "CAST"
+		(property "Role" "DEVICE"
 			(at 138.43 132.969 0)
 			(hide yes)
@@
 			)
 		)
+		(property "Appliance" "head"
+			(at 149.86 137.16 0)
+			(hide yes)
+			(show_name no)
+			(do_not_autoplace no)
+			(effects
+				(font
+					(size 1.27 1.27)
+				)
+			)
+		)
 		(property "Style" "CPL"
 			(at 138.43 132.207 0)
@@
 			)
 		)
-		(property "Role" "CAST"
+		(property "Role" "DEVICE"
 			(at 138.43 138.049 0)
 			(hide yes)
@@
 			)
 		)
+		(property "Appliance" "head"
+			(at 149.86 142.24 0)
+			(hide yes)
+			(show_name no)
+			(do_not_autoplace no)
+			(effects
+				(font
+					(size 1.27 1.27)
+				)
+			)
+		)
 		(property "Style" "CPL"
 			(at 138.43 137.287 0)
@@
 			)
 		)
-		(property "Role" "CAST"
+		(property "Role" "DEVICE"
 			(at 186.69 122.682 0)
 			(hide yes)
@@
 			)
 		)
+		(property "Appliance" "head"
+			(at 207.01 120.65 0)
+			(hide yes)
+			(show_name no)
+			(do_not_autoplace no)
+			(effects
+				(font
+					(size 1.27 1.27)
+				)
+			)
+		)
 		(property "Style" "UQ"
 			(at 195.58 120.65 0)
@@
 			)
 		)
-		(property "Role" "CAST"
+		(property "Role" "DEVICE"
 			(at 138.43 117.729 0)
 			(hide yes)
@@
 			)
 		)
+		(property "Appliance" "head"
+			(at 149.86 123.19 0)
+			(hide yes)
+			(show_name no)
+			(do_not_autoplace no)
+			(effects
+				(font
+					(size 1.27 1.27)
+				)
+			)
+		)
 		(property "Style" "UQ"
 			(at 131.699 117.856 0)
@@
 			)
 		)
-		(property "Role" "CAST"
+		(property "Role" "DEVICE"
 			(at 138.43 125.349 0)
 			(hide yes)
@@
 				)
 			)
+		)
+		(property "Appliance" "head"
+			(at 149.86 130.81 0)
+			(hide yes)
+			(show_name no)
+			(do_not_autoplace no)
+			(effects
+				(font
+					(size 1.27 1.27)
+				)
+			)

Commit message: chore(kicad): owner edits (2026-10-23): Address off Processor, Interlocking and Machine off PanelColumn, Railroad off Encoding-AAR, Broker default cleared; Host and Address off four instances; Sargent Cast4 Style back to the library's CL
Baseline before the scripted removal of the same fields from the remaining placed instances.

Verified: production/fields-after.net against roles-after.net: connectivity identical (820 nets, 1850 nodes,
743 parts); field delta is exactly Cast4 Style UQ->CL, Proc2 Address, Transport2005 Host, Transport2009 Host.
lint_symbol_fields: 96 symbols, 0 errors. ERC: two new lib_symbol_mismatch warnings on Transport-MQTT, the
cached copy still carrying the Broker default; nothing else.

Co-Authored-By: Claude Fable 5.1 <noreply@anthropic.com>
Parts:
- Cast4: Style UQ -> CL
Changed lines of the file:
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@@
 			)
 		)
-		(property "Style" "UQ"
+		(property "Style" "CL"
 			(at 131.699 117.856 0)
 			(hide yes)

Commit message: refactor(kicad): model board lamps leave the columns; stale instance fields follow the libraries; PanelLamp-* retired
The owner's ruling (2026-10-23): the PanelColumn is the logical column, tied to a control point; the panel
I/O hardware is not. Every PanelLamp was a model board lamp except the maintainer-call lamp on the column's
pin 8. 34 lamps are now ModelLamp-<color> (no Column pin, Style board); 8 MC lamps are PanelMCall-Lamp.
Wires untouched: ~{LAMP} keeps its pin and the Column wire of a model lamp ends on nothing. Instance fields
the libraries dropped in c1d446b are gone from the sheets: Address on 7 processors, Interlocking and Machine
on 14 columns, Host on 2 transports. Railroad stays on the AAR encoding because its Topic template reads
${Railroad}; where Railroad lives is pending. Cached definitions refreshed for Processor, PanelColumn,
Transport-MQTT and Encoding-AAR. Scripted: SPCoast/edits/2026-10-23-model-lamps.py (edit, --check, --retire).

Verified: the script's gate on production/fields-after.net vs model-lamps-after.net: same 743 parts, lib ids
change only on the 42 lamps to the expected targets, fields change only as listed (Style indication->board
x34, the 37 drops), connectivity after == before minus the model lamps' pin 1, ERC 0 violations (the two
lib_symbol_mismatch warnings gone). lint_symbol_fields: 97 symbols, 0 errors (PanelLamp-BLUE, -GREEN, -RED, -YELLOW retired; there was no AMBER). Subdivision tests: 157 OK.

Co-Authored-By: Claude Fable 5.1 <noreply@anthropic.com>
Changed lines of the file:
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@@
-			)
-		)
-		(property "Address" ""
-			(at 44.45 22.86 0)
-			(hide yes)
-			(show_name no)
-			(do_not_autoplace no)
-			(effects
-				(font
-					(size 1.27 1.27)
-				)
 			)
 		)

Commit message: refactor(kicad): layout-wide facts on the Railroad symbol; the AAR Topic is the macro ctc/<STRUCTURE:RAILROAD:Name>/codeline/; Name on processors and transports
The owner's rulings (2026-10-23): a Railroad symbol on the root sheet (STRUCTURE/RAILROAD; Name, Railroad, Region,
Era, Rulebook) carries the layout-wide facts; a field may reference another symbol's field with <ROLE:KIND:Field>,
keyed by the fields the libraries key symbols by, resolved to the one instance in scope and expanded by the
compiler, never by KiCad (KIND empty for a Role without one); Name is the identity key everywhere, Value is never
read. The placed AAR encoding loses its Railroad field and its Topic becomes the macro; the library default follows.
The OfficeUnit instance loses Railroad and Era (off the library already). Processor and the four Transport-* gain
Name = ${Value}, library and 12 placed instances. Cached Encoding-AAR, OfficeUnit, Railroad, processors and
transports refreshed; no pin moved. Scripted: SPCoast/edits/2026-10-23-railroad.py (edit, --check).

Verified: the script's gate on production/model-lamps-after.net vs railroad-after.net: connectivity identical;
parts identical but for RAILROAD1; fields change only Topic (the macro, expanded against the one STRUCTURE/RAILROAD
symbol, equals the before value ctc/SPCoast/codeline/), Railroad x2 and Era x1 dropped, Name added on 12
processors and transports with Name == Value; ERC 0 violations. lint_symbol_fields: 98 symbols, 0 errors.

Co-Authored-By: Claude Fable 5.1 <noreply@anthropic.com>
Parts:
- Proc6: Name (none) -> ${Value}
Changed lines of the file:
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@@
+			)
+		)
+		(property "Name" "${Value}"
+			(at 43.18 26.67 0)
+			(hide yes)
+			(show_name no)
+			(do_not_autoplace no)
+			(effects
+				(font
+					(size 1.27 1.27)
+				)
 			)
 		)

Commit message: refactor(kicad): Name on every device, office unit and encoding; Kind on the JMRI drivers; Driver-JMRI-Light
The owner's rulings of 2026-10-24 on the review of ADR 0008 rev 4: Name = ${Value}
is the identity key everywhere, devices included; the OfficeUnit's Columns is
derived and struck; a JMRI driver carries no address and is keyed by its object
class and the device it serves, the class carried by Kind (TURNOUT, SENSOR,
SIGNALMAST, LIGHT); Driver-JMRI-Light (ADR 0005 §8: ON, INTENSITY) for a lamp
JMRI drives, and the two Gilroy Interchange maintainer-call lamps MC1 and MC2
become Lights (they were Sensors, which JMRI only displays).

Script: SPCoast/edits/2026-10-24-names-kind-light.py. Libraries: Name on 36
symbols (OfficeUnit, 5 encodings, 12 PANEL, 18 DEVICE), Columns off OfficeUnit,
Kind on 5 JMRI drivers, Driver-JMRI-Light added (the Sensor's pin positions,
INTENSITY as pin 3 below, no-connect on the two placed instances). Sheets: 359
Name instance fields, 16 Kind, 2 lib_id swaps, caches refreshed (no pin moved on
a refreshed symbol).

Verified: gate --check production/SPCoast.net production/names-after.net PASS:
same parts, same connectivity, Name == Value on all 273 named instances (47
heads with Value "~" resolve to an empty Name), Columns dropped once, Kind on 16
drivers, 2 Sensor -> Light with pin 1 reading ON; ERC 0 before and after.
Subdivision lint_symbol_fields: 99 symbols, 0 errors (Kind now allowed on
IODRIVER). production/SPCoast.net is the new export (production/ is untracked).

Co-Authored-By: Claude Fable 5.1 <noreply@anthropic.com>
Parts:
- Cast1, Cast2, Cast3, Cast4, Cast5, DevLamp1, DevLamp2, DevMast1, DevMast2, DevMast8, DevSW5, DevSW8, DevTC1, DevTC2, DevTC3, LK2, SW2: Name (none) -> ${Value}

Commit message: refactor(kicad): Name = ${Value} on every Trackplan appliance, so no key is read from Value
The owner (2026-10-24), on review finding 4: no exception for appliance names
read from Value. Data model keys are functional descriptions of their content
and the symbol attribute names reflect that choice; Value is generic. Every
Railroad-Trackplan APPLIANCE symbol (switches, derails, masts, heads, track
circuits, maintainer calls, auxiliaries) gains Name = ${Value}: the appliance's
own name, a head's letter. The compiler reads Name, never Value.

Script: SPCoast/edits/2026-10-24-trackplan-names.py (library symbols, placed
instances, caches refreshed; no pin moved).

Verified: gate --check production/SPCoast.net production/trackplan-names-after.net
PASS: same parts, lib ids, Values and connectivity; the only field change is Name
added on every Trackplan appliance with Name == Value; ERC 0 before and after.
Subdivision lint_symbol_fields: 99 symbols, 0 errors. production/SPCoast.net is
the new export.

Co-Authored-By: Claude Fable 5.1 <noreply@anthropic.com>
Parts:
- AUX1, H1, H2, H3, H4, MC1, S1, S2, S3, SW3, SW4, TC1, TC2, TC3, TC4: Name (none) -> ${Value}
Changed lines of the file:
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@@
 			)
 		)
+		(property "Name" "${Value}"
+			(at 147.32 73.66 0)
+			(hide yes)
+			(show_name no)
+			(do_not_autoplace no)
+			(effects
+				(font
+					(size 1.27 1.27)
+				)
+			)
+		)
 		(property "IndicationCeiling" ""
 			(at 133.985 73.025 0)
@@
 			)
 		)
+		(property "Name" "${Value}"
+			(at 97.79 57.15 0)
+			(hide yes)
+			(show_name no)
+			(do_not_autoplace no)
+			(effects
+				(font
+					(size 1.27 1.27)
+				)
+			)
+		)
 		(property "IndicationCeiling" "RESTRICTING/RESTRICTING"
 			(at 86.36 56.515 0)
@@
 			)
 		)
+		(property "Name" "${Value}"
+			(at 85.09 73.66 0)
+			(hide yes)
+			(show_name no)
+			(do_not_autoplace no)
+			(effects
+				(font
+					(size 1.27 1.27)
+				)
+			)
+		)
 		(property "Appliance" "track_circuit"
 			(at 85.09 73.66 0)
@@
 			)
 		)
+		(property "Name" "${Value}"
+			(at 109.22 73.66 0)
+			(hide yes)
+			(show_name no)
+			(do_not_autoplace no)
+			(effects
+				(font
+					(size 1.27 1.27)
+				)
+			)
+		)
 		(property "CP" "Sargent"
 			(at 109.22 76.2 0)
@@
 			)
 		)
+		(property "Name" "${Value}"
+			(at 132.08 77.47 0)
+			(hide yes)
+			(show_name no)
+			(do_not_autoplace no)
+			(effects
+				(font
+					(size 1.27 1.27)
+				)
+			)
+		)
 		(property "Appliance" "head"
 			(at 132.08 77.47 0)
@@
 			)
 		)
+		(property "Name" "${Value}"
+			(at 127 60.96 0)
+			(hide yes)
+			(show_name no)
+			(do_not_autoplace no)
+			(effects
+				(font
+					(size 1.27 1.27)
+				)
+			)
+		)
 		(property "Appliance" "head"
 			(at 127 60.96 0)
@@
 			)
 		)
+		(property "Name" "${Value}"
+			(at 156.21 69.85 0)
+			(hide yes)
+			(show_name no)
+			(do_not_autoplace no)
+			(effects
+				(font
+					(size 1.27 1.27)
+				)
+			)
+		)
 		(property "Appliance" "head"
 			(at 156.21 69.85 0)
@@
 			)
 		)
+		(property "Name" "${Value}"
+			(at 160.02 40.64 0)
+			(hide yes)
+			(show_name no)
+			(do_not_autoplace no)
+			(effects
+				(font
+					(size 1.27 1.27)
+				)
+			)
+		)
 		(property "Appliance" "lamp"
 			(at 156.21 35.56 0)
@@
 			)
 		)
+		(property "Name" "${Value}"
+			(at 158.75 69.85 0)
+			(hide yes)
+			(show_name no)
+			(do_not_autoplace no)
+			(effects
+				(font
+					(size 1.27 1.27)
+				)
+			)
+		)
 		(property "Appliance" "head"
 			(at 158.75 69.85 0)
@@
 			)
 		)
+		(property "Name" "${Value}"
+			(at 128.27 60.96 0)
+			(hide yes)
+			(show_name no)
+			(do_not_autoplace no)
+			(effects
+				(font
+					(size 1.27 1.27)
+				)
+			)
+		)
 		(property "Appliance" "mast"
 			(at 128.27 60.96 0)
@@
 			)
 		)
+		(property "Name" "${Value}"
+			(at 175.26 73.66 0)
+			(hide yes)
+			(show_name no)
+			(do_not_autoplace no)
+			(effects
+				(font
+					(size 1.27 1.27)
+				)
+			)
+		)
 		(property "Appliance" "track_circuit"
 			(at 175.26 73.66 0)
@@
 			)
 		)
+		(property "Name" "${Value}"
+			(at 128.27 77.47 0)
+			(hide yes)
+			(show_name no)
+			(do_not_autoplace no)
+			(effects
+				(font
+					(size 1.27 1.27)
+				)
+			)
+		)
 		(property "Appliance" "mast"
 			(at 128.27 77.47 0)
@@
 			)
 		)
+		(property "Name" "${Value}"
+			(at 160.02 69.85 0)
+			(hide yes)
+			(show_name no)
+			(do_not_autoplace no)
+			(effects
+				(font
+					(size 1.27 1.27)
+				)
+			)
+		)
 		(property "Appliance" "mast"
 			(at 160.02 69.85 0)
@@
 			)
 		)
+		(property "Name" "${Value}"
+			(at 119.38 73.66 0)
+			(hide yes)
+			(show_name no)
+			(do_not_autoplace no)
+			(effects
+				(font
+					(size 1.27 1.27)
+				)
+			)
+		)
 		(property "Appliance" "track_circuit"
 			(at 119.38 73.66 0)
@@
 			(at 116.84 57.15 0)
 			(hide yes)
+			(show_name no)
+			(do_not_autoplace no)
+			(effects
+				(font
+					(size 1.27 1.27)
+				)
+			)
+		)
+		(property "Name" "${Value}"
+			(at 116.84 57.15 0)
+			(hide yes)

Commit message: feat(kicad): owner edit (2026-10-24): Industry symbol (TRACK, Kind INDUSTRY) replaces the dark stubs at Sargent, Corporal and Luchessa
Railroad-Trackplan gains Industry: Role TRACK, Kind INDUSTRY, one pin EoT at
(1.27, 0), description "Track exists past this point, but is not drawn". It is
visually distinct from Bumper and carries its own Kind, so a reader can tell
"track ends" from "track continues, not drawn" (ADR 0009 §3.10 amended in
FieldUnit-Subdivision).

Sargent B8, B9 and Corporal B6, B7 sit directly on the N and R ports of the
hand-thrown switch beyond END CTC; the wires drawn into dark track are gone.
Luchessa's industry spur: the Bumper B7007 and the wire into dark track are
gone; B7010 becomes Industry, and a new IRJ-END_CTC B11008 stands beside it.

The other sheets change only in their embedded library cache. On
GilroyInterchange KiCad renamed the cached Driver-JMRI-Light's second Kind
property to Kind_1: the library itself still carries two Kind properties on
that symbol (LIGHT and SENSOR, from 6882aa6), to be fixed separately. No placed
symbol is affected.

Verified:
- kicad-cli ERC: 0 violations
- lint_symbol_fields.py: 100 symbols, 0 errors, 0 warnings
- component field diff, previous netlist vs fresh export: only the five added
  Industry symbols, the added END CTC, the removed Bumper and B7010's Kind
- compile_layout.py output unchanged except provenance
- no lock files; owner reports KiCad project closed and files saved

Co-Authored-By: Claude Fable 5.1 <noreply@anthropic.com>
Parts:
- added B8, B9: (no value), symbol Railroad-Trackplan:Industry
Connections:
- net at SW3.2 (N): now also B9.2 (EoT)
- net at SW3.3 (R): now also B8.2 (EoT)
- no-connect marks 24 -> 20
Changed lines of the file:
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@@
 	)
 	(no_connect
-		(at 80.01 57.15)
-	)
-	(no_connect
 		(at 207.01 151.13)
 	)
@@
 	)
 	(no_connect
-		(at 68.58 40.64)
-	)
-	(no_connect
 		(at 207.01 128.27)
 	)
@@
 	)
 	(no_connect
-		(at 68.58 57.15)
-	)
-	(no_connect
 		(at 207.01 153.67)
 	)
@@
 	)
 	(no_connect
-		(at 80.01 40.64)
-	)
-	(no_connect
 		(at 207.01 158.75)
 	)
@@
 	(wire
 		(pts
-			(xy 68.58 57.15) (xy 80.01 57.15)
-		)
-		(stroke
-			(width 0.4064)
-			(type dash)
-			(color 72 72 72 1)
-		)
-	)
-	(wire
-		(pts
 			(xy 63.5 26.67) (xy 63.5 29.21)
 		)
@@
 	(wire
 		(pts
-			(xy 68.58 40.64) (xy 80.01 40.64)
-		)
-		(stroke
-			(width 0.4064)
-			(type dash)
-			(color 72 72 72 1)
-		)
-	)
-	(wire
-		(pts
 			(xy 119.38 73.66) (xy 127 73.66)
 		)
@@
 	)
 	(symbol
+		(lib_id "Railroad-Trackplan:Industry")
+		(at 78.74 57.15 0)
+		(unit 1)
+		(body_style 1)
+		(exclude_from_sim no)
+		(in_bom yes)
+		(on_board yes)
+		(in_pos_files yes)
+		(dnp no)
+		(fields_autoplaced yes)
+		(property "Reference" "B9"
+			(at 78.74 59.69 0)
+			(hide yes)
+			(show_name no)
+			(do_not_autoplace no)
+			(effects
+				(font
+					(size 1.27 1.27)
+				)
+			)
+		)
+		(property "Value" ""
+			(at 78.74 57.15 0)
+			(hide yes)
+			(show_name no)
+			(do_not_autoplace no)
+			(effects
+				(font
+					(size 1.27 1.27)
+				)
+			)
+		)
+		(property "Footprint" ""
+			(at 78.74 57.15 0)
+			(hide yes)
+			(show_name no)
+			(do_not_autoplace no)
+			(effects
+				(font
+					(size 1.27 1.27)
+				)
+			)
+		)
+		(property "Datasheet" ""
+			(at 78.74 57.15 0)
+			(hide yes)
+			(show_name no)
+			(do_not_autoplace no)
+			(effects
+				(font
+					(size 1.27 1.27)
+				)
+			)
+		)
+		(property "Description" "Track exists past this point, but is not drawn"
+			(at 78.74 62.23 0)
+			(hide yes)
+			(show_name no)
+			(do_not_autoplace no)
+			(effects
+				(font
+					(size 1.27 1.27)
+				)
+			)
+		)
+		(property "Role" "TRACK"
+			(at 78.74 62.23 0)
+			(hide yes)
+			(show_name no)
+			(do_not_autoplace no)
+			(effects
+				(font
+					(size 1.27 1.27)
+				)
+			)
+		)
+		(property "Kind" "INDUSTRY"
+			(at 78.74 62.23 0)
+			(hide yes)
+			(show_name no)
+			(do_not_autoplace no)
+			(effects
+				(font
+					(size 1.27 1.27)
+				)
+			)
+		)
+		(pin "2"
+		)
+		(instances
+			(project "SPCoast"
+				(path "/528348b2-add8-5367-a5f7-439c76f0ca33/2ed995e3-3819-55cd-b8d9-5c2af048ccb4/f687a7a3-8fc1-435d-a0f4-b6b97af39a7e"
+					(reference "B9")
+					(unit 1)
+				)
+			)
+		)
+	)
+	(symbol
 		(lib_id "Railroad-Trackplan:IRJ")
 		(at 95.25 73.66 0)
@@
 					(unit 1)
 				)
+			)
+		)
+	)
+	(symbol
+		(lib_id "Railroad-Trackplan:Industry")
+		(at 78.74 40.64 0)
+		(unit 1)
+		(body_style 1)
+		(exclude_from_sim no)
+		(in_bom yes)
+		(on_board yes)
+		(in_pos_files yes)
+		(dnp no)
+		(fields_autoplaced yes)
+		(property "Reference" "B8"
+			(at 78.74 43.18 0)
+			(hide yes)
+			(show_name no)
+			(do_not_autoplace no)
+			(effects
+				(font
+					(size 1.27 1.27)
+				)
+			)
+		)
+		(property "Value" ""
+			(at 78.74 40.64 0)
+			(hide yes)
+			(show_name no)
+			(do_not_autoplace no)
+			(effects
+				(font
+					(size 1.27 1.27)
+				)
+			)
+		)
+		(property "Footprint" ""
+			(at 78.74 40.64 0)
+			(hide yes)
+			(show_name no)
+			(do_not_autoplace no)
+			(effects
+				(font
+					(size 1.27 1.27)
+				)
+			)
+		)
+		(property "Datasheet" ""
+			(at 78.74 40.64 0)
+			(hide yes)
+			(show_name no)
+			(do_not_autoplace no)
+			(effects
+				(font
+					(size 1.27 1.27)
+				)
+			)
+		)
+		(property "Description" "Track exists past this point, but is not drawn"
+			(at 78.74 45.72 0)
+			(hide yes)
+			(show_name no)
+			(do_not_autoplace no)
+			(effects
+				(font
+					(size 1.27 1.27)
+				)
+			)
+		)
+		(property "Role" "TRACK"
+			(at 78.74 45.72 0)
+			(hide yes)
+			(show_name no)
+			(do_not_autoplace no)
+			(effects
+				(font
+					(size 1.27 1.27)
+				)
+			)
+		)
+		(property "Kind" "INDUSTRY"
+			(at 78.74 45.72 0)
+			(hide yes)
+			(show_name no)
+			(do_not_autoplace no)
+			(effects
+				(font
+					(size 1.27 1.27)
+				)
+			)
+		)
+		(pin "2"
+		)
+		(instances
+			(project "SPCoast"
+				(path "/528348b2-add8-5367-a5f7-439c76f0ca33/2ed995e3-3819-55cd-b8d9-5c2af048ccb4/f687a7a3-8fc1-435d-a0f4-b6b97af39a7e"
+					(reference "B8")
+					(unit 1)
+				)
