File: SPCoast/Sargent.kicad_sch (KiCad schematic)
At the start: 52 parts, among them SW2 835, SW3 1, SW4 835

Commit message: feat(kicad): owner edit (2026-10-26): NextCP carries Interlocking; Industry carries Name; HBA leaves the track
The owner's edits after the trackplan review:
- NextCP gains Interlocking = ${Value}, a key the compiler reads for the destination; every instance takes it.
  Christopher's two NextCPs toward Corporal now say Corporal (both said Sargent).
- Industry gains Name = ${VALUE}. The five Industries are named: Gilroy Industry at Luchessa, Beet Loader 1
  and 2 at Corporal and at Sargent.
- Sargent's HBA (hot box alarm) is moved off 1SAT's net; its MC pin is unconnected and it carries Milepost 83.4.
- Watsonville: one Rule 93 (YARD) symbol is moved to the yard side of its joint.
Panels/ is left untracked.

Verified:
- Netlist exported by the owner 2026-10-26 12:37, newer than every sheet and the library.
- lint_symbol_fields: 100 symbols, 0 errors, 0 warnings.

Co-Authored-By: Claude Opus 5.5 <noreply@anthropic.com>
Parts:
- AUX1: Milepost (none) -> 83.4
- B8: value (none) -> Beet Loader 1; Name (none) -> ${VALUE}
- B9: value (none) -> Beet Loader 2; Name (none) -> ${VALUE}
- CP1, CP2: Interlocking (none) -> ${Value}
Connections:
- net at B1.2 (B), B4.2 (B), TC3.1 (TC): no longer AUX1.1 (MC)
Changed lines of the file:
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@@
 	)
 	(junction
-		(at 109.22 73.66)
-		(diameter 0)
-		(color 0 0 0 0)
-	)
-	(junction
 		(at 189.23 73.66)
 		(diameter 0)
@@
 	(wire
 		(pts
-			(xy 96.52 73.66) (xy 109.22 73.66)
+			(xy 96.52 73.66) (xy 119.38 73.66)
 		)
 		(stroke
@@
 	(wire
 		(pts
-			(xy 109.22 73.66) (xy 119.38 73.66)
-		)
-		(stroke
-			(width 0.4064)
-			(type default)
-		)
-	)
-	(wire
-		(pts
 			(xy 119.38 73.66) (xy 127 73.66)
 		)
@@
 		)
 		(property "Value" "Watsonville"
-			(at 187.325 73.66 0)
+			(at 191.77 82.55 0)
+			(hide yes)
 			(show_name no)
-			(do_not_autoplace no)
+			(do_not_autoplace yes)
 			(effects
 				(font
@@
 			)
 		)
+		(property "Interlocking" "${Value}"
+			(at 191.77 82.55 0)
+			(hide yes)
+			(show_name no)
+			(do_not_autoplace no)
+			(effects
+				(font
+					(size 1.27 1.27)
+				)
+			)
+		)
 		(pin "1"
 		)
@@
 	)
 	(symbol
-		(lib_id "Railroad-Trackplan:AUXILIARY")
-		(at 109.22 73.66 0)
-		(unit 1)
-		(body_style 1)
-		(exclude_from_sim no)
-		(in_bom yes)
-		(on_board yes)
-		(in_pos_files yes)
-		(dnp no)
-		(property "Reference" "AUX1"
-			(at 109.22 78.105 0)
-			(hide yes)
-			(show_name no)
-			(do_not_autoplace yes)
-			(effects
-				(font
-					(size 1.27 1.27)
-				)
-			)
-		)
-		(property "Value" "HBA"
-			(at 109.22 71.12 0)
-			(show_name no)
-			(do_not_autoplace yes)
-			(effects
-				(font
-					(size 1.27 1.27)
-				)
-			)
-		)
-		(property "Footprint" ""
-			(at 109.22 73.66 0)
-			(hide yes)
-			(show_name no)
-			(do_not_autoplace no)
-			(effects
-				(font
-					(size 1.27 1.27)
-				)
-			)
-		)
-		(property "Datasheet" ""
-			(at 109.22 73.66 0)
-			(hide yes)
-			(show_name no)
-			(do_not_autoplace no)
-			(effects
-				(font
-					(size 1.27 1.27)
-				)
-			)
-		)
-		(property "Description" ""
-			(at 109.22 73.66 0)
-			(hide yes)
-			(show_name no)
-			(do_not_autoplace no)
-			(effects
-				(font
-					(size 1.27 1.27)
-				)
-			)
-		)
-		(property "Role" "APPLIANCE"
-			(at 109.22 73.66 0)
-			(hide yes)
-			(show_name no)
-			(do_not_autoplace no)
-			(effects
-				(font
-					(size 1.27 1.27)
-				)
-			)
-		)
-		(property "Name" "${Value}"
-			(at 109.22 73.66 0)
-			(hide yes)
-			(show_name no)
-			(do_not_autoplace no)
-			(effects
-				(font
-					(size 1.27 1.27)
-				)
-			)
-		)
-		(property "CP" "Sargent"
-			(at 109.22 76.2 0)
-			(show_name no)
-			(do_not_autoplace yes)
-			(effects
-				(font
-					(size 0.762 0.762)
-				)
-			)
-		)
-		(property "Appliance" "lamp"
-			(at 109.22 73.66 0)
-			(hide yes)
-			(show_name no)
-			(do_not_autoplace no)
-			(effects
-				(font
-					(size 1.27 1.27)
-				)
-			)
-		)
-		(property "Style" "non_vital"
-			(at 109.22 73.66 0)
-			(hide yes)
-			(show_name no)
-			(do_not_autoplace no)
-			(effects
-				(font
-					(size 1.27 1.27)
-				)
-			)
-		)
-		(pin "1"
-		)
-		(instances
-			(project "SPCoast"
-				(path "/528348b2-add8-5367-a5f7-439c76f0ca33/2ed995e3-3819-55cd-b8d9-5c2af048ccb4/f687a7a3-8fc1-435d-a0f4-b6b97af39a7e"
-					(reference "AUX1")
-					(unit 1)
-				)
-			)
-		)
-	)
-	(symbol
 		(lib_id "Railroad-Field:Device-Switch-OS")
 		(at 69.85 144.78 0)
@@
 			)
 		)
-		(property "Value" ""
+		(property "Value" "Beet Loader 2"
 			(at 78.74 57.15 0)
 			(hide yes)
@@
 			)
 		)
+		(property "Name" "${VALUE}"
+			(at 78.74 57.15 0)
+			(hide yes)
+			(show_name no)
+			(do_not_autoplace no)
+			(effects
+				(font
+					(size 1.27 1.27)
+				)
+			)
+		)
 		(pin "2"
 		)
@@
 	)
 	(symbol
+		(lib_id "Railroad-Trackplan:AUXILIARY")
+		(at 109.22 78.74 0)
+		(unit 1)
+		(body_style 1)
+		(exclude_from_sim no)
+		(in_bom yes)
+		(on_board yes)
+		(in_pos_files yes)
+		(dnp no)
+		(property "Reference" "AUX1"
+			(at 109.22 83.185 0)
+			(hide yes)
+			(show_name no)
+			(do_not_autoplace yes)
+			(effects
+				(font
+					(size 1.27 1.27)
+				)
+			)
+		)
+		(property "Value" "HBA"
+			(at 109.22 76.2 0)
+			(show_name no)
+			(do_not_autoplace yes)
+			(effects
+				(font
+					(size 1.27 1.27)
+				)
+			)
+		)
+		(property "Footprint" ""
+			(at 109.22 78.74 0)
+			(hide yes)
+			(show_name no)
+			(do_not_autoplace no)
+			(effects
+				(font
+					(size 1.27 1.27)
+				)
+			)
+		)
+		(property "Datasheet" ""
+			(at 109.22 78.74 0)
+			(hide yes)
+			(show_name no)
+			(do_not_autoplace no)
+			(effects
+				(font
+					(size 1.27 1.27)
+				)
+			)
+		)
+		(property "Description" ""
+			(at 109.22 78.74 0)
+			(hide yes)
+			(show_name no)
+			(do_not_autoplace no)
+			(effects
+				(font
+					(size 1.27 1.27)
+				)
+			)
+		)
+		(property "Role" "APPLIANCE"
+			(at 109.22 78.74 0)
+			(hide yes)
+			(show_name no)
+			(do_not_autoplace no)
+			(effects
+				(font
+					(size 1.27 1.27)
+				)
+			)
+		)
+		(property "Name" "${Value}"
+			(at 109.22 78.74 0)
+			(hide yes)
+			(show_name no)
+			(do_not_autoplace no)
+			(effects
+				(font
+					(size 1.27 1.27)
+				)
+			)
+		)
+		(property "CP" "Sargent"
+			(at 109.22 81.28 0)
+			(show_name no)
+			(do_not_autoplace yes)
+			(effects
+				(font
+					(size 0.762 0.762)
+				)
+			)
+		)
+		(property "Appliance" "lamp"
+			(at 109.22 78.74 0)
+			(hide yes)
+			(show_name no)
+			(do_not_autoplace no)
+			(effects
+				(font
+					(size 1.27 1.27)
+				)
+			)
+		)
+		(property "Style" "non_vital"
+			(at 109.22 78.74 0)
+			(hide yes)
+			(show_name no)
+			(do_not_autoplace no)
+			(effects
+				(font
+					(size 1.27 1.27)
+				)
+			)
+		)
+		(property "Milepost" "83.4"
+			(at 109.474 82.804 0)
+			(show_name no)
+			(do_not_autoplace no)
+			(effects
+				(font
+					(size 1.27 1.27)
+				)
+			)
+		)
+		(pin "1"
+		)
+		(instances
+			(project "SPCoast"
+				(path "/528348b2-add8-5367-a5f7-439c76f0ca33/2ed995e3-3819-55cd-b8d9-5c2af048ccb4/f687a7a3-8fc1-435d-a0f4-b6b97af39a7e"
+					(reference "AUX1")
+					(unit 1)
+				)
+			)
+		)
+	)
+	(symbol
 		(lib_id "Railroad-Field:Local-Switch")
 		(at 62.23 133.35 0)
@@
 		)
 		(property "Value" "Corporal"
-			(at 66.675 73.66 0)
+			(at 71.12 82.55 0)
+			(hide yes)
 			(show_name no)
-			(do_not_autoplace no)
+			(do_not_autoplace yes)
 			(effects
 				(font
@@
 			)
 		)
+		(property "Interlocking" "${Value}"
+			(at 71.12 82.55 0)
+			(hide yes)
+			(show_name no)
+			(do_not_autoplace no)
+			(effects
+				(font
+					(size 1.27 1.27)
+				)
+			)
+		)
 		(pin "1"
 		)
@@
 			)
 		)
-		(property "Value" ""
+		(property "Value" "Beet Loader 1"
 			(at 78.74 40.64 0)
 			(hide yes)
@@
 			(hide yes)
 			(show_name no)
+			(do_not_autoplace no)
+			(effects
+				(font
+					(size 1.27 1.27)
+				)
+			)
+		)
+		(property "Name" "${VALUE}"
+			(at 78.74 40.64 0)
+			(hide yes)
+			(show_name no)
