File: SPCoast/Christopher-Panel.kicad_sch (KiCad schematic)
At the start: 23 parts, among them U10028 0x27, U10029 0x28, U10030 0x29

Commit message: feat(kicad): Sargent, Watsonville, Corporal, Christopher as local units with the four ports; all panels on the desk bus
SPCoast/edits/2026-10-21-local-units.py (owner's instruction 2026-10-21: assume each is like
Sargent, a local cpNode-Xiao with I2C I/O; prepopulate, tidy by hand later).

- Watsonville, Corporal, Christopher: a Processor '<unit>' (cpNode-Xiao) above the Interlocking,
  Host wired to it; an IOBus port on its bus pin. Sargent: IOBus port on Proc6 with its three
  expanders labelled onto it, and a Host port.
- Every Panel box gains an I2C pin carrying the OfficeIOBus port; every MAX7313 bus pin on the
  four panels is labelled I2C.
- South-cTc: the three units host themselves (their drops from the SPCoastApp host line removed,
  the line shortened to the Gilroy pair); the four boxes gain IOBus and OfficeIOBus (Sargent also
  Host), Host and IOBus no-connected, OfficeIOBus dropped onto the office line, extended right
  with junctions.

Verified: --check on production/local-units-before.net vs -after.net: desk bus = JohnCTC plus all
14 panel expanders; each unit's Host net is its own processor; SPCoastApp hosts Gilroy Caltrain,
Gilroy Interchange and the two I/O transports; Sargent's bus = Proc6 plus three expanders;
MQTT, TIMECODE, CMRInet, JMRI_MQTT unchanged; nothing else changed; parts added Proc8-10 only.
ERC: 0 violations. Rendered South-cTc and Sargent and inspected.

Co-Authored-By: Claude Fable 5.1 <noreply@anthropic.com>
Connections:
- net I2C: now reaches U10029.17 (I2C)
- net I2C: now also U10028.17 (I2C), U10030.17 (I2C)
Changed lines of the file:
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@@
 		(at 87.63 80.01)
+	)
+	(hierarchical_label "I2C"
+		(shape bidirectional)
+		(at 160.02 111.76 0)
+		(effects
+			(font
+				(size 1.27 1.27)
+			)
+			(justify left)
+		)
+	)
+	(hierarchical_label "I2C"
+		(shape bidirectional)
+		(at 210.82 111.76 0)
+		(effects
+			(font
+				(size 1.27 1.27)
+			)
+			(justify left)
+		)
+	)
+	(hierarchical_label "I2C"
+		(shape bidirectional)
+		(at 109.22 111.76 0)
+		(effects
+			(font
+				(size 1.27 1.27)
+			)
+			(justify left)
+		)
 	)
 	(symbol
