File: SPCoast/Christopher-Panel.kicad_sch (KiCad schematic)
At the start: 23 parts, among them U10028 0x27, U10029 0x28, U10030 0x29

Commit message: chore(kicad): owner edits: Remote-IO node fields (Kind CMRI / MQTT-JMRI, bytes, UA), Interlocking Name, IOBus pins on remote drivers, sheet cleanup
Owner's edits of 2026-10-22, committed as they stand before the read-back.
Connections:
- net I2C renamed IOBus
