File: SPCoast/Christopher-Panel.kicad_sch (KiCad schematic)
At the start: 23 parts, among them U10028 0x27, U10029 0x28, U10030 0x29

Commit message: refactor(kicad): seam vocabulary after the naming audit: Processor, IOBus, PanelIOBus, House, Style, TimeCode, LocoNet, NodeType, MQTT-JMRI
SPCoast/edits/2026-10-22-vocabulary.py, the owner's rulings on
FieldUnit-Subdivision docs/review/naming-audit-2026-10-22.md:
- Host stays only on the transport symbols; the Interlocking, OfficeUnit and Processor pins, the unit
  sheets' port and labels are Processor.
- IOBus on the Processor pin; the office side is PanelIOBus on the unit ports, the Panel boxes' pins,
  the panel labels and the root sheet pins.
- MAIN HOUSE is House; its H pin is MC and hidden, as asked.
- OfficeUnit Type -> Style = US&S; TimeCode and LocoNet spellings, the LocoNet transport's pin is
  Transport; the one input Codeline sheet pin is bidirectional.
- The CMRInet node's Board -> NodeType (body text follows); JMRI drivers' IC = MQTT-JMRI.

Verified: --check on production/vocab-before.net vs vocab-after.net: identical connectivity under the
pin map, same parts (MAIN HOUSE -> House), only the ruled fields changed; field-io --check passes;
ERC 0 violations.

Co-Authored-By: Claude Fable 5.1 <noreply@anthropic.com>
Connections:
- net IOBus renamed PanelIOBus
Changed lines of the file:
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@@
 		(at 87.63 80.01)
 	)
-	(hierarchical_label "IOBus"
+	(hierarchical_label "PanelIOBus"
 		(shape bidirectional)
 		(at 213.36 111.76 0)
@@
 		)
 	)
-	(hierarchical_label "IOBus"
+	(hierarchical_label "PanelIOBus"
 		(shape bidirectional)
 		(at 111.76 111.76 0)
@@
 		)
 	)
-	(hierarchical_label "IOBus"
+	(hierarchical_label "PanelIOBus"
 		(shape bidirectional)
 		(at 162.56 111.76 0)

Commit message: refactor(kicad): model board lamps leave the columns; stale instance fields follow the libraries; PanelLamp-* retired
The owner's ruling (2026-10-23): the PanelColumn is the logical column, tied to a control point; the panel
I/O hardware is not. Every PanelLamp was a model board lamp except the maintainer-call lamp on the column's
pin 8. 34 lamps are now ModelLamp-<color> (no Column pin, Style board); 8 MC lamps are PanelMCall-Lamp.
Wires untouched: ~{LAMP} keeps its pin and the Column wire of a model lamp ends on nothing. Instance fields
the libraries dropped in c1d446b are gone from the sheets: Address on 7 processors, Interlocking and Machine
on 14 columns, Host on 2 transports. Railroad stays on the AAR encoding because its Topic template reads
${Railroad}; where Railroad lives is pending. Cached definitions refreshed for Processor, PanelColumn,
Transport-MQTT and Encoding-AAR. Scripted: SPCoast/edits/2026-10-23-model-lamps.py (edit, --check, --retire).

Verified: the script's gate on production/fields-after.net vs model-lamps-after.net: same 743 parts, lib ids
change only on the 42 lamps to the expected targets, fields change only as listed (Style indication->board
x34, the 37 drops), connectivity after == before minus the model lamps' pin 1, ERC 0 violations (the two
lib_symbol_mismatch warnings gone). lint_symbol_fields: 97 symbols, 0 errors (PanelLamp-BLUE, -GREEN, -RED, -YELLOW retired; there was no AMBER). Subdivision tests: 157 OK.

Co-Authored-By: Claude Fable 5.1 <noreply@anthropic.com>
Parts:
- COL10028, COL10029, COL10030: Interlocking Christopher -> (none); Machine SPCoast South -> (none)
- LMP10081, LMP10083, LMP10101, LMP10102: symbol Railroad-Office:PanelLamp-YELLOW -> Railroad-Office:ModelLamp-YELLOW; Style indication -> board
- LMP10082, LMP10091, LMP10092, LMP10093: symbol Railroad-Office:PanelLamp-RED -> Railroad-Office:ModelLamp-RED; Style indication -> board
- MCK10008, MCK10010: symbol Railroad-Office:PanelLamp-YELLOW -> Railroad-Office:PanelMCall-Lamp
Connections:
- net at COL10029.1 (Column): no longer LMP10091.1 (Column)
- net at COL10030.2 (Column): no longer LMP10102.1 (Column)
- net at COL10028.3 (Column): no longer LMP10083.1 (Column)
- net at COL10030.3 (Column): no longer LMP10093.1 (Column)
- net at COL10028.2 (Column): no longer LMP10082.1 (Column)
- net at COL10030.1 (Column): no longer LMP10101.1 (Column)
- net at COL10028.1 (Column): no longer LMP10081.1 (Column)
- net at COL10029.2 (Column): no longer LMP10092.1 (Column)

Commit message: refactor(kicad): Name on every device, office unit and encoding; Kind on the JMRI drivers; Driver-JMRI-Light
The owner's rulings of 2026-10-24 on the review of ADR 0008 rev 4: Name = ${Value}
is the identity key everywhere, devices included; the OfficeUnit's Columns is
derived and struck; a JMRI driver carries no address and is keyed by its object
class and the device it serves, the class carried by Kind (TURNOUT, SENSOR,
SIGNALMAST, LIGHT); Driver-JMRI-Light (ADR 0005 §8: ON, INTENSITY) for a lamp
JMRI drives, and the two Gilroy Interchange maintainer-call lamps MC1 and MC2
become Lights (they were Sensors, which JMRI only displays).

Script: SPCoast/edits/2026-10-24-names-kind-light.py. Libraries: Name on 36
symbols (OfficeUnit, 5 encodings, 12 PANEL, 18 DEVICE), Columns off OfficeUnit,
Kind on 5 JMRI drivers, Driver-JMRI-Light added (the Sensor's pin positions,
INTENSITY as pin 3 below, no-connect on the two placed instances). Sheets: 359
Name instance fields, 16 Kind, 2 lib_id swaps, caches refreshed (no pin moved on
a refreshed symbol).

Verified: gate --check production/SPCoast.net production/names-after.net PASS:
same parts, same connectivity, Name == Value on all 273 named instances (47
heads with Value "~" resolve to an empty Name), Columns dropped once, Kind on 16
drivers, 2 Sensor -> Light with pin 1 reading ON; ERC 0 before and after.
Subdivision lint_symbol_fields: 99 symbols, 0 errors (Kind now allowed on
IODRIVER). production/SPCoast.net is the new export (production/ is untracked).

Co-Authored-By: Claude Fable 5.1 <noreply@anthropic.com>
Parts:
- CDE10010, LKL10008, LKL10010, LMP10081, LMP10082, LMP10083, LMP10091, LMP10092, LMP10093, LMP10101, LMP10102, MCK10008, MCK10010, MCL10008, MCL10010, SGL10009, SWL10009: Name (none) -> ${Value}
Changed lines of the file:
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@@
 			)
 		)
+		(property "Name" "${Value}"
+			(at 130.81 83.82 0)
+			(hide yes)
+			(show_name no)
+			(do_not_autoplace no)
+			(effects
+				(font
+					(size 1.27 1.27)
+				)
+			)
+		)
 		(property "Appliance" "lever"
 			(at 130.81 92.71 0)
@@
 			)
 		)
+		(property "Name" "${Value}"
+			(at 181.61 104.14 0)
+			(hide yes)
+			(show_name no)
+			(do_not_autoplace no)
+			(effects
+				(font
+					(size 1.27 1.27)
+				)
+			)
+		)
 		(property "Appliance" "lamp"
 			(at 181.61 101.6 0)
@@
 			)
 		)
+		(property "Name" "${Value}"
+			(at 130.81 26.67 0)
+			(hide yes)
+			(show_name no)
+			(do_not_autoplace no)
+			(effects
+				(font
+					(size 1.27 1.27)
+				)
+			)
+		)
 		(property "Appliance" "lamp"
 			(at 130.81 29.21 0)
@@
 			)
 		)
+		(property "Name" "${Value}"
+			(at 181.61 31.75 0)
+			(hide yes)
+			(show_name no)
+			(do_not_autoplace no)
+			(effects
+				(font
+					(size 1.27 1.27)
+				)
+			)
+		)
 		(property "Appliance" "lamp"
 			(at 181.61 29.21 0)
@@
 			)
 		)
+		(property "Name" "${Value}"
+			(at 80.01 36.83 0)
+			(hide yes)
+			(show_name no)
+			(do_not_autoplace no)
+			(effects
+				(font
+					(size 1.27 1.27)
+				)
+			)
+		)
 		(property "Appliance" "lamp"
 			(at 80.01 34.29 0)
@@
 			)
 		)
+		(property "Name" "${Value}"
+			(at 80.01 63.5 0)
+			(hide yes)
+			(show_name no)
+			(do_not_autoplace no)
+			(effects
+				(font
+					(size 1.27 1.27)
+				)
+			)
+		)
 		(property "Appliance" "lever"
 			(at 80.645 74.93 0)
@@
 			)
 		)
+		(property "Name" "${Value}"
+			(at 130.81 83.82 0)
+			(hide yes)
+			(show_name no)
+			(do_not_autoplace no)
+			(effects
+				(font
+					(size 1.27 1.27)
+				)
+			)
+		)
 		(property "Appliance" "lever"
 			(at 130.81 92.71 0)
@@
 			)
 		)
+		(property "Name" "${Value}"
+			(at 181.61 36.83 0)
+			(hide yes)
+			(show_name no)
+			(do_not_autoplace no)
+			(effects
+				(font
+					(size 1.27 1.27)
+				)
+			)
+		)
 		(property "Appliance" "lamp"
 			(at 181.61 39.37 0)
@@
 			)
 		)
+		(property "Name" "${Value}"
+			(at 80.01 31.75 0)
+			(hide yes)
+			(show_name no)
+			(do_not_autoplace no)
+			(effects
+				(font
+					(size 1.27 1.27)
+				)
+			)
+		)
 		(property "Appliance" "lamp"
 			(at 80.01 34.29 0)
@@
 			)
 		)
+		(property "Name" "${Value}"
+			(at 80.01 26.67 0)
+			(hide yes)
+			(show_name no)
+			(do_not_autoplace no)
+			(effects
+				(font
+					(size 1.27 1.27)
+				)
+			)
+		)
 		(property "Appliance" "lamp"
 			(at 80.01 24.13 0)
@@
 			)
 		)
+		(property "Name" "${Value}"
+			(at 181.61 97.79 0)
+			(hide yes)
+			(show_name no)
+			(do_not_autoplace no)
+			(effects
+				(font
+					(size 1.27 1.27)
+				)
+			)
+		)
 		(property "Appliance" "lever"
 			(at 181.61 90.17 0)
@@
 			)
 		)
+		(property "Name" "${Value}"
+			(at 181.61 63.5 0)
+			(hide yes)
+			(show_name no)
+			(do_not_autoplace no)
+			(effects
+				(font
+					(size 1.27 1.27)
+				)
+			)
+		)
 		(property "Appliance" "lever"
 			(at 182.245 74.93 0)
@@
 			)
 		)
+		(property "Name" "${Value}"
+			(at 80.01 63.5 0)
+			(hide yes)
+			(show_name no)
+			(do_not_autoplace no)
+			(effects
+				(font
+					(size 1.27 1.27)
+				)
+			)
+		)
 		(property "Appliance" "lever"
 			(at 80.645 74.93 0)
@@
 			)
 		)
+		(property "Name" "${Value}"
+			(at 80.01 104.14 0)
+			(hide yes)
+			(show_name no)
+			(do_not_autoplace no)
+			(effects
+				(font
+					(size 1.27 1.27)
+				)
+			)
+		)
 		(property "Appliance" "lamp"
 			(at 80.01 101.6 0)
@@
 			)
 		)
+		(property "Name" "${Value}"
+			(at 130.81 63.5 0)
+			(hide yes)
+			(show_name no)
+			(do_not_autoplace no)
+			(effects
+				(font
+					(size 1.27 1.27)
+				)
+			)
+		)
 		(property "Appliance" "lever"
 			(at 131.445 76.2 0)
@@
 			)
 		)
+		(property "Name" "${Value}"
+			(at 130.81 31.75 0)
+			(hide yes)
+			(show_name no)
+			(do_not_autoplace no)
+			(effects
+				(font
+					(size 1.27 1.27)
+				)
+			)
+		)
 		(property "Appliance" "lamp"
 			(at 130.81 34.29 0)
@@
 			)
 		)
+		(property "Name" "${Value}"
+			(at 181.61 48.26 0)
+			(hide yes)
+			(show_name no)
+			(do_not_autoplace no)
+			(effects
+				(font
+					(size 1.27 1.27)
+				)
+			)
+		)
 		(property "Appliance" "lever"
 			(at 187.96 44.45 0)
@@
 			)
 		)
+		(property "Name" "${Value}"
+			(at 80.01 48.26 0)
+			(hide yes)
+			(show_name no)
+			(do_not_autoplace no)
+			(effects
+				(font
+					(size 1.27 1.27)
+				)
+			)
+		)
 		(property "Appliance" "lever"
 			(at 86.36 44.45 0)
@@
 			)
 		)
+		(property "Name" "${Value}"
+			(at 181.61 63.5 0)
+			(hide yes)
+			(show_name no)
+			(do_not_autoplace no)
+			(effects
+				(font
+					(size 1.27 1.27)
+				)
+			)
+		)
 		(property "Appliance" "lever"
 			(at 182.245 74.93 0)
@@
 			)
 		)
+		(property "Name" "${Value}"
+			(at 181.61 26.67 0)
+			(hide yes)
+			(show_name no)
+			(do_not_autoplace no)
+			(effects
+				(font
+					(size 1.27 1.27)
+				)
+			)
+		)
 		(property "Appliance" "lamp"
 			(at 181.61 24.13 0)
@@
 			(hide yes)
 			(show_name no)
+			(do_not_autoplace no)
+			(effects
+				(font
+					(size 1.27 1.27)
+				)
+			)
+		)
+		(property "Name" "${Value}"
+			(at 130.81 63.5 0)
+			(hide yes)
+			(show_name no)

Commit message: feat(spcoast): every desk column names its CP Name
The owner's edit in KiCad: each PanelColumn carries a CP Name. On an
AAR codeline it may name the interlocking (Christopher, Gilroy
Interchange); on the 506 it names the house.

Verified: a fresh kicad-cli netlist compiles with no column.cp_name
diagnostics; the three column.house errors (columns 3, 4, 9) are
resolved by the importer rule, not the drawing.

Co-Authored-By: Claude Opus 5.5 <noreply@anthropic.com>
Parts:
- COL10028: CP Name (none) -> Christopher North
- COL10029: CP Name (none) -> Christopher
- COL10030: CP Name (none) -> Christopher South
Changed lines of the file:
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@@
 			)
 		)
-		(property "CP Name" ""
+		(property "CP Name" "Christopher South"
 			(at 182.245 132.08 0)
 			(show_name yes)
@@
 			)
 		)
-		(property "CP Name" ""
+		(property "CP Name" "Christopher"
 			(at 131.445 132.08 0)
 			(show_name yes)
@@
 			)
 		)
-		(property "CP Name" ""
+		(property "CP Name" "Christopher North"
 			(at 80.645 132.08 0)
 			(show_name yes)

Commit message: feat(spcoast): per-pin token fields on the panels, lamp Indication expressions, maintainer calls named 1MC
Applies the symbol rulings of 2026-10-28 to every sheet: the lib_symbols
caches of the changed symbols are the library's copies (this also clears
the stale PanelMCall and MaintainerCall caches), and every placed
instance gets the new hidden Control.*/Indication.* fields, loses
PanelLock Invert, and PanelMCall's whole-symbol Control and Indication
(Pin.MCK binary). Model lamps' IndicationToken becomes Indication: each
comma-separated circuit gets its K, qualifiers kept, joined with " | "
(795T1,01T,799T1 -> 795T1K | 01TK | 799T1K).

Maintainer calls in Christopher (1, 2), Corporal, Luchessa and Sargent
follow Gilroy Interchange (5dad54f): Value MC<n> -> <n>, Name ${Value}MC,
and the separate PanelMCall-Lamp is replaced by unit 2 of the same
PanelMCall at the old lamp's position, so its MCK pin sits where the
LAMP pin was. The old lamps' Column pin touched PanelColumn pin 8
directly (no wire); that pin is now unconnected, as on Gilroy
Interchange. Gilroy Interchange's local MaintainerCall_1 cache and its
two trackplan calls lose Indication.

Verified: fresh netlist before/after: components 752 -> 747 (the five
lamps), nets 1028 -> 1028; each old LAMP-pin net now holds the lever's
unit-2 MCK pin (pin 3) on the same expander pin (B1, pin 9); the levers'
nets are renamed only (~{S} -> ~{MCS}, unit suffix A); no other net
changed. Every field difference is an intended one. ERC 18 -> 1
violations (lib_symbol_mismatch 17 -> 0; pre-existing Sargent AUX1
pin_not_connected remains).

Co-Authored-By: Claude Opus 5.5 <noreply@anthropic.com>
Parts:
- removed MCK10008, MCK10010: MC, symbol Railroad-Office:PanelMCall-Lamp
- added unit 2 of MCL10008
- added unit 2 of MCL10010
- LKL10008, LKL10010: Control.WLS (none) -> ${Value}WLS; Indication.WLK (none) -> !${Value}WLK; Indication.WLQK (none) -> ${Value}WLQK; Invert WLK -> (none)
- LMP10081: Indication (none) -> 1SATK; IndicationToken 1SAT -> (none)
- LMP10082: Indication (none) -> 813T1K; IndicationToken 813T1 -> (none)
- LMP10083: Indication (none) -> 2SATK; IndicationToken 2SAT -> (none)
- LMP10091: Indication (none) -> 815T1K; IndicationToken 815T1 -> (none)
- LMP10092: Indication (none) -> 815AT1K; IndicationToken 815AT1 -> (none)
- LMP10093: Indication (none) -> 817T1K; IndicationToken 817T1 -> (none)
- LMP10101: Indication (none) -> 1NATK; IndicationToken 1NAT -> (none)
- LMP10102: Indication (none) -> 2NATK; IndicationToken 2NAT -> (none)
- MCL10008: value MC1 -> 1; Control.MCS (none) -> ${Value}MCS; Indication.MCK (none) -> ${Value}MCK; Name ${Value} -> ${Value}MC; Pin.MCK (none) -> binary; Pin.MCS (none) -> binary; Pin.S binary -> (none)
- MCL10010: value MC2 -> 2; Control.MCS (none) -> ${Value}MCS; Indication.MCK (none) -> ${Value}MCK; Name ${Value} -> ${Value}MC; Pin.MCK (none) -> binary; Pin.MCS (none) -> binary; Pin.S binary -> (none)
- SGL10009: Control.HS (none) -> ${Value}HS; Control.NGS (none) -> ${Value}NGS; Control.SGS (none) -> ${Value}SGS; Indication.NGK (none) -> ${Value}NGK; Indication.SGK (none) -> ${Value}SGK; Indication.TEK (none) -> ${Value}TEK
- SWL10009: Control.NWS (none) -> ${Value}NWS; Control.RWS (none) -> ${Value}RWS; Indication.NWK (none) -> ${Value}NWK; Indication.RWK (none) -> ${Value}RWK
Connections:
- net at U10030.9 (B1): now also MCL10010.3 (~{MCK})
- net at U10028.9 (B1): now also MCL10008.3 (~{MCK})
