File: SPCoast/Christopher.kicad_sch (KiCad schematic)
At the start: 42 parts, among them SW9813 813, SW9815 815, SW9817 817, SW9900 815A

Commit message: chore(kicad): owner mockup: explicit seam wiring on Luchessa and South-cTc, host and bus pins
Owner's edits, committed as they stand (2026-10-21), before scripted edits build on them.

- Interlocking gains Codeline and Host pins; MAIN HOUSE's Interlocking pin is Codeline.
- OfficeUnit gains Host and Codeline pins; JohnCTC desk processor drawn on South-cTc.
- Processor gains Transport and IO pins; MAX7313 and MCP23017 gain an I2C bus pin.
- Transports: Codeline pin renamed Host; JMRI_MQTT instance added; Loconet removed.
- Encodings' pin renamed Transport; Luchessa's 506 and Bit Packing instances removed.
- SPCoastApp virtual host (FieldUnit_Virtual) hosts CMRInet and JMRI_MQTT.
- Luchessa: unit, houses and Time Coded on one net; Host to its own processor;
  panel MAX7313s on the desk bus (OfficeBus).
- Watsonville, Caltrain, Interchange: first-pass Processor placeholders, to be redrawn.

Verified: netlist and ERC exported from the saved project; field diff against the
committed netlist shows no per-instance field lost.
Changed lines of the file:
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@@
 		(pin "1"
+		)
+		(pin "2"
 		)
 		(instances
