File: SPCoast/Christopher.kicad_sch (KiCad schematic)
At the start: 72 parts, among them SW9813 813, SW9815 815, SW9817 817, SW9900 815A, SW9901 813, SW9902 817

Commit message: chore(kicad): owner edits: CMRInet node on the transport net, sheet tidying (2026-10-23)
Changed lines of the file:
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@@
 		)
 	)
-	(hierarchical_label "Codeline"
-		(shape bidirectional)
-		(at 86.36 39.37 0)
+	(label "IOBus"
+		(at 86.36 34.29 0)
 		(effects
 			(font
@@
 	)
 	(label "IOBus"
-		(at 86.36 34.29 0)
+		(at 200.66 137.16 0)
 		(effects
 			(font
@@
 	)
 	(label "IOBus"
-		(at 200.66 137.16 0)
+		(at 256.54 137.16 0)
 		(effects
 			(font
@@
 	)
 	(label "IOBus"
-		(at 256.54 137.16 0)
+		(at 87.63 137.16 0)
 		(effects
 			(font
@@
 		)
 	)
-	(hierarchical_label "PanelIOBus"
-		(shape bidirectional)
-		(at 86.36 26.67 0)
+	(label "IOBus"
+		(at 144.78 137.16 0)
 		(effects
 			(font
@@
 		)
 	)
-	(label "IOBus"
-		(at 87.63 137.16 0)
+	(hierarchical_label "Codeline"
+		(shape bidirectional)
+		(at 86.36 39.37 0)
 		(effects
 			(font
@@
 		)
 	)
-	(label "IOBus"
-		(at 144.78 137.16 0)
+	(hierarchical_label "PanelIOBus"
+		(shape bidirectional)
+		(at 86.36 26.67 0)
 		(effects
 			(font
@@
 		)
 		(property "Value" "Christopher"
-			(at 57.15 31.75 0)
+			(at 55.88 34.036 0)
 			(show_name no)
 			(do_not_autoplace yes)
@@
 					(size 1.27 1.27)
 				)
-				(justify left)
 			)
 		)
@@
 			(hide yes)
 			(show_name no)
+			(do_not_autoplace no)
+			(effects
+				(font
+					(size 1.27 1.27)
+				)
+			)
+		)
+		(property "Address" ""
+			(at 57.15 29.21 0)
+			(hide yes)
+			(show_name no)
