File: SPCoast/Christopher.kicad_sch (KiCad schematic)
At the start: 72 parts, among them SW9813 813, SW9815 815, SW9817 817, SW9900 815A, SW9901 813, SW9902 817

Commit message: refactor(kicad): head devices are DEVICE with Appliance head; the OfficeUnit's Role is OFFICE_UNIT; stale instance Roles follow the libraries
SPCoast/edits/2026-10-23-roles.py, ADR 0009 §3.10 as approved: CAST and MACHINE were implementation
words. The seven Device-Head-* symbols and their 57 placed instances carry Role DEVICE and Appliance head;
the OfficeUnit carries OFFICE_UNIT; the four transport instances still saying CODELINE_TRANSPORT say
TRANSPORT. Descriptions: Device-Switch loses "cast", the JMRI drivers say FieldUnit, the OfficeUnit says
what it is. Every cached definition that differed from its library copy refreshed.

Verified: netlist connectivity and parts identical; no field changed beyond Role, Appliance and
Description; no CAST, MACHINE or CODELINE_TRANSPORT remains on any instance; ERC 0.

Co-Authored-By: Claude Fable 5.1 <noreply@anthropic.com>
Parts:
- Cast9001, Cast9002, Cast9003, Cast9004, Cast9005, Cast9006: Appliance (none) -> head; Role CAST -> DEVICE
Changed lines of the file:
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@@
 			)
 		)
-		(property "Role" "CAST"
+		(property "Role" "DEVICE"
 			(at 53.34 152.019 0)
 			(hide yes)
@@
 			)
 		)
+		(property "Appliance" "head"
+			(at 64.77 156.21 0)
+			(hide yes)
+			(show_name no)
+			(do_not_autoplace no)
+			(effects
+				(font
+					(size 1.27 1.27)
+				)
+			)
+		)
 		(property "Style" "CPL"
 			(at 53.34 151.257 0)
@@
 			)
 		)
-		(property "Role" "CAST"
+		(property "Role" "DEVICE"
 			(at 53.34 141.859 0)
 			(hide yes)
@@
 			)
 		)
+		(property "Appliance" "head"
+			(at 64.77 146.05 0)
+			(hide yes)
+			(show_name no)
+			(do_not_autoplace no)
+			(effects
+				(font
+					(size 1.27 1.27)
+				)
+			)
+		)
 		(property "Style" "CPL"
 			(at 53.34 141.097 0)
@@
 			)
 		)
-		(property "Role" "CAST"
+		(property "Role" "DEVICE"
 			(at 53.34 136.779 0)
 			(hide yes)
@@
 			)
 		)
+		(property "Appliance" "head"
+			(at 64.77 140.97 0)
+			(hide yes)
+			(show_name no)
+			(do_not_autoplace no)
+			(effects
+				(font
+					(size 1.27 1.27)
+				)
+			)
+		)
 		(property "Style" "CPL"
 			(at 53.34 136.017 0)
@@
 			)
 		)
-		(property "Role" "CAST"
+		(property "Role" "DEVICE"
 			(at 53.34 146.939 0)
 			(hide yes)
@@
 			)
 		)
+		(property "Appliance" "head"
+			(at 64.77 151.13 0)
+			(hide yes)
+			(show_name no)
+			(do_not_autoplace no)
+			(effects
+				(font
+					(size 1.27 1.27)
+				)
+			)
+		)
 		(property "Style" "CPL"
 			(at 53.34 146.177 0)
@@
 			)
 		)
-		(property "Role" "CAST"
+		(property "Role" "DEVICE"
 			(at 53.34 131.699 0)
 			(hide yes)
@@
 			)
 		)
+		(property "Appliance" "head"
+			(at 64.77 135.89 0)
+			(hide yes)
+			(show_name no)
+			(do_not_autoplace no)
+			(effects
+				(font
+					(size 1.27 1.27)
+				)
+			)
+		)
 		(property "Style" "CPL"
 			(at 53.34 130.937 0)
@@
 			)
 		)
-		(property "Role" "CAST"
+		(property "Role" "DEVICE"
 			(at 53.34 126.619 0)
 			(hide yes)
@@
 				)
 			)
+		)
+		(property "Appliance" "head"
+			(at 64.77 130.81 0)
+			(hide yes)
+			(show_name no)
+			(do_not_autoplace no)
+			(effects
+				(font
+					(size 1.27 1.27)
+				)
+			)

Commit message: refactor(kicad): model board lamps leave the columns; stale instance fields follow the libraries; PanelLamp-* retired
The owner's ruling (2026-10-23): the PanelColumn is the logical column, tied to a control point; the panel
I/O hardware is not. Every PanelLamp was a model board lamp except the maintainer-call lamp on the column's
pin 8. 34 lamps are now ModelLamp-<color> (no Column pin, Style board); 8 MC lamps are PanelMCall-Lamp.
Wires untouched: ~{LAMP} keeps its pin and the Column wire of a model lamp ends on nothing. Instance fields
the libraries dropped in c1d446b are gone from the sheets: Address on 7 processors, Interlocking and Machine
on 14 columns, Host on 2 transports. Railroad stays on the AAR encoding because its Topic template reads
${Railroad}; where Railroad lives is pending. Cached definitions refreshed for Processor, PanelColumn,
Transport-MQTT and Encoding-AAR. Scripted: SPCoast/edits/2026-10-23-model-lamps.py (edit, --check, --retire).

Verified: the script's gate on production/fields-after.net vs model-lamps-after.net: same 743 parts, lib ids
change only on the 42 lamps to the expected targets, fields change only as listed (Style indication->board
x34, the 37 drops), connectivity after == before minus the model lamps' pin 1, ERC 0 violations (the two
lib_symbol_mismatch warnings gone). lint_symbol_fields: 97 symbols, 0 errors (PanelLamp-BLUE, -GREEN, -RED, -YELLOW retired; there was no AMBER). Subdivision tests: 157 OK.

Co-Authored-By: Claude Fable 5.1 <noreply@anthropic.com>
Changed lines of the file:
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@@
-			)
-		)
-		(property "Address" ""
-			(at 57.15 29.21 0)
-			(hide yes)
-			(show_name no)
-			(do_not_autoplace no)
-			(effects
-				(font
-					(size 1.27 1.27)
-				)
 			)
 		)

Commit message: refactor(kicad): layout-wide facts on the Railroad symbol; the AAR Topic is the macro ctc/<STRUCTURE:RAILROAD:Name>/codeline/; Name on processors and transports
The owner's rulings (2026-10-23): a Railroad symbol on the root sheet (STRUCTURE/RAILROAD; Name, Railroad, Region,
Era, Rulebook) carries the layout-wide facts; a field may reference another symbol's field with <ROLE:KIND:Field>,
keyed by the fields the libraries key symbols by, resolved to the one instance in scope and expanded by the
compiler, never by KiCad (KIND empty for a Role without one); Name is the identity key everywhere, Value is never
read. The placed AAR encoding loses its Railroad field and its Topic becomes the macro; the library default follows.
The OfficeUnit instance loses Railroad and Era (off the library already). Processor and the four Transport-* gain
Name = ${Value}, library and 12 placed instances. Cached Encoding-AAR, OfficeUnit, Railroad, processors and
transports refreshed; no pin moved. Scripted: SPCoast/edits/2026-10-23-railroad.py (edit, --check).

Verified: the script's gate on production/model-lamps-after.net vs railroad-after.net: connectivity identical;
parts identical but for RAILROAD1; fields change only Topic (the macro, expanded against the one STRUCTURE/RAILROAD
symbol, equals the before value ctc/SPCoast/codeline/), Railroad x2 and Era x1 dropped, Name added on 12
processors and transports with Name == Value; ERC 0 violations. lint_symbol_fields: 98 symbols, 0 errors.

Co-Authored-By: Claude Fable 5.1 <noreply@anthropic.com>
Parts:
- Proc10: Name (none) -> ${Value}
Changed lines of the file:
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@@
+			)
+		)
+		(property "Name" "${Value}"
+			(at 55.88 33.02 0)
+			(hide yes)
+			(show_name no)
+			(do_not_autoplace no)
+			(effects
+				(font
+					(size 1.27 1.27)
+				)
 			)
 		)

Commit message: refactor(kicad): Name on every device, office unit and encoding; Kind on the JMRI drivers; Driver-JMRI-Light
The owner's rulings of 2026-10-24 on the review of ADR 0008 rev 4: Name = ${Value}
is the identity key everywhere, devices included; the OfficeUnit's Columns is
derived and struck; a JMRI driver carries no address and is keyed by its object
class and the device it serves, the class carried by Kind (TURNOUT, SENSOR,
SIGNALMAST, LIGHT); Driver-JMRI-Light (ADR 0005 §8: ON, INTENSITY) for a lamp
JMRI drives, and the two Gilroy Interchange maintainer-call lamps MC1 and MC2
become Lights (they were Sensors, which JMRI only displays).

Script: SPCoast/edits/2026-10-24-names-kind-light.py. Libraries: Name on 36
symbols (OfficeUnit, 5 encodings, 12 PANEL, 18 DEVICE), Columns off OfficeUnit,
Kind on 5 JMRI drivers, Driver-JMRI-Light added (the Sensor's pin positions,
INTENSITY as pin 3 below, no-connect on the two placed instances). Sheets: 359
Name instance fields, 16 Kind, 2 lib_id swaps, caches refreshed (no pin moved on
a refreshed symbol).

Verified: gate --check production/SPCoast.net production/names-after.net PASS:
same parts, same connectivity, Name == Value on all 273 named instances (47
heads with Value "~" resolve to an empty Name), Columns dropped once, Kind on 16
drivers, 2 Sensor -> Light with pin 1 reading ON; ERC 0 before and after.
Subdivision lint_symbol_fields: 99 symbols, 0 errors (Kind now allowed on
IODRIVER). production/SPCoast.net is the new export (production/ is untracked).

Co-Authored-By: Claude Fable 5.1 <noreply@anthropic.com>
Parts:
- Cast9001, Cast9002, Cast9003, Cast9004, Cast9005, Cast9006, DevLamp9001, DevLamp9002, DevMast9001, DevMast9002, DevMast9003, DevMast9004, DevSW9001, DevSW9002, DevSW9003, DevSW9004, DevTC9001, DevTC9002, DevTC9003, DevTC9004, DevTC9005, LK9001, LK9002, SW9901, SW9902: Name (none) -> ${Value}

Commit message: refactor(kicad): Name = ${Value} on every Trackplan appliance, so no key is read from Value
The owner (2026-10-24), on review finding 4: no exception for appliance names
read from Value. Data model keys are functional descriptions of their content
and the symbol attribute names reflect that choice; Value is generic. Every
Railroad-Trackplan APPLIANCE symbol (switches, derails, masts, heads, track
circuits, maintainer calls, auxiliaries) gains Name = ${Value}: the appliance's
own name, a head's letter. The compiler reads Name, never Value.

Script: SPCoast/edits/2026-10-24-trackplan-names.py (library symbols, placed
instances, caches refreshed; no pin moved).

Verified: gate --check production/SPCoast.net production/trackplan-names-after.net
PASS: same parts, lib ids, Values and connectivity; the only field change is Name
added on every Trackplan appliance with Name == Value; ERC 0 before and after.
Subdivision lint_symbol_fields: 99 symbols, 0 errors. production/SPCoast.net is
the new export.

Co-Authored-By: Claude Fable 5.1 <noreply@anthropic.com>
Parts:
- H9003, H9005, H9006, H9008, H9009, H9010, MC9001, MC9002, S9003, S9004, S9005, S9006, SW9813, SW9815, SW9817, SW9900, TC9001, TC9002, TC9003, TC9004, TC9005: Name (none) -> ${Value}
Changed lines of the file:
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@@
 			)
 		)
+		(property "Name" "${Value}"
+			(at 55.88 100.33 0)
+			(hide yes)
+			(show_name no)
+			(do_not_autoplace no)
+			(effects
+				(font
+					(size 1.27 1.27)
+				)
+			)
+		)
 		(property "Appliance" "track_circuit"
 			(at 55.88 100.33 0)
@@
 			)
 		)
+		(property "Name" "${Value}"
+			(at 72.39 71.12 0)
+			(hide yes)
+			(show_name no)
+			(do_not_autoplace no)
+			(effects
+				(font
+					(size 1.27 1.27)
+				)
+			)
+		)
 		(property "Appliance" "mast"
 			(at 72.39 71.12 0)
@@
 			)
 		)
+		(property "Name" "${Value}"
+			(at 194.31 63.5 0)
+			(hide yes)
+			(show_name no)
+			(do_not_autoplace no)
+			(effects
+				(font
+					(size 1.27 1.27)
+				)
+			)
+		)
 		(property "Appliance" "head"
 			(at 194.31 63.5 0)
@@
 			)
 		)
+		(property "Name" "${Value}"
+			(at 132.08 100.33 0)
+			(hide yes)
+			(show_name no)
+			(do_not_autoplace no)
+			(effects
+				(font
+					(size 1.27 1.27)
+				)
+			)
+		)
 		(property "IndicationCeiling" ""
 			(at 145.415 99.695 0)
@@
 			)
 		)
+		(property "Name" "${Value}"
+			(at 83.82 100.33 0)
+			(hide yes)
+			(show_name no)
+			(do_not_autoplace no)
+			(effects
+				(font
+					(size 1.27 1.27)
+				)
+			)
+		)
 		(property "IndicationCeiling" ""
 			(at 97.155 100.965 0)
@@
 			)
 		)
+		(property "Name" "${Value}"
+			(at 71.12 104.14 0)
+			(hide yes)
+			(show_name no)
+			(do_not_autoplace no)
+			(effects
+				(font
+					(size 1.27 1.27)
+				)
+			)
+		)
 		(property "Appliance" "mast"
 			(at 71.12 104.14 0)
@@
 			)
 		)
+		(property "Name" "${Value}"
+			(at 73.66 49.53 0)
+			(hide yes)
+			(show_name no)
+			(do_not_autoplace no)
+			(effects
+				(font
+					(size 1.27 1.27)
+				)
+			)
+		)
 		(property "Appliance" "lamp"
 			(at 69.85 44.45 0)
@@
 			)
 		)
+		(property "Name" "${Value}"
+			(at 130.81 116.84 0)
+			(hide yes)
+			(show_name no)
+			(do_not_autoplace no)
+			(effects
+				(font
+					(size 1.27 1.27)
+				)
+			)
+		)
 		(property "Appliance" "track_circuit"
 			(at 130.81 116.84 0)
@@
 			)
 		)
+		(property "Name" "${Value}"
+			(at 193.04 96.52 0)
+			(hide yes)
+			(show_name no)
+			(do_not_autoplace no)
+			(effects
+				(font
+					(size 1.27 1.27)
+				)
+			)
+		)
 		(property "Appliance" "head"
 			(at 193.04 96.52 0)
@@
 			)
 		)
+		(property "Name" "${Value}"
+			(at 170.18 67.31 0)
+			(hide yes)
+			(show_name no)
+			(do_not_autoplace no)
+			(effects
+				(font
+					(size 1.27 1.27)
+				)
+			)
+		)
 		(property "IndicationCeiling" ""
 			(at 156.845 67.945 0)
@@
 			)
 		)
+		(property "Name" "${Value}"
+			(at 74.93 104.14 0)
+			(hide yes)
+			(show_name no)
+			(do_not_autoplace no)
+			(effects
+				(font
+					(size 1.27 1.27)
+				)
+			)
+		)
 		(property "Appliance" "head"
 			(at 74.93 104.14 0)
@@
 			)
 		)
+		(property "Name" "${Value}"
+			(at 196.85 49.53 0)
+			(hide yes)
+			(show_name no)
+			(do_not_autoplace no)
+			(effects
+				(font
+					(size 1.27 1.27)
+				)
+			)
+		)
 		(property "Appliance" "lamp"
 			(at 193.04 44.45 0)
@@
 			)
 		)
+		(property "Name" "${Value}"
+			(at 210.82 67.31 0)
+			(hide yes)
+			(show_name no)
+			(do_not_autoplace no)
+			(effects
+				(font
+					(size 1.27 1.27)
+				)
+			)
+		)
 		(property "Appliance" "track_circuit"
 			(at 210.82 67.31 0)
@@
 			)
 		)
+		(property "Name" "${Value}"
+			(at 72.39 104.14 0)
+			(hide yes)
+			(show_name no)
+			(do_not_autoplace no)
+			(effects
+				(font
+					(size 1.27 1.27)
+				)
+			)
+		)
 		(property "Appliance" "head"
 			(at 72.39 104.14 0)
@@
 			)
 		)
+		(property "Name" "${Value}"
+			(at 196.85 96.52 0)
+			(hide yes)
+			(show_name no)
+			(do_not_autoplace no)
+			(effects
+				(font
+					(size 1.27 1.27)
+				)
+			)
+		)
 		(property "Appliance" "mast"
 			(at 196.85 96.52 0)
@@
 			)
 		)
+		(property "Name" "${Value}"
+			(at 210.82 100.33 0)
+			(hide yes)
+			(show_name no)
+			(do_not_autoplace no)
+			(effects
+				(font
+					(size 1.27 1.27)
+				)
+			)
+		)
 		(property "Appliance" "track_circuit"
 			(at 210.82 100.33 0)
@@
 			)
 		)
+		(property "Name" "${Value}"
+			(at 76.2 71.12 0)
+			(hide yes)
+			(show_name no)
+			(do_not_autoplace no)
+			(effects
+				(font
+					(size 1.27 1.27)
+				)
+			)
+		)
 		(property "Appliance" "head"
 			(at 76.2 71.12 0)
@@
 			)
 		)
+		(property "Name" "${Value}"
+			(at 184.15 100.33 0)
+			(hide yes)
+			(show_name no)
+			(do_not_autoplace no)
+			(effects
+				(font
+					(size 1.27 1.27)
+				)
+			)
+		)
 		(property "IndicationCeiling" ""
 			(at 170.815 100.965 0)
@@
 			)
 		)
+		(property "Name" "${Value}"
+			(at 191.77 63.5 0)
+			(hide yes)
+			(show_name no)
+			(do_not_autoplace no)
+			(effects
+				(font
+					(size 1.27 1.27)
+				)
+			)
+		)
 		(property "Appliance" "head"
 			(at 191.77 63.5 0)
@@
 			)
 		)
+		(property "Name" "${Value}"
+			(at 195.58 63.5 0)
+			(hide yes)
+			(show_name no)
+			(do_not_autoplace no)
+			(effects
+				(font
+					(size 1.27 1.27)
+				)
+			)
+		)
 		(property "Appliance" "mast"
 			(at 195.58 63.5 0)
@@
 			(at 55.88 67.31 0)
 			(hide yes)
+			(show_name no)
+			(do_not_autoplace no)
+			(effects
+				(font
+					(size 1.27 1.27)
+				)
+			)
+		)
+		(property "Name" "${Value}"
+			(at 55.88 67.31 0)
+			(hide yes)
