File: SPCoast/GilroyCalTrain-Panel.kicad_sch (KiCad schematic)
At the start: 15 parts, among them U4021 ${ADDRESS}, U4022 ${ADDRESS}

Commit message: feat(kicad): explicit seams on every sheet: Codeline and Host wires, remote I/O attachments, CP Name
The Luchessa pattern (owner mockup 5288025) applied to the whole project by
SPCoast/edits/2026-10-21-explicit-seams.py, gated by its -gate.py.

Libraries
- Processor: pins Host (passive) and IO_Bus; Transport and Address fields dropped.
- Processor-Virtual (Role STRUCTURE, Kind PROCESSOR, Type VIRTUAL, Host pin, no bus),
  Remote-IO-CMRInet and Remote-IO-JMRI (Kind REMOTE_IO, Board, Address, Transport pin).
- Transports: attachment pin Encoding -> Transport; MQTT loses Station. Encodings lose
  Station and Address. FieldUnit and FieldUnit_Virtual removed. OfficeUnit's Host pin numbered.
- MAIN HOUSE: CP Name, the one key every join reads; Value is a display macro of it.

Sheets
- Every unit: Interlocking Codeline and Host as hierarchical pins; houses on the Codeline net.
  Luchessa rides Time Coded, every other unit MQTT (AAR Tokens). Luchessa and Sargent host
  themselves; Watsonville, Caltrain, Interchange, Corporal, Christopher run on SPCoastApp.
- Caltrain: the Processor placeholder is Remote-IO-CMRInet 'Caltrain' (cpNode, UA 30) on
  CMRInet. Interchange: Remote-IO-JMRI 'JMRI' on JMRI_MQTT. Their Codeline ports now go to
  MQTT, not to the I/O transports. Watsonville's placeholder removed.
- South-cTc: SPCoastApp is a Processor-Virtual hosting the two I/O transports and five units;
  ten sheet pins with labels and wires; JohnCTC loses the node fields.
- Luchessa: 17 appliances' CP 'CP X' -> 'X', matching the panel columns' CP Name.
- GilroyCalTrain-Panel: a stray, unconnected AAR Tokens instance (Station Luchessa) removed.

Verified: gate passed on production/explicit-seams-before.net vs -after.net: every unit's
Codeline and Host net is exactly as expected, remote I/O and desk bus nets as expected,
connectivity away from the seams unchanged, no field changed except where the ruling says,
parts removed Proc1-3/HOST1/Encoding1 and added RIO1/RIO2/Proc6/Proc7. ERC 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
Parts:
- removed Encoding1: AAR Tokens, symbol Railroad-Office:Codeline-Encoding-AAR
Changed lines of the file:
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@@
-	)
-	(symbol
-		(lib_id "Railroad-Office:Codeline-Encoding-AAR")
-		(at 27.94 180.34 0)
-		(unit 1)
-		(body_style 1)
-		(exclude_from_sim no)
-		(in_bom yes)
-		(on_board yes)
-		(in_pos_files yes)
-		(dnp no)
-		(fields_autoplaced yes)
-		(property "Reference" "Encoding1"
-			(at 34.925 193.04 0)
-			(hide yes)
-			(show_name no)
-			(do_not_autoplace no)
-			(effects
-				(font
-					(size 1.27 1.27)
-				)
-			)
-		)
-		(property "Value" "AAR Tokens"
-			(at 40.64 182.245 0)
-			(show_name no)
-			(do_not_autoplace yes)
-			(effects
-				(font
-					(size 1.27 1.27)
-				)
-				(justify right)
-			)
-		)
-		(property "Footprint" ""
-			(at 27.94 180.34 0)
-			(hide yes)
-			(show_name no)
-			(do_not_autoplace no)
-			(effects
-				(font
-					(size 1.27 1.27)
-				)
-			)
-		)
-		(property "Datasheet" ""
-			(at 27.94 180.34 0)
-			(hide yes)
-			(show_name no)
-			(do_not_autoplace no)
-			(effects
-				(font
-					(size 1.27 1.27)
-				)
-			)
-		)
-		(property "Description" "Advanced Train Control System protocol AAR Specification 250 Message Formats"
-			(at 41.91 194.945 0)
-			(hide yes)
-			(show_name no)
-			(do_not_autoplace no)
-			(effects
-				(font
-					(size 1.27 1.27)
-				)
-			)
-		)
-		(property "Role" "CODELINE_ENCODING"
-			(at 27.94 177.8 0)
-			(hide yes)
-			(show_name no)
-			(do_not_autoplace no)
-			(effects
-				(font
-					(size 1.27 1.27)
-				)
-			)
-		)
-		(property "Kind" "AAR"
-			(at 41.91 193.04 0)
-			(hide yes)
-			(show_name no)
-			(do_not_autoplace yes)
-			(effects
-				(font
-					(size 1.27 1.27)
-				)
-				(justify left)
-			)
-		)
-		(property "Station" "Luchessa"
-			(at 33.655 184.785 0)
-			(show_name no)
-			(do_not_autoplace yes)
-			(effects
-				(font
-					(size 1.27 1.27)
-				)
-				(justify left)
-			)
-		)
-		(pin "1"
-		)
-		(instances
-			(project "SPCoast"
-				(path "/528348b2-add8-5367-a5f7-439c76f0ca33/2ed995e3-3819-55cd-b8d9-5c2af048ccb4/61cd2495-14f3-42a6-a7c2-38f34b91ee1e/8ecebbd2-e7a6-5949-8793-5f9acfb44e33"
-					(reference "Encoding1")
-					(unit 1)
-				)
-			)
-		)
 	)
 	(symbol
