File: SPCoast/GilroyCalTrain-Panel.kicad_sch (KiCad schematic)
At the start: 14 parts, among them U4021 ${ADDRESS}, U4022 ${ADDRESS}

Commit message: refactor(kicad): model board lamps leave the columns; stale instance fields follow the libraries; PanelLamp-* retired
The owner's ruling (2026-10-23): the PanelColumn is the logical column, tied to a control point; the panel
I/O hardware is not. Every PanelLamp was a model board lamp except the maintainer-call lamp on the column's
pin 8. 34 lamps are now ModelLamp-<color> (no Column pin, Style board); 8 MC lamps are PanelMCall-Lamp.
Wires untouched: ~{LAMP} keeps its pin and the Column wire of a model lamp ends on nothing. Instance fields
the libraries dropped in c1d446b are gone from the sheets: Address on 7 processors, Interlocking and Machine
on 14 columns, Host on 2 transports. Railroad stays on the AAR encoding because its Topic template reads
${Railroad}; where Railroad lives is pending. Cached definitions refreshed for Processor, PanelColumn,
Transport-MQTT and Encoding-AAR. Scripted: SPCoast/edits/2026-10-23-model-lamps.py (edit, --check, --retire).

Verified: the script's gate on production/fields-after.net vs model-lamps-after.net: same 743 parts, lib ids
change only on the 42 lamps to the expected targets, fields change only as listed (Style indication->board
x34, the 37 drops), connectivity after == before minus the model lamps' pin 1, ERC 0 violations (the two
lib_symbol_mismatch warnings gone). lint_symbol_fields: 97 symbols, 0 errors (PanelLamp-BLUE, -GREEN, -RED, -YELLOW retired; there was no AMBER). Subdivision tests: 157 OK.

Co-Authored-By: Claude Fable 5.1 <noreply@anthropic.com>
Parts:
- COL4021, COL4022: Interlocking Gilroy Caltrain -> (none); Machine SPCoast South -> (none)
- LMP4011: symbol Railroad-Office:PanelLamp-RED -> Railroad-Office:ModelLamp-RED; Style indication -> board
- LMP4012, LMP4021, LMP4022, LMP4023: symbol Railroad-Office:PanelLamp-YELLOW -> Railroad-Office:ModelLamp-YELLOW; Style indication -> board
- MCK4001: symbol Railroad-Office:PanelLamp-YELLOW -> Railroad-Office:PanelMCall-Lamp
Connections:
- net at COL4021.1 (Column): no longer LMP4011.1 (Column)
- net at COL4021.2 (Column): no longer LMP4012.1 (Column)
- net at COL4022.1 (Column): no longer LMP4021.1 (Column)
- net at COL4022.2 (Column): no longer LMP4022.1 (Column)
- net at COL4022.3 (Column): no longer LMP4023.1 (Column)
Changed lines of the file:
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@@
 	)
 	(symbol
-		(lib_id "Railroad-Office:PanelLamp-RED")
+		(lib_id "Railroad-Office:ModelLamp-RED")
 		(at 80.01 26.67 0)
 		(unit 1)
@@
 			)
 		)
-		(property "Description" "One physical model board lamp. Value is a free descriptive label (e.g. OS, TRACK, MC) and is not used elsewhere. IndicationToken is a comma-separated list of indication names (track circuits such as 795T1,2NAA,799T1, or tokens such as MC1K) OR'd to drive this one lamp. All listed indications are still individually on the CodeLine wire"
+		(property "Description" "One physical model board lamp. Value is a free descriptive label (e.g. OS, TRACK ...) and is not used elsewhere. IndicationToken is a comma-separated list of indication names (tokens from the CodeLine) OR'd to drive this one lamp."
 			(at 79.375 36.195 0)
 			(hide yes)
@@
 			)
 		)
-		(property "Style" "indication"
+		(property "Style" "board"
 			(at 80.01 29.21 0)
 			(hide yes)
@@
 				)
 			)
-		)
-		(pin "1"
 		)
 		(pin "2"
@@
 			)
 		)
-		(property "Interlocking" "Gilroy Caltrain"
-			(at 80.01 129.54 0)
-			(show_name yes)
-			(do_not_autoplace yes)
-			(effects
-				(font
-					(size 1.27 1.27)
-				)
-			)
-		)
-		(property "Machine" "SPCoast South"
-			(at 80.645 125.73 0)
-			(show_name no)
-			(do_not_autoplace yes)
-			(effects
-				(font
-					(size 1.905 1.905)
-				)
-			)
-		)
 		(property "Role" "COLUMN"
 			(at 80.645 122.555 0)
@@
 	)
 	(symbol
-		(lib_id "Railroad-Office:PanelLamp-YELLOW")
+		(lib_id "Railroad-Office:ModelLamp-YELLOW")
 		(at 130.81 26.67 0)
 		(unit 1)
@@
 			)
 		)
-		(property "Description" "One physical model board lamp. Value is a free descriptive label (e.g. OS, TRACK, MC) and is not used elsewhere. IndicationToken is a comma-separated list of indication names (track circuits such as 795T1,2NAA,799T1, or tokens such as MC1K) OR'd to drive this one lamp. All listed indications are still individually on the CodeLine wire"
+		(property "Description" "One physical model board lamp. Value is a free descriptive label (e.g. OS, TRACK ...) and is not used elsewhere. IndicationToken is a comma-separated list of indication names (tokens from the CodeLine) OR'd to drive this one lamp."
 			(at 130.81 34.29 0)
 			(hide yes)
@@
 			)
 		)
-		(property "Style" "indication"
+		(property "Style" "board"
 			(at 130.81 24.13 0)
 			(hide yes)
@@
 				)
 			)
-		)
-		(pin "1"
 		)
 		(pin "2"
@@
 	)
 	(symbol
-		(lib_id "Railroad-Office:PanelLamp-YELLOW")
+		(lib_id "Railroad-Office:ModelLamp-YELLOW")
 		(at 130.81 31.75 0)
 		(unit 1)
@@
 			)
 		)
-		(property "Description" "One physical model board lamp. Value is a free descriptive label (e.g. OS, TRACK, MC) and is not used elsewhere. IndicationToken is a comma-separated list of indication names (track circuits such as 795T1,2NAA,799T1, or tokens such as MC1K) OR'd to drive this one lamp. All listed indications are still individually on the CodeLine wire"
+		(property "Description" "One physical model board lamp. Value is a free descriptive label (e.g. OS, TRACK ...) and is not used elsewhere. IndicationToken is a comma-separated list of indication names (tokens from the CodeLine) OR'd to drive this one lamp."
 			(at 130.81 39.37 0)
 			(hide yes)
@@
 			)
 		)
-		(property "Style" "indication"
+		(property "Style" "board"
 			(at 130.81 29.21 0)
 			(hide yes)
@@
 				)
 			)
-		)
-		(pin "1"
 		)
 		(pin "2"
@@
 	)
 	(symbol
-		(lib_id "Railroad-Office:PanelLamp-YELLOW")
+		(lib_id "Railroad-Office:ModelLamp-YELLOW")
 		(at 130.81 36.83 0)
 		(unit 1)
@@
 			)
 		)
-		(property "Description" "One physical model board lamp. Value is a free descriptive label (e.g. OS, TRACK, MC) and is not used elsewhere. IndicationToken is a comma-separated list of indication names (track circuits such as 795T1,2NAA,799T1, or tokens such as MC1K) OR'd to drive this one lamp. All listed indications are still individually on the CodeLine wire"
+		(property "Description" "One physical model board lamp. Value is a free descriptive label (e.g. OS, TRACK ...) and is not used elsewhere. IndicationToken is a comma-separated list of indication names (tokens from the CodeLine) OR'd to drive this one lamp."
 			(at 130.81 44.45 0)
 			(hide yes)
@@
 			)
 		)
-		(property "Style" "indication"
+		(property "Style" "board"
 			(at 130.81 34.29 0)
 			(hide yes)
@@
 				)
 			)
-		)
-		(pin "1"
 		)
 		(pin "2"
@@
 	)
 	(symbol
-		(lib_id "Railroad-Office:PanelLamp-YELLOW")
+		(lib_id "Railroad-Office:PanelMCall-Lamp")
 		(at 80.01 104.14 0)
 		(unit 1)
@@
 			)
 		)
-		(property "Description" "One physical model board lamp. Value is a free descriptive label (e.g. OS, TRACK, MC) and is not used elsewhere. IndicationToken is a comma-separated list of indication names (track circuits such as 795T1,2NAA,799T1, or tokens such as MC1K) OR'd to drive this one lamp. All listed indications are still individually on the CodeLine wire"
+		(property "Description" "One physical Maintainer Call lamp.  IndicationToken is a comma-separated list of indication names (tokens such as MC1K)"
 			(at 80.01 111.76 0)
 			(hide yes)
@@
 			)
 		)
-		(property "Interlocking" "Gilroy Caltrain"
-			(at 130.81 129.54 0)
-			(show_name yes)
-			(do_not_autoplace yes)
-			(effects
-				(font
-					(size 1.27 1.27)
-				)
-			)
-		)
-		(property "Machine" "SPCoast South"
-			(at 131.445 125.73 0)
-			(show_name no)
-			(do_not_autoplace yes)
-			(effects
-				(font
-					(size 1.905 1.905)
-				)
-			)
-		)
 		(property "Role" "COLUMN"
 			(at 131.445 122.555 0)
@@
 	)
 	(symbol
-		(lib_id "Railroad-Office:PanelLamp-YELLOW")
+		(lib_id "Railroad-Office:ModelLamp-YELLOW")
 		(at 80.01 31.75 0)
 		(unit 1)
@@
 			)
 		)
-		(property "Description" "One physical model board lamp. Value is a free descriptive label (e.g. OS, TRACK, MC) and is not used elsewhere. IndicationToken is a comma-separated list of indication names (track circuits such as 795T1,2NAA,799T1, or tokens such as MC1K) OR'd to drive this one lamp. All listed indications are still individually on the CodeLine wire"
+		(property "Description" "One physical model board lamp. Value is a free descriptive label (e.g. OS, TRACK ...) and is not used elsewhere. IndicationToken is a comma-separated list of indication names (tokens from the CodeLine) OR'd to drive this one lamp."
 			(at 80.01 39.37 0)
 			(hide yes)
@@
 			)
 		)
-		(property "Style" "indication"
+		(property "Style" "board"
 			(at 80.01 29.21 0)
 			(hide yes)
@@
 			)
 		)
-		(pin "1"
-		)
 		(pin "2"

Commit message: refactor(kicad): Name on every device, office unit and encoding; Kind on the JMRI drivers; Driver-JMRI-Light
The owner's rulings of 2026-10-24 on the review of ADR 0008 rev 4: Name = ${Value}
is the identity key everywhere, devices included; the OfficeUnit's Columns is
derived and struck; a JMRI driver carries no address and is keyed by its object
class and the device it serves, the class carried by Kind (TURNOUT, SENSOR,
SIGNALMAST, LIGHT); Driver-JMRI-Light (ADR 0005 §8: ON, INTENSITY) for a lamp
JMRI drives, and the two Gilroy Interchange maintainer-call lamps MC1 and MC2
become Lights (they were Sensors, which JMRI only displays).

Script: SPCoast/edits/2026-10-24-names-kind-light.py. Libraries: Name on 36
symbols (OfficeUnit, 5 encodings, 12 PANEL, 18 DEVICE), Columns off OfficeUnit,
Kind on 5 JMRI drivers, Driver-JMRI-Light added (the Sensor's pin positions,
INTENSITY as pin 3 below, no-connect on the two placed instances). Sheets: 359
Name instance fields, 16 Kind, 2 lib_id swaps, caches refreshed (no pin moved on
a refreshed symbol).

Verified: gate --check production/SPCoast.net production/names-after.net PASS:
same parts, same connectivity, Name == Value on all 273 named instances (47
heads with Value "~" resolve to an empty Name), Columns dropped once, Kind on 16
drivers, 2 Sensor -> Light with pin 1 reading ON; ERC 0 before and after.
Subdivision lint_symbol_fields: 99 symbols, 0 errors (Kind now allowed on
IODRIVER). production/SPCoast.net is the new export (production/ is untracked).

Co-Authored-By: Claude Fable 5.1 <noreply@anthropic.com>
Parts:
- CDE4002, LMP4011, LMP4012, LMP4021, LMP4022, LMP4023, MCK4001, MCL4001, SWL4001, SWL4002: Name (none) -> ${Value}
Changed lines of the file:
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@@
+			)
+		)
+		(property "Name" "${Value}"
+			(at 80.01 26.67 0)
+			(hide yes)
+			(show_name no)
+			(do_not_autoplace no)
+			(effects
+				(font
+					(size 1.27 1.27)
+				)
 			)
 		)
@@
 			)
 		)
+		(property "Name" "${Value}"
+			(at 130.81 63.5 0)
+			(hide yes)
+			(show_name no)
+			(do_not_autoplace no)
+			(effects
+				(font
+					(size 1.27 1.27)
+				)
+			)
+		)
 		(property "Appliance" "lever"
 			(at 131.445 76.2 0)
@@
 			)
 		)
+		(property "Name" "${Value}"
+			(at 80.01 63.5 0)
+			(hide yes)
+			(show_name no)
+			(do_not_autoplace no)
+			(effects
+				(font
+					(size 1.27 1.27)
+				)
+			)
+		)
 		(property "Appliance" "lever"
 			(at 80.645 76.2 0)
@@
 			)
 		)
+		(property "Name" "${Value}"
+			(at 130.81 97.79 0)
+			(hide yes)
+			(show_name no)
+			(do_not_autoplace no)
+			(effects
+				(font
+					(size 1.27 1.27)
+				)
+			)
+		)
 		(property "Appliance" "lever"
 			(at 130.81 90.17 0)
@@
 			)
 		)
+		(property "Name" "${Value}"
+			(at 130.81 63.5 0)
+			(hide yes)
+			(show_name no)
+			(do_not_autoplace no)
+			(effects
+				(font
+					(size 1.27 1.27)
+				)
+			)
+		)
 		(property "Appliance" "lever"
 			(at 131.445 76.2 0)
@@
 			)
 		)
+		(property "Name" "${Value}"
+			(at 80.01 63.5 0)
+			(hide yes)
+			(show_name no)
+			(do_not_autoplace no)
+			(effects
+				(font
+					(size 1.27 1.27)
+				)
+			)
+		)
 		(property "Appliance" "lever"
 			(at 80.645 76.2 0)
@@
 			)
 		)
+		(property "Name" "${Value}"
+			(at 130.81 26.67 0)
+			(hide yes)
+			(show_name no)
+			(do_not_autoplace no)
+			(effects
+				(font
+					(size 1.27 1.27)
+				)
+			)
+		)
 		(property "Appliance" "lamp"
 			(at 130.81 24.13 0)
@@
 			)
 		)
+		(property "Name" "${Value}"
+			(at 80.01 48.26 0)
+			(hide yes)
+			(show_name no)
+			(do_not_autoplace no)
+			(effects
+				(font
+					(size 1.27 1.27)
+				)
+			)
+		)
 		(property "Appliance" "lever"
 			(at 86.36 44.45 0)
@@
 			)
 		)
+		(property "Name" "${Value}"
+			(at 130.81 31.75 0)
+			(hide yes)
+			(show_name no)
+			(do_not_autoplace no)
+			(effects
+				(font
+					(size 1.27 1.27)
+				)
+			)
+		)
 		(property "Appliance" "lamp"
 			(at 130.81 29.21 0)
@@
 			)
 		)
+		(property "Name" "${Value}"
+			(at 130.81 36.83 0)
+			(hide yes)
+			(show_name no)
+			(do_not_autoplace no)
+			(effects
+				(font
+					(size 1.27 1.27)
+				)
+			)
+		)
 		(property "Appliance" "lamp"
 			(at 130.81 34.29 0)
@@
 			)
 		)
+		(property "Name" "${Value}"
+			(at 80.01 104.14 0)
+			(hide yes)
+			(show_name no)
+			(do_not_autoplace no)
+			(effects
+				(font
+					(size 1.27 1.27)
+				)
+			)
+		)
 		(property "Appliance" "lamp"
 			(at 80.01 101.6 0)
@@
 			(hide yes)
 			(show_name no)
+			(do_not_autoplace no)
+			(effects
+				(font
+					(size 1.27 1.27)
+				)
+			)
+		)
+		(property "Name" "${Value}"
+			(at 80.01 31.75 0)
+			(hide yes)
+			(show_name no)

Commit message: feat(kicad): owner edit (2026-10-27): Gilroy Caltrain loses its maintainer call; Corporal gets lever 832
Gilroy Caltrain's field has no maintainer call, so the owner removed the MC1
lever and the MC lamp (MCK4001, IndicationToken MC1K) from its desk column. The
owner also added a signal lever for 832 to Corporal's desk (column 12), because
Corporal's field sends 832's indications and the desk had no lever for them.

Verified: a fresh kicad-cli export compiles with the reference derivation on
FieldUnit-Subdivision feat/derive with 0 errors, 0 warnings, 8 info and 16
missing. Corporal's controls include 832HS, 832NGS and 832SGS, and every
Corporal desk device is in its column. KiCad was closed (no lock files).

Co-Authored-By: Claude Opus 5.5 <noreply@anthropic.com>
Parts:
- removed MCK4001: MC, symbol Railroad-Office:PanelMCall-Lamp
- removed MCL4001: MC1, symbol Railroad-Office:PanelMCall
Connections:
- no-connect marks 16 -> 18

Commit message: feat(spcoast): every desk column names its CP Name
The owner's edit in KiCad: each PanelColumn carries a CP Name. On an
AAR codeline it may name the interlocking (Christopher, Gilroy
Interchange); on the 506 it names the house.

Verified: a fresh kicad-cli netlist compiles with no column.cp_name
diagnostics; the three column.house errors (columns 3, 4, 9) are
resolved by the importer rule, not the drawing.

Co-Authored-By: Claude Opus 5.5 <noreply@anthropic.com>
Parts:
- COL4021, COL4022: CP Name (none) -> Gilroy Caltrain
Changed lines of the file:
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@@
 			)
 		)
-		(property "CP Name" ""
+		(property "CP Name" "Gilroy Caltrain"
 			(at 80.645 132.08 0)
 			(show_name yes)
@@
 			)
 		)
-		(property "CP Name" ""
+		(property "CP Name" "Gilroy Caltrain"
 			(at 131.445 132.08 0)
 			(show_name yes)

Commit message: feat(spcoast): per-pin token fields on the panels, lamp Indication expressions, maintainer calls named 1MC
Applies the symbol rulings of 2026-10-28 to every sheet: the lib_symbols
caches of the changed symbols are the library's copies (this also clears
the stale PanelMCall and MaintainerCall caches), and every placed
instance gets the new hidden Control.*/Indication.* fields, loses
PanelLock Invert, and PanelMCall's whole-symbol Control and Indication
(Pin.MCK binary). Model lamps' IndicationToken becomes Indication: each
comma-separated circuit gets its K, qualifiers kept, joined with " | "
(795T1,01T,799T1 -> 795T1K | 01TK | 799T1K).

Maintainer calls in Christopher (1, 2), Corporal, Luchessa and Sargent
follow Gilroy Interchange (5dad54f): Value MC<n> -> <n>, Name ${Value}MC,
and the separate PanelMCall-Lamp is replaced by unit 2 of the same
PanelMCall at the old lamp's position, so its MCK pin sits where the
LAMP pin was. The old lamps' Column pin touched PanelColumn pin 8
directly (no wire); that pin is now unconnected, as on Gilroy
Interchange. Gilroy Interchange's local MaintainerCall_1 cache and its
two trackplan calls lose Indication.

Verified: fresh netlist before/after: components 752 -> 747 (the five
lamps), nets 1028 -> 1028; each old LAMP-pin net now holds the lever's
unit-2 MCK pin (pin 3) on the same expander pin (B1, pin 9); the levers'
nets are renamed only (~{S} -> ~{MCS}, unit suffix A); no other net
changed. Every field difference is an intended one. ERC 18 -> 1
violations (lib_symbol_mismatch 17 -> 0; pre-existing Sargent AUX1
pin_not_connected remains).

Co-Authored-By: Claude Opus 5.5 <noreply@anthropic.com>
Parts:
- LMP4011: Indication (none) -> 773T1K | 775T1K; IndicationToken 773T1,775T1 -> (none)
- LMP4012: Indication (none) -> 1SATK; IndicationToken 1SAT -> (none)
- LMP4021: Indication (none) -> 01TK; IndicationToken 01T -> (none)
- LMP4022: Indication (none) -> 02TK; IndicationToken 02T -> (none)
- LMP4023: Indication (none) -> 03TK; IndicationToken 03T -> (none)
- SWL4001, SWL4002: Control.NWS (none) -> ${Value}NWS; Control.RWS (none) -> ${Value}RWS; Indication.NWK (none) -> ${Value}NWK; Indication.RWK (none) -> ${Value}RWK
Changed lines of the file:
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@@
 			)
 		)
-		(property "IndicationToken" "773T1,775T1"
+		(property "Indication" "773T1K | 775T1K"
 			(at 78.105 26.67 0)
 			(show_name no)
@@
 			)
 		)
+		(property "Control.NWS" "${Value}NWS"
+			(at 131.445 76.2 0)
+			(hide yes)
+			(show_name no)
+			(do_not_autoplace no)
+			(effects
+				(font
+					(size 1.27 1.27)
+				)
+			)
+		)
+		(property "Control.RWS" "${Value}RWS"
+			(at 131.445 76.2 0)
+			(hide yes)
+			(show_name no)
+			(do_not_autoplace no)
+			(effects
+				(font
+					(size 1.27 1.27)
+				)
+			)
+		)
+		(property "Indication.NWK" "${Value}NWK"
+			(at 131.445 76.2 0)
+			(hide yes)
+			(show_name no)
+			(do_not_autoplace no)
+			(effects
+				(font
+					(size 1.27 1.27)
+				)
+			)
+		)
+		(property "Indication.RWK" "${Value}RWK"
+			(at 131.445 76.2 0)
+			(hide yes)
+			(show_name no)
+			(do_not_autoplace no)
+			(effects
+				(font
+					(size 1.27 1.27)
+				)
+			)
+		)
 		(pin "1"
 		)
@@
 			)
 		)
+		(property "Control.NWS" "${Value}NWS"
+			(at 80.645 76.2 0)
+			(hide yes)
+			(show_name no)
+			(do_not_autoplace no)
+			(effects
+				(font
+					(size 1.27 1.27)
+				)
+			)
+		)
+		(property "Control.RWS" "${Value}RWS"
+			(at 80.645 76.2 0)
+			(hide yes)
+			(show_name no)
+			(do_not_autoplace no)
+			(effects
+				(font
+					(size 1.27 1.27)
+				)
+			)
+		)
+		(property "Indication.NWK" "${Value}NWK"
+			(at 80.645 76.2 0)
+			(hide yes)
+			(show_name no)
+			(do_not_autoplace no)
+			(effects
+				(font
+					(size 1.27 1.27)
+				)
+			)
+		)
+		(property "Indication.RWK" "${Value}RWK"
+			(at 80.645 76.2 0)
+			(hide yes)
+			(show_name no)
+			(do_not_autoplace no)
+			(effects
+				(font
+					(size 1.27 1.27)
+				)
+			)
+		)
 		(pin "4"
 		)
@@
 			)
 		)
+		(property "Control.CODE" ""
+			(at 130.81 90.17 0)
+			(hide yes)
+			(show_name no)
+			(do_not_autoplace no)
+			(effects
+				(font
+					(size 1.27 1.27)
+				)
+			)
+		)
 		(pin "1"
 		)
@@
 			)
 		)
+		(property "Control.NWS" "${Value}NWS"
+			(at 131.445 76.2 0)
+			(hide yes)
+			(show_name no)
+			(do_not_autoplace no)
+			(effects
+				(font
+					(size 1.27 1.27)
+				)
+			)
+		)
+		(property "Control.RWS" "${Value}RWS"
+			(at 131.445 76.2 0)
+			(hide yes)
+			(show_name no)
+			(do_not_autoplace no)
+			(effects
+				(font
+					(size 1.27 1.27)
+				)
+			)
+		)
+		(property "Indication.NWK" "${Value}NWK"
+			(at 131.445 76.2 0)
+			(hide yes)
+			(show_name no)
+			(do_not_autoplace no)
+			(effects
+				(font
+					(size 1.27 1.27)
+				)
+			)
+		)
+		(property "Indication.RWK" "${Value}RWK"
+			(at 131.445 76.2 0)
+			(hide yes)
+			(show_name no)
+			(do_not_autoplace no)
+			(effects
+				(font
+					(size 1.27 1.27)
+				)
+			)
+		)
 		(pin "4"
 		)
@@
 			)
 		)
+		(property "Control.NWS" "${Value}NWS"
+			(at 80.645 76.2 0)
+			(hide yes)
+			(show_name no)
+			(do_not_autoplace no)
+			(effects
+				(font
+					(size 1.27 1.27)
+				)
+			)
+		)
+		(property "Control.RWS" "${Value}RWS"
+			(at 80.645 76.2 0)
+			(hide yes)
+			(show_name no)
+			(do_not_autoplace no)
+			(effects
+				(font
+					(size 1.27 1.27)
+				)
+			)
+		)
+		(property "Indication.NWK" "${Value}NWK"
+			(at 80.645 76.2 0)
+			(hide yes)
+			(show_name no)
+			(do_not_autoplace no)
+			(effects
+				(font
+					(size 1.27 1.27)
+				)
+			)
+		)
+		(property "Indication.RWK" "${Value}RWK"
+			(at 80.645 76.2 0)
+			(hide yes)
+			(show_name no)
+			(do_not_autoplace no)
+			(effects
+				(font
+					(size 1.27 1.27)
+				)
+			)
+		)
 		(pin "1"
 		)
@@
 			)
 		)
-		(property "IndicationToken" "01T"
+		(property "Indication" "01TK"
 			(at 128.905 26.67 0)
 			(show_name no)
@@
 			)
 		)
-		(property "IndicationToken" "02T"
+		(property "Indication" "02TK"
 			(at 128.905 31.75 0)
 			(show_name no)
@@
 			)
 		)
-		(property "IndicationToken" "03T"
+		(property "Indication" "03TK"
 			(at 128.905 36.83 0)
 			(show_name no)
@@
 			)
 		)
-		(property "IndicationToken" "1SAT"
+		(property "Indication" "1SATK"
 			(at 78.105 31.75 0)
 			(show_name no)
