File: SPCoast/GilroyCalTrain.kicad_sch (KiCad schematic)
At the start: 94 parts, among them SW3771 771, SW3773 773, SW3775 775

Commit message: feat(kicad): explicit seams on every sheet: Codeline and Host wires, remote I/O attachments, CP Name
The Luchessa pattern (owner mockup 5288025) applied to the whole project by
SPCoast/edits/2026-10-21-explicit-seams.py, gated by its -gate.py.

Libraries
- Processor: pins Host (passive) and IO_Bus; Transport and Address fields dropped.
- Processor-Virtual (Role STRUCTURE, Kind PROCESSOR, Type VIRTUAL, Host pin, no bus),
  Remote-IO-CMRInet and Remote-IO-JMRI (Kind REMOTE_IO, Board, Address, Transport pin).
- Transports: attachment pin Encoding -> Transport; MQTT loses Station. Encodings lose
  Station and Address. FieldUnit and FieldUnit_Virtual removed. OfficeUnit's Host pin numbered.
- MAIN HOUSE: CP Name, the one key every join reads; Value is a display macro of it.

Sheets
- Every unit: Interlocking Codeline and Host as hierarchical pins; houses on the Codeline net.
  Luchessa rides Time Coded, every other unit MQTT (AAR Tokens). Luchessa and Sargent host
  themselves; Watsonville, Caltrain, Interchange, Corporal, Christopher run on SPCoastApp.
- Caltrain: the Processor placeholder is Remote-IO-CMRInet 'Caltrain' (cpNode, UA 30) on
  CMRInet. Interchange: Remote-IO-JMRI 'JMRI' on JMRI_MQTT. Their Codeline ports now go to
  MQTT, not to the I/O transports. Watsonville's placeholder removed.
- South-cTc: SPCoastApp is a Processor-Virtual hosting the two I/O transports and five units;
  ten sheet pins with labels and wires; JohnCTC loses the node fields.
- Luchessa: 17 appliances' CP 'CP X' -> 'X', matching the panel columns' CP Name.
- GilroyCalTrain-Panel: a stray, unconnected AAR Tokens instance (Station Luchessa) removed.

Verified: gate passed on production/explicit-seams-before.net vs -after.net: every unit's
Codeline and Host net is exactly as expected, remote I/O and desk bus nets as expected,
connectivity away from the seams unchanged, no field changed except where the ruling says,
parts removed Proc1-3/HOST1/Encoding1 and added RIO1/RIO2/Proc6/Proc7. ERC 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
Parts:
- removed Proc1: SPCoastApp, symbol Railroad-HardwareIO:Processor
- added RIO1: Caltrain, symbol Railroad-HardwareIO:Remote-IO-CMRInet
- HOUSE3001: value Gilroy Caltrain -> ${CP Name}; CP Name (none) -> Gilroy Caltrain
Connections:
- net Host: now reaches Plant3001.2 (Host)
- new net CMRInet: RIO1.1 (Transport)
Changed lines of the file:
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@@
 	(wire
 		(pts
-			(xy 87.63 21.59) (xy 87.63 26.67)
-		)
-		(stroke
-			(width 0)
-			(type default)
-		)
-	)
-	(wire
-		(pts
 			(xy 125.73 91.44) (xy 110.49 76.2)
 		)
@@
 		)
 	)
+	(hierarchical_label "CMRInet"
+		(shape bidirectional)
+		(at 87.63 21.59 0)
+		(effects
+			(font
+				(size 1.27 1.27)
+			)
+			(justify left)
+		)
+	)
+	(hierarchical_label "Host"
+		(shape bidirectional)
+		(at 87.63 26.67 0)
+		(effects
+			(font
+				(size 1.27 1.27)
+			)
+			(justify left)
+		)
+	)
 	(symbol
 		(lib_id "Railroad-Trackplan:Bumper")
@@
 			)
 		)
-		(property "Value" "Gilroy Caltrain"
+		(property "Value" "${CP Name}"
 			(at 69.85 40.005 0)
 			(show_name no)
@@
 			)
 		)
+		(property "CP Name" "Gilroy Caltrain"
+			(at 69.85 34.29 0)
+			(hide yes)
+			(show_name no)
+			(do_not_autoplace no)
+			(effects
+				(font
+					(size 1.27 1.27)
+				)
+			)
+		)
 		(pin "1"
 		)
@@
 	)
 	(symbol
-		(lib_id "Railroad-HardwareIO:Processor")
+		(lib_id "Railroad-HardwareIO:Remote-IO-CMRInet")
 		(at 74.93 16.51 0)
 		(unit 1)
@@
 		(in_pos_files yes)
 		(dnp no)
-		(property "Reference" "Proc1"
+		(property "Reference" "RIO1"
 			(at 60.706 10.668 0)
 			(hide yes)
@@
 			)
 		)
-		(property "Value" "SPCoastApp"
+		(property "Value" "Caltrain"
 			(at 67.691 16.51 0)
 			(show_name no)
-			(do_not_autoplace yes)
+			(do_not_autoplace no)
 			(effects
 				(font
@@
 			)
 		)
-		(property "Description" "A processor: declares the I2C bus and GPIO pins of the chips and drivers in its scope; with Transport and Address it is a node on that code line (ADR 0005)."
-			(at 76.2 20.32 0)
+		(property "Description" "Remote I/O over CMRInet: one node (Board, Address = UA) behind the transport's host; its CMRI drivers attach by sheet (ADR 0008)."
+			(at 74.93 16.51 0)
 			(hide yes)
 			(show_name no)
@@
 		)
 		(property "Role" "STRUCTURE"
-			(at 63.627 6.858 0)
+			(at 74.93 16.51 0)
 			(hide yes)
 			(show_name no)
@@
 			)
 		)
-		(property "Kind" "PROCESSOR"
-			(at 65.024 8.509 0)
+		(property "Kind" "REMOTE_IO"
+			(at 74.93 16.51 0)
 			(hide yes)
 			(show_name no)
@@
 			)
 		)
-		(property "Transport" "CMRInet"
+		(property "Address" "30"
 			(at 74.93 16.51 0)
 			(hide yes)
@@
 			)
 		)
-		(property "Address" "30"
+		(property "Transport" ""
 			(at 74.93 16.51 0)
 			(hide yes)
@@
 		(pin "1"
 		)
-		(pin "2"
-		)
 		(instances
 			(project "SPCoast"
 				(path "/528348b2-add8-5367-a5f7-439c76f0ca33/2ed995e3-3819-55cd-b8d9-5c2af048ccb4/61cd2495-14f3-42a6-a7c2-38f34b91ee1e"
-					(reference "Proc1")
+					(reference "RIO1")
 					(unit 1)
 				)
