File: SPCoast/GilroyCalTrain.kicad_sch (KiCad schematic)
At the start: 93 parts, among them SW3771 771, SW3773 773, SW3775 775

Commit message: refactor(kicad): head devices are DEVICE with Appliance head; the OfficeUnit's Role is OFFICE_UNIT; stale instance Roles follow the libraries
SPCoast/edits/2026-10-23-roles.py, ADR 0009 §3.10 as approved: CAST and MACHINE were implementation
words. The seven Device-Head-* symbols and their 57 placed instances carry Role DEVICE and Appliance head;
the OfficeUnit carries OFFICE_UNIT; the four transport instances still saying CODELINE_TRANSPORT say
TRANSPORT. Descriptions: Device-Switch loses "cast", the JMRI drivers say FieldUnit, the OfficeUnit says
what it is. Every cached definition that differed from its library copy refreshed.

Verified: netlist connectivity and parts identical; no field changed beyond Role, Appliance and
Description; no CAST, MACHINE or CODELINE_TRANSPORT remains on any instance; ERC 0.

Co-Authored-By: Claude Fable 5.1 <noreply@anthropic.com>
Parts:
- Cast10, Cast11, Cast12, Cast6, Cast7, Cast8, Cast9: Appliance (none) -> head; Role CAST -> DEVICE
Changed lines of the file:
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@@
 			)
 		)
-		(property "Role" "CAST"
+		(property "Role" "DEVICE"
 			(at 116.84 185.039 0)
 			(hide yes)
@@
 			)
 		)
+		(property "Appliance" "head"
+			(at 128.27 190.5 0)
+			(hide yes)
+			(show_name no)
+			(do_not_autoplace no)
+			(effects
+				(font
+					(size 1.27 1.27)
+				)
+			)
+		)
 		(property "Style" "CPL"
 			(at 116.84 184.277 0)
@@
 			)
 		)
-		(property "Role" "CAST"
+		(property "Role" "DEVICE"
 			(at 116.84 176.149 0)
 			(hide yes)
@@
 			)
 		)
+		(property "Appliance" "head"
+			(at 128.27 181.61 0)
+			(hide yes)
+			(show_name no)
+			(do_not_autoplace no)
+			(effects
+				(font
+					(size 1.27 1.27)
+				)
+			)
+		)
 		(property "Style" "CPL"
 			(at 116.84 175.387 0)
@@
 			)
 		)
-		(property "Role" "CAST"
+		(property "Role" "DEVICE"
 			(at 116.84 148.209 0)
 			(hide yes)
@@
 			)
 		)
+		(property "Appliance" "head"
+			(at 128.27 152.4 0)
+			(hide yes)
+			(show_name no)
+			(do_not_autoplace no)
+			(effects
+				(font
+					(size 1.27 1.27)
+				)
+			)
+		)
 		(property "Style" "CPL"
 			(at 116.84 147.447 0)
@@
 			)
 		)
-		(property "Role" "CAST"
+		(property "Role" "DEVICE"
 			(at 116.84 167.259 0)
 			(hide yes)
@@
 			)
 		)
+		(property "Appliance" "head"
+			(at 128.27 172.72 0)
+			(hide yes)
+			(show_name no)
+			(do_not_autoplace no)
+			(effects
+				(font
+					(size 1.27 1.27)
+				)
+			)
+		)
 		(property "Style" "CPL"
 			(at 116.84 166.497 0)
@@
 			)
 		)
-		(property "Role" "CAST"
+		(property "Role" "DEVICE"
 			(at 116.84 143.129 0)
 			(hide yes)
@@
 			)
 		)
+		(property "Appliance" "head"
+			(at 128.27 147.32 0)
+			(hide yes)
+			(show_name no)
+			(do_not_autoplace no)
+			(effects
+				(font
+					(size 1.27 1.27)
+				)
+			)
+		)
 		(property "Style" "CPL"
 			(at 116.84 142.367 0)
@@
 			)
 		)
-		(property "Role" "CAST"
+		(property "Role" "DEVICE"
 			(at 116.84 160.909 0)
 			(hide yes)
@@
 			)
 		)
+		(property "Appliance" "head"
+			(at 128.27 165.1 0)
+			(hide yes)
+			(show_name no)
+			(do_not_autoplace no)
+			(effects
+				(font
+					(size 1.27 1.27)
+				)
+			)
+		)
 		(property "Style" "CPL"
 			(at 116.84 160.147 0)
@@
 			)
 		)
-		(property "Role" "CAST"
+		(property "Role" "DEVICE"
 			(at 116.84 155.829 0)
 			(hide yes)
@@
 				)
 			)
+		)
+		(property "Appliance" "head"
+			(at 128.27 160.02 0)
+			(hide yes)
+			(show_name no)
+			(do_not_autoplace no)
+			(effects
+				(font
+					(size 1.27 1.27)
+				)
+			)

Commit message: refactor(kicad): Name on every device, office unit and encoding; Kind on the JMRI drivers; Driver-JMRI-Light
The owner's rulings of 2026-10-24 on the review of ADR 0008 rev 4: Name = ${Value}
is the identity key everywhere, devices included; the OfficeUnit's Columns is
derived and struck; a JMRI driver carries no address and is keyed by its object
class and the device it serves, the class carried by Kind (TURNOUT, SENSOR,
SIGNALMAST, LIGHT); Driver-JMRI-Light (ADR 0005 §8: ON, INTENSITY) for a lamp
JMRI drives, and the two Gilroy Interchange maintainer-call lamps MC1 and MC2
become Lights (they were Sensors, which JMRI only displays).

Script: SPCoast/edits/2026-10-24-names-kind-light.py. Libraries: Name on 36
symbols (OfficeUnit, 5 encodings, 12 PANEL, 18 DEVICE), Columns off OfficeUnit,
Kind on 5 JMRI drivers, Driver-JMRI-Light added (the Sensor's pin positions,
INTENSITY as pin 3 below, no-connect on the two placed instances). Sheets: 359
Name instance fields, 16 Kind, 2 lib_id swaps, caches refreshed (no pin moved on
a refreshed symbol).

Verified: gate --check production/SPCoast.net production/names-after.net PASS:
same parts, same connectivity, Name == Value on all 273 named instances (47
heads with Value "~" resolve to an empty Name), Columns dropped once, Kind on 16
drivers, 2 Sensor -> Light with pin 1 reading ON; ERC 0 before and after.
Subdivision lint_symbol_fields: 99 symbols, 0 errors (Kind now allowed on
IODRIVER). production/SPCoast.net is the new export (production/ is untracked).

Co-Authored-By: Claude Fable 5.1 <noreply@anthropic.com>
Parts:
- Cast10, Cast11, Cast12, Cast6, Cast7, Cast8, Cast9, DevMast3, DevMast4, DevMast5, DevMast6, DevMast7, DevSW1, DevSW3, DevSW4, DevTC4, DevTC5, DevTC6, DevTC7, DevTC8: Name (none) -> ${Value}

Commit message: refactor(kicad): Name = ${Value} on every Trackplan appliance, so no key is read from Value
The owner (2026-10-24), on review finding 4: no exception for appliance names
read from Value. Data model keys are functional descriptions of their content
and the symbol attribute names reflect that choice; Value is generic. Every
Railroad-Trackplan APPLIANCE symbol (switches, derails, masts, heads, track
circuits, maintainer calls, auxiliaries) gains Name = ${Value}: the appliance's
own name, a head's letter. The compiler reads Name, never Value.

Script: SPCoast/edits/2026-10-24-trackplan-names.py (library symbols, placed
instances, caches refreshed; no pin moved).

Verified: gate --check production/SPCoast.net production/trackplan-names-after.net
PASS: same parts, lib ids, Values and connectivity; the only field change is Name
added on every Trackplan appliance with Name == Value; ERC 0 before and after.
Subdivision lint_symbol_fields: 99 symbols, 0 errors. production/SPCoast.net is
the new export.

Co-Authored-By: Claude Fable 5.1 <noreply@anthropic.com>
Parts:
- H3001, H3002, H3003, H3004, H3005, H3006, H3007, S3001, S3002, S3003, S3004, S3005, SW3771, SW3773, SW3775, TC3001, TC3002, TC3003, TC3004, TC3005: Name (none) -> ${Value}
Changed lines of the file:
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@@
 			)
 		)
+		(property "Name" "${Value}"
+			(at 140.97 91.44 0)
+			(hide yes)
+			(show_name no)
+			(do_not_autoplace no)
+			(effects
+				(font
+					(size 1.27 1.27)
+				)
+			)
+		)
 		(property "IndicationCeiling" ""
 			(at 154.305 92.075 0)
@@
 			)
 		)
+		(property "Name" "${Value}"
+			(at 158.75 55.88 0)
+			(hide yes)
+			(show_name no)
+			(do_not_autoplace no)
+			(effects
+				(font
+					(size 1.27 1.27)
+				)
+			)
+		)
 		(property "Appliance" "mast"
 			(at 158.75 55.88 0)
@@
 			)
 		)
+		(property "Name" "${Value}"
+			(at 69.85 63.5 0)
+			(hide yes)
+			(show_name no)
+			(do_not_autoplace no)
+			(effects
+				(font
+					(size 1.27 1.27)
+				)
+			)
+		)
 		(property "Appliance" "mast"
 			(at 69.85 63.5 0)
@@
 			)
 		)
+		(property "Name" "${Value}"
+			(at 193.04 87.63 0)
+			(hide yes)
+			(show_name no)
+			(do_not_autoplace no)
+			(effects
+				(font
+					(size 1.27 1.27)
+				)
+			)
+		)
 		(property "Appliance" "head"
 			(at 193.04 87.63 0)
@@
 			)
 		)
+		(property "Name" "${Value}"
+			(at 73.66 63.5 0)
+			(hide yes)
+			(show_name no)
+			(do_not_autoplace no)
+			(effects
+				(font
+					(size 1.27 1.27)
+				)
+			)
+		)
 		(property "Appliance" "head"
 			(at 73.66 63.5 0)
@@
 			)
 		)
+		(property "Name" "${Value}"
+			(at 172.72 91.44 0)
+			(hide yes)
+			(show_name no)
+			(do_not_autoplace no)
+			(effects
+				(font
+					(size 1.27 1.27)
+				)
+			)
+		)
 		(property "IndicationCeiling" ""
 			(at 186.055 90.805 0)
@@
 			)
 		)
+		(property "Name" "${Value}"
+			(at 191.77 87.63 0)
+			(hide yes)
+			(show_name no)
+			(do_not_autoplace no)
+			(effects
+				(font
+					(size 1.27 1.27)
+				)
+			)
+		)
 		(property "Appliance" "mast"
 			(at 191.77 87.63 0)
@@
 			)
 		)
+		(property "Name" "${Value}"
+			(at 193.04 71.12 0)
+			(hide yes)
+			(show_name no)
+			(do_not_autoplace no)
+			(effects
+				(font
+					(size 1.27 1.27)
+				)
+			)
+		)
 		(property "Appliance" "head"
 			(at 193.04 71.12 0)
@@
 			)
 		)
+		(property "Name" "${Value}"
+			(at 191.77 104.14 0)
+			(hide yes)
+			(show_name no)
+			(do_not_autoplace no)
+			(effects
+				(font
+					(size 1.27 1.27)
+				)
+			)
+		)
 		(property "Appliance" "head"
 			(at 191.77 104.14 0)
@@
 			)
 		)
+		(property "Name" "${Value}"
+			(at 200.66 107.95 0)
+			(hide yes)
+			(show_name no)
+			(do_not_autoplace no)
+			(effects
+				(font
+					(size 1.27 1.27)
+				)
+			)
+		)
 		(property "Appliance" "track_circuit"
 			(at 200.66 107.95 0)
@@
 			)
 		)
+		(property "Name" "${Value}"
+			(at 154.94 55.88 0)
+			(hide yes)
+			(show_name no)
+			(do_not_autoplace no)
+			(effects
+				(font
+					(size 1.27 1.27)
+				)
+			)
+		)
 		(property "Appliance" "head"
 			(at 154.94 55.88 0)
@@
 			)
 		)
+		(property "Name" "${Value}"
+			(at 191.77 71.12 0)
+			(hide yes)
+			(show_name no)
+			(do_not_autoplace no)
+			(effects
+				(font
+					(size 1.27 1.27)
+				)
+			)
+		)
 		(property "Appliance" "mast"
 			(at 191.77 71.12 0)
@@
 			)
 		)
+		(property "Name" "${Value}"
+			(at 92.71 59.69 0)
+			(hide yes)
+			(show_name no)
+			(do_not_autoplace no)
+			(effects
+				(font
+					(size 1.27 1.27)
+				)
+			)
+		)
 		(property "IndicationCeiling" ""
 			(at 106.045 60.325 0)
@@
 			)
 		)
+		(property "Name" "${Value}"
+			(at 200.66 91.44 0)
+			(hide yes)
+			(show_name no)
+			(do_not_autoplace no)
+			(effects
+				(font
+					(size 1.27 1.27)
+				)
+			)
+		)
 		(property "Appliance" "track_circuit"
 			(at 200.66 91.44 0)
@@
 			)
 		)
+		(property "Name" "${Value}"
+			(at 200.66 59.69 0)
+			(hide yes)
+			(show_name no)
+			(do_not_autoplace no)
+			(effects
+				(font
+					(size 1.27 1.27)
+				)
+			)
+		)
 		(property "Appliance" "track_circuit"
 			(at 200.66 59.69 0)
@@
 			)
 		)
+		(property "Name" "${Value}"
+			(at 71.12 63.5 0)
+			(hide yes)
+			(show_name no)
+			(do_not_autoplace no)
+			(effects
+				(font
+					(size 1.27 1.27)
+				)
+			)
+		)
 		(property "Appliance" "head"
 			(at 71.12 63.5 0)
@@
 			)
 		)
+		(property "Name" "${Value}"
+			(at 58.42 59.69 0)
+			(hide yes)
+			(show_name no)
+			(do_not_autoplace no)
+			(effects
+				(font
+					(size 1.27 1.27)
+				)
+			)
+		)
 		(property "Appliance" "track_circuit"
 			(at 58.42 59.69 0)
@@
 			)
 		)
+		(property "Name" "${Value}"
+			(at 200.66 74.93 0)
+			(hide yes)
+			(show_name no)
+			(do_not_autoplace no)
+			(effects
+				(font
+					(size 1.27 1.27)
+				)
+			)
+		)
 		(property "Appliance" "track_circuit"
 			(at 200.66 74.93 0)
@@
 			)
 		)
+		(property "Name" "${Value}"
+			(at 190.5 104.14 0)
+			(hide yes)
+			(show_name no)
+			(do_not_autoplace no)
+			(effects
+				(font
+					(size 1.27 1.27)
+				)
+			)
+		)
 		(property "Appliance" "mast"
 			(at 190.5 104.14 0)
@@
 			(at 157.48 55.88 0)
 			(hide yes)
+			(show_name no)
+			(do_not_autoplace no)
+			(effects
+				(font
+					(size 1.27 1.27)
+				)
+			)
+		)
+		(property "Name" "${Value}"
+			(at 157.48 55.88 0)
+			(hide yes)

Commit message: feat(kicad): owner edit (2026-10-25): Milepost carries Name = ${Value}; mileposts ground the region at Lick
The Milepost symbol gains Name = ${Value} like every other keyed symbol, so the
compiler reads no Value for it. The two Luchessa mileposts take the field, and
three new mileposts are placed: 55.3 (Lick) and 77.1 at Gilroy Caltrain, 77.0 at
Gilroy Interchange. Panels/ is left untracked.

Verified: lint_symbol_fields 100 symbols, 0 errors, 0 warnings; the diff is
additions only, no instance field reset; FieldUnit-Subdivision 201 tests against
a fresh export; compile_layout.py --geometry writes mileposts 55.3, 77.1, 77.0,
78.3, 79.3 with no geometry info.

Co-Authored-By: Claude Fable 5.1 <noreply@anthropic.com>
Parts:
- added MP7003: 55.3, symbol Railroad-Trackplan:Milepost
- added MP7004: 77.1, symbol Railroad-Trackplan:Milepost
Changed lines of the file:
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@@
 	)
 	(symbol
+		(lib_id "Railroad-Trackplan:Milepost")
+		(at 48.26 48.26 0)
+		(unit 1)
+		(body_style 1)
+		(exclude_from_sim no)
+		(in_bom yes)
+		(on_board yes)
+		(in_pos_files yes)
+		(dnp no)
+		(property "Reference" "MP7003"
+			(at 44.45 45.085 0)
+			(hide yes)
+			(show_name no)
+			(do_not_autoplace no)
+			(effects
+				(font
+					(size 1.27 1.27)
+				)
+				(justify left)
+			)
+		)
+		(property "Value" "55.3"
+			(at 48.26 41.275 0)
+			(show_name no)
+			(do_not_autoplace yes)
+			(effects
+				(font
+					(size 1.27 1.27)
+				)
+			)
+		)
+		(property "Footprint" ""
+			(at 48.26 48.26 0)
+			(hide yes)
+			(show_name no)
+			(do_not_autoplace no)
+			(effects
+				(font
+					(size 1.27 1.27)
+				)
+			)
+		)
+		(property "Datasheet" ""
+			(at 48.26 48.26 0)
+			(hide yes)
+			(show_name no)
+			(do_not_autoplace no)
+			(effects
+				(font
+					(size 1.27 1.27)
+				)
+			)
+		)
+		(property "Description" "Milepost: a track anchor carrying the milepost of the point it sits on."
+			(at 48.26 48.26 0)
+			(hide yes)
+			(show_name no)
+			(do_not_autoplace no)
+			(effects
+				(font
+					(size 1.27 1.27)
+				)
+			)
+		)
+		(property "Role" "TRACK"
+			(at 48.26 48.26 0)
+			(hide yes)
+			(show_name no)
+			(do_not_autoplace no)
+			(effects
+				(font
+					(size 1.27 1.27)
+				)
+			)
+		)
+		(property "Kind" "MILEPOST"
+			(at 48.26 48.26 0)
+			(hide yes)
+			(show_name no)
+			(do_not_autoplace no)
+			(effects
+				(font
+					(size 1.27 1.27)
+				)
+			)
+		)
+		(property "Name" "${Value}"
+			(at 48.26 48.26 0)
+			(hide yes)
+			(show_name no)
+			(do_not_autoplace no)
+			(effects
+				(font
+					(size 1.27 1.27)
+				)
+			)
+		)
+		(instances
+			(project "SPCoast"
+				(path "/528348b2-add8-5367-a5f7-439c76f0ca33/2ed995e3-3819-55cd-b8d9-5c2af048ccb4/61cd2495-14f3-42a6-a7c2-38f34b91ee1e"
+					(reference "MP7003")
+					(unit 1)
+				)
+			)
+		)
+	)
+	(symbol
 		(lib_id "Railroad-Field:Device-TrackCircuit-Optical")
 		(at 35.56 198.12 0)
@@
 					(unit 1)
 				)
+			)
+		)
+	)
+	(symbol
+		(lib_id "Railroad-Trackplan:Milepost")
+		(at 92.71 48.26 0)
+		(unit 1)
+		(body_style 1)
+		(exclude_from_sim no)
+		(in_bom yes)
+		(on_board yes)
+		(in_pos_files yes)
+		(dnp no)
+		(property "Reference" "MP7004"
+			(at 88.9 45.085 0)
+			(hide yes)
+			(show_name no)
+			(do_not_autoplace no)
+			(effects
+				(font
+					(size 1.27 1.27)
+				)
+				(justify left)
+			)
+		)
+		(property "Value" "77.1"
+			(at 92.71 41.275 0)
+			(show_name no)
+			(do_not_autoplace yes)
+			(effects
+				(font
+					(size 1.27 1.27)
+				)
+			)
+		)
+		(property "Footprint" ""
+			(at 92.71 48.26 0)
+			(hide yes)
+			(show_name no)
+			(do_not_autoplace no)
+			(effects
+				(font
+					(size 1.27 1.27)
+				)
+			)
+		)
+		(property "Datasheet" ""
+			(at 92.71 48.26 0)
+			(hide yes)
+			(show_name no)
+			(do_not_autoplace no)
+			(effects
+				(font
+					(size 1.27 1.27)
+				)
+			)
+		)
+		(property "Description" "Milepost: a track anchor carrying the milepost of the point it sits on."
+			(at 92.71 48.26 0)
+			(hide yes)
+			(show_name no)
+			(do_not_autoplace no)
+			(effects
+				(font
+					(size 1.27 1.27)
+				)
+			)
+		)
+		(property "Role" "TRACK"
+			(at 92.71 48.26 0)
+			(hide yes)
+			(show_name no)
+			(do_not_autoplace no)
+			(effects
+				(font
+					(size 1.27 1.27)
+				)
+			)
+		)
+		(property "Kind" "MILEPOST"
+			(at 92.71 48.26 0)
+			(hide yes)
+			(show_name no)
+			(do_not_autoplace no)
+			(effects
+				(font
+					(size 1.27 1.27)
+				)
+			)
+		)
+		(property "Name" "${Value}"
+			(at 92.71 48.26 0)
+			(hide yes)
+			(show_name no)
+			(do_not_autoplace no)
+			(effects
+				(font
+					(size 1.27 1.27)
+				)
+			)
+		)
+		(instances
+			(project "SPCoast"
+				(path "/528348b2-add8-5367-a5f7-439c76f0ca33/2ed995e3-3819-55cd-b8d9-5c2af048ccb4/61cd2495-14f3-42a6-a7c2-38f34b91ee1e"
+					(reference "MP7004")
+					(unit 1)
+				)

Commit message: feat(kicad): owner edit (2026-10-26): NextCP carries Interlocking; Industry carries Name; HBA leaves the track
The owner's edits after the trackplan review:
- NextCP gains Interlocking = ${Value}, a key the compiler reads for the destination; every instance takes it.
  Christopher's two NextCPs toward Corporal now say Corporal (both said Sargent).
- Industry gains Name = ${VALUE}. The five Industries are named: Gilroy Industry at Luchessa, Beet Loader 1
  and 2 at Corporal and at Sargent.
- Sargent's HBA (hot box alarm) is moved off 1SAT's net; its MC pin is unconnected and it carries Milepost 83.4.
- Watsonville: one Rule 93 (YARD) symbol is moved to the yard side of its joint.
Panels/ is left untracked.

Verified:
- Netlist exported by the owner 2026-10-26 12:37, newer than every sheet and the library.
- lint_symbol_fields: 100 symbols, 0 errors, 0 warnings.

Co-Authored-By: Claude Opus 5.5 <noreply@anthropic.com>
Parts:
- CP3001, CP3002: Interlocking (none) -> ${Value}
Changed lines of the file:
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@@
 		)
 		(property "Value" "Lick"
-			(at 46.355 59.69 0)
+			(at 50.8 68.58 0)
+			(hide yes)
 			(show_name no)
-			(do_not_autoplace no)
+			(do_not_autoplace yes)
 			(effects
 				(font
@@
 			)
 		)
+		(property "Interlocking" "${Value}"
+			(at 50.8 68.58 0)
+			(hide yes)
+			(show_name no)
+			(do_not_autoplace no)
+			(effects
+				(font
+					(size 1.27 1.27)
+				)
+			)
+		)
 		(pin "1"
 		)
@@
 	(symbol
 		(lib_id "Railroad-Trackplan:NextCP")
-		(at 212.09 59.69 180)
+		(at 212.09 59.69 0)
 		(unit 1)
 		(body_style 1)
@@
 		(fields_autoplaced yes)
 		(property "Reference" "CP3002"
-			(at 208.915 57.785 0)
+			(at 215.265 61.595 0)
 			(hide yes)
 			(show_name no)
@@
 		)
 		(property "Value" "Gilroy Interchange"
-			(at 214.63 59.6899 0)
+			(at 214.63 68.58 0)
+			(hide yes)
 			(show_name no)
-			(do_not_autoplace no)
+			(do_not_autoplace yes)
 			(effects
 				(font
@@
 		)
 		(property "Footprint" ""
-			(at 215.9 59.69 0)
+			(at 208.28 59.69 0)
 			(hide yes)
 			(show_name no)
@@
 		)
 		(property "Datasheet" ""
-			(at 215.9 59.69 0)
+			(at 208.28 59.69 0)
 			(hide yes)
 			(show_name no)
@@
 		)
 		(property "Description" "Identifies the next control point on this track"
-			(at 215.265 52.705 0)
+			(at 208.915 66.675 0)
 			(hide yes)
 			(show_name no)
@@
 			(hide yes)
 			(show_name no)
+			(do_not_autoplace no)
+			(effects
+				(font
+					(size 1.27 1.27)
+				)
+			)
+		)
+		(property "Interlocking" "${Value}"
+			(at 214.63 68.58 0)
+			(hide yes)
+			(show_name no)

Commit message: refactor(symbols): the CP field is CP Name on every trackplan symbol
One fact, which house an appliance or circuit stands in, had two field
names: CP Name on the House and PanelColumn, CP on 17 trackplan
symbols. Every CP is now CP Name, in the library and in each placed
symbol, by a text rename of the field name only (KiCad's update
symbols was not used; it resets per-instance fields).

Verified: fresh kicad-cli netlists before and after: 754 components on
both, 136 had CP, every field identical once CP is read as CP Name, no
CP left. lint_symbol_fields: 100 symbols, 0 errors, 0 warnings.

Co-Authored-By: Claude Opus 5.5 <noreply@anthropic.com>
Parts:
- B3001, B3002, B3003, B3004, B3008, SW3771, SW3773, SW3775, TC3001, TC3002, TC3003, TC3004, TC3005: CP Gilroy Caltrain -> (none); CP Name (none) -> Gilroy Caltrain
Changed lines of the file:
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@@
 			)
 		)
-		(property "CP" "Gilroy Caltrain"
+		(property "CP Name" "Gilroy Caltrain"
 			(at 69.85 57.15 0)
 			(show_name no)
@@
 			)
 		)
-		(property "CP" "Gilroy Caltrain"
+		(property "CP Name" "Gilroy Caltrain"
 			(at 140.97 86.995 0)
 			(show_name no)
@@
 			)
 		)
-		(property "CP" "Gilroy Caltrain"
+		(property "CP Name" "Gilroy Caltrain"
 			(at 190.5 110.49 0)
 			(show_name no)
@@
 			)
 		)
-		(property "CP" "Gilroy Caltrain"
+		(property "CP Name" "Gilroy Caltrain"
 			(at 191.77 93.98 0)
 			(show_name no)
@@
 			)
 		)
-		(property "CP" "Gilroy Caltrain"
+		(property "CP Name" "Gilroy Caltrain"
 			(at 172.72 95.885 0)
 			(show_name no)
@@
 			)
 		)
-		(property "CP" "Gilroy Caltrain"
+		(property "CP Name" "Gilroy Caltrain"
 			(at 191.77 77.47 0)
 			(show_name no)
@@
 			)
 		)
-		(property "CP" "Gilroy Caltrain"
+		(property "CP Name" "Gilroy Caltrain"
 			(at 200.66 109.855 0)
 			(show_name no)
@@
 			)
 		)
-		(property "CP" "Gilroy Caltrain"
+		(property "CP Name" "Gilroy Caltrain"
 			(at 92.71 55.245 0)
 			(show_name no)
@@
 			)
 		)
-		(property "CP" "Gilroy Caltrain"
+		(property "CP Name" "Gilroy Caltrain"
 			(at 200.66 93.345 0)
 			(show_name no)
@@
 			)
 		)
-		(property "CP" "Gilroy Caltrain"
+		(property "CP Name" "Gilroy Caltrain"
 			(at 200.66 61.595 0)
 			(show_name no)
@@
 			)
 		)
-		(property "CP" "Gilroy Caltrain"
+		(property "CP Name" "Gilroy Caltrain"
 			(at 58.42 61.595 0)
 			(show_name no)
@@
 			)
 		)
-		(property "CP" "Gilroy Caltrain"
+		(property "CP Name" "Gilroy Caltrain"
 			(at 158.75 62.23 0)
 			(show_name no)
@@
 			)
 		)
-		(property "CP" "Gilroy Caltrain"
+		(property "CP Name" "Gilroy Caltrain"
 			(at 200.66 76.835 0)
 			(show_name no)
