File: SPCoast/GilroyInterchange.kicad_sch (KiCad schematic)
At the start: 72 parts, among them SW5777 777, SW5781 781

Commit message: feat(kicad): explicit seams on every sheet: Codeline and Host wires, remote I/O attachments, CP Name
The Luchessa pattern (owner mockup 5288025) applied to the whole project by
SPCoast/edits/2026-10-21-explicit-seams.py, gated by its -gate.py.

Libraries
- Processor: pins Host (passive) and IO_Bus; Transport and Address fields dropped.
- Processor-Virtual (Role STRUCTURE, Kind PROCESSOR, Type VIRTUAL, Host pin, no bus),
  Remote-IO-CMRInet and Remote-IO-JMRI (Kind REMOTE_IO, Board, Address, Transport pin).
- Transports: attachment pin Encoding -> Transport; MQTT loses Station. Encodings lose
  Station and Address. FieldUnit and FieldUnit_Virtual removed. OfficeUnit's Host pin numbered.
- MAIN HOUSE: CP Name, the one key every join reads; Value is a display macro of it.

Sheets
- Every unit: Interlocking Codeline and Host as hierarchical pins; houses on the Codeline net.
  Luchessa rides Time Coded, every other unit MQTT (AAR Tokens). Luchessa and Sargent host
  themselves; Watsonville, Caltrain, Interchange, Corporal, Christopher run on SPCoastApp.
- Caltrain: the Processor placeholder is Remote-IO-CMRInet 'Caltrain' (cpNode, UA 30) on
  CMRInet. Interchange: Remote-IO-JMRI 'JMRI' on JMRI_MQTT. Their Codeline ports now go to
  MQTT, not to the I/O transports. Watsonville's placeholder removed.
- South-cTc: SPCoastApp is a Processor-Virtual hosting the two I/O transports and five units;
  ten sheet pins with labels and wires; JohnCTC loses the node fields.
- Luchessa: 17 appliances' CP 'CP X' -> 'X', matching the panel columns' CP Name.
- GilroyCalTrain-Panel: a stray, unconnected AAR Tokens instance (Station Luchessa) removed.

Verified: gate passed on production/explicit-seams-before.net vs -after.net: every unit's
Codeline and Host net is exactly as expected, remote I/O and desk bus nets as expected,
connectivity away from the seams unchanged, no field changed except where the ruling says,
parts removed Proc1-3/HOST1/Encoding1 and added RIO1/RIO2/Proc6/Proc7. ERC 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
Parts:
- removed Proc2: SPCoastApp, symbol Railroad-HardwareIO:Processor
- added RIO2: JMRI, symbol Railroad-HardwareIO:Remote-IO-JMRI
- HOUSE5001: value Gilroy North -> ${CP Name}; CP Name (none) -> Gilroy North
- HOUSE5002: value Gilroy South -> ${CP Name}; CP Name (none) -> Gilroy South
Connections:
- net Codeline: now also HOUSE5001.2 (Codeline), HOUSE5002.2 (Codeline), Plant5001.1 (Codeline)
- net Host: now reaches Plant5001.2 (Host)
- new net JMRI_MQTT: RIO2.1 (Transport)
Changed lines of the file:
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@@
 		)
 	)
+	(hierarchical_label "JMRI_MQTT"
+		(shape bidirectional)
+		(at 87.63 21.59 0)
+		(effects
+			(font
+				(size 1.27 1.27)
+			)
+			(justify left)
+		)
+	)
 	(hierarchical_label "Codeline"
 		(shape bidirectional)
-		(at 74.93 25.4 180)
+		(at 74.93 35.56 180)
 		(effects
 			(font
@@
 		)
 	)
+	(hierarchical_label "Host"
+		(shape bidirectional)
+		(at 92.71 33.02 0)
+		(effects
+			(font
+				(size 1.27 1.27)
+			)
+			(justify left)
+		)
+	)
+	(symbol
+		(lib_id "Railroad-HardwareIO:Remote-IO-JMRI")
+		(at 74.93 16.51 0)
+		(unit 1)
+		(body_style 1)
+		(exclude_from_sim no)
+		(in_bom yes)
+		(on_board yes)
+		(in_pos_files yes)
+		(dnp no)
+		(property "Reference" "RIO2"
+			(at 60.706 10.668 0)
+			(hide yes)
+			(show_name no)
+			(do_not_autoplace yes)
+			(effects
+				(font
+					(size 1.27 1.27)
+				)
+			)
+		)
+		(property "Value" "JMRI"
+			(at 67.691 16.51 0)
+			(show_name no)
+			(do_not_autoplace no)
+			(effects
+				(font
+					(size 1.27 1.27)
+				)
+				(justify left)
+			)
+		)
+		(property "Footprint" ""
+			(at 74.93 16.51 0)
+			(hide yes)
+			(show_name no)
+			(do_not_autoplace no)
+			(effects
+				(font
+					(size 1.27 1.27)
+				)
+			)
+		)
+		(property "Datasheet" ""
+			(at 74.93 16.51 0)
+			(hide yes)
+			(show_name no)
+			(do_not_autoplace no)
+			(effects
+				(font
+					(size 1.27 1.27)
+				)
+			)
+		)
+		(property "Description" "Remote I/O through JMRI over MQTT: the JMRI objects of this sheet behind the transport's host; its JMRI drivers attach by sheet (ADR 0008)."
+			(at 74.93 16.51 0)
+			(hide yes)
+			(show_name no)
+			(do_not_autoplace no)
+			(effects
+				(font
+					(size 1.27 1.27)
+				)
+			)
+		)
+		(property "Role" "STRUCTURE"
+			(at 74.93 16.51 0)
+			(hide yes)
+			(show_name no)
+			(do_not_autoplace no)
+			(effects
+				(font
+					(size 1.27 1.27)
+				)
+			)
+		)
+		(property "Kind" "REMOTE_IO"
+			(at 74.93 16.51 0)
+			(hide yes)
+			(show_name no)
+			(do_not_autoplace no)
+			(effects
+				(font
+					(size 1.27 1.27)
+				)
+			)
+		)
+		(property "Board" "JMRI"
+			(at 74.93 16.51 0)
+			(hide yes)
+			(show_name no)
+			(do_not_autoplace no)
+			(effects
+				(font
+					(size 1.27 1.27)
+				)
+			)
+		)
+		(property "Address" ""
+			(at 74.93 16.51 0)
+			(hide yes)
+			(show_name no)
+			(do_not_autoplace no)
+			(effects
+				(font
+					(size 1.27 1.27)
+				)
+			)
+		)
+		(property "Transport" ""
+			(at 74.93 16.51 0)
+			(hide yes)
+			(show_name no)
+			(do_not_autoplace no)
+			(effects
+				(font
+					(size 1.27 1.27)
+				)
+			)
+		)
+		(pin "1"
+		)
+		(instances
+			(project "SPCoast"
+				(path "/528348b2-add8-5367-a5f7-439c76f0ca33/2ed995e3-3819-55cd-b8d9-5c2af048ccb4/defc570c-1f61-4751-be37-2827b304f837"
+					(reference "RIO2")
+					(unit 1)
+				)
+			)
+		)
+	)
 	(symbol
 		(lib_id "Railroad-Trackplan:IRJ-Signal")
@@
 	)
 	(symbol
-		(lib_id "Railroad-HardwareIO:Processor")
-		(at 74.93 29.21 0)
-		(unit 1)
-		(body_style 1)
-		(exclude_from_sim no)
-		(in_bom yes)
-		(on_board yes)
-		(in_pos_files yes)
-		(dnp no)
-		(fields_autoplaced yes)
-		(property "Reference" "Proc2"
-			(at 60.706 23.368 0)
-			(hide yes)
-			(show_name no)
-			(do_not_autoplace yes)
-			(effects
-				(font
-					(size 1.27 1.27)
-				)
-			)
-		)
-		(property "Value" "SPCoastApp"
-			(at 67.691 29.21 0)
-			(show_name no)
-			(do_not_autoplace yes)
-			(effects
-				(font
-					(size 1.27 1.27)
-				)
-				(justify left)
-			)
-		)
-		(property "Footprint" ""
-			(at 74.93 29.21 0)
-			(hide yes)
-			(show_name no)
-			(do_not_autoplace no)
-			(effects
-				(font
-					(size 1.27 1.27)
-				)
-			)
-		)
-		(property "Datasheet" ""
-			(at 74.93 29.21 0)
-			(hide yes)
-			(show_name no)
-			(do_not_autoplace no)
-			(effects
-				(font
-					(size 1.27 1.27)
-				)
-			)
-		)
-		(property "Description" "A processor: declares the I2C bus and GPIO pins of the chips and drivers in its scope; with Transport and Address it is a node on that code line."
-			(at 76.2 33.02 0)
-			(hide yes)
-			(show_name no)
-			(do_not_autoplace no)
-			(effects
-				(font
-					(size 1.27 1.27)
-				)
-			)
-		)
-		(property "Role" "STRUCTURE"
-			(at 63.627 19.558 0)
-			(hide yes)
-			(show_name no)
-			(do_not_autoplace no)
-			(effects
-				(font
-					(size 1.27 1.27)
-				)
-			)
-		)
-		(property "Kind" "PROCESSOR"
-			(at 65.024 21.209 0)
-			(hide yes)
-			(show_name no)
-			(do_not_autoplace no)
-			(effects
-				(font
-					(size 1.27 1.27)
-				)
-			)
-		)
-		(property "Board" ""
-			(at 74.93 29.21 0)
-			(hide yes)
-			(show_name no)
-			(do_not_autoplace no)
-			(effects
-				(font
-					(size 1.27 1.27)
-				)
-			)
-		)
-		(property "Transport" ""
-			(at 74.93 29.21 0)
-			(hide yes)
-			(show_name no)
-			(do_not_autoplace no)
-			(effects
-				(font
-					(size 1.27 1.27)
-				)
-			)
-		)
-		(property "Address" "WhatGoesHere"
-			(at 74.93 29.21 0)
-			(hide yes)
-			(show_name no)
-			(do_not_autoplace no)
-			(effects
-				(font
-					(size 1.27 1.27)
-				)
-			)
-		)
-		(pin "1"
-		)
-		(pin "2"
-		)
-		(instances
-			(project "SPCoast"
-				(path "/528348b2-add8-5367-a5f7-439c76f0ca33/2ed995e3-3819-55cd-b8d9-5c2af048ccb4/defc570c-1f61-4751-be37-2827b304f837"
-					(reference "Proc2")
-					(unit 1)
-				)
-			)
-		)
-	)
-	(symbol
 		(lib_id "Railroad-HardwareIO:Driver-JMRI-Turnout")
 		(at 55.88 113.03 0)
@@
 			)
 		)
-		(property "Value" "Gilroy South"
+		(property "Value" "${CP Name}"
 			(at 168.91 46.355 0)
 			(show_name no)
@@
 			)
 		)
+		(property "CP Name" "Gilroy South"
+			(at 168.91 40.64 0)
+			(hide yes)
+			(show_name no)
+			(do_not_autoplace no)
+			(effects
+				(font
+					(size 1.27 1.27)
+				)
+			)
+		)
 		(pin "1"
 		)
@@
 			)
 		)
-		(property "Value" "Gilroy North"
+		(property "Value" "${CP Name}"
 			(at 74.93 46.355 0)
 			(show_name no)
@@
 			(hide yes)
 			(show_name no)
+			(do_not_autoplace no)
+			(effects
+				(font
+					(size 1.27 1.27)
+				)
+			)
+		)
+		(property "CP Name" "Gilroy North"
+			(at 74.93 40.64 0)
+			(hide yes)
+			(show_name no)
