File: SPCoast/South-cTc.kicad_sch (KiCad schematic)
At the start: 9 parts

Commit message: feat(kicad): explicit seams on every sheet: Codeline and Host wires, remote I/O attachments, CP Name
The Luchessa pattern (owner mockup 5288025) applied to the whole project by
SPCoast/edits/2026-10-21-explicit-seams.py, gated by its -gate.py.

Libraries
- Processor: pins Host (passive) and IO_Bus; Transport and Address fields dropped.
- Processor-Virtual (Role STRUCTURE, Kind PROCESSOR, Type VIRTUAL, Host pin, no bus),
  Remote-IO-CMRInet and Remote-IO-JMRI (Kind REMOTE_IO, Board, Address, Transport pin).
- Transports: attachment pin Encoding -> Transport; MQTT loses Station. Encodings lose
  Station and Address. FieldUnit and FieldUnit_Virtual removed. OfficeUnit's Host pin numbered.
- MAIN HOUSE: CP Name, the one key every join reads; Value is a display macro of it.

Sheets
- Every unit: Interlocking Codeline and Host as hierarchical pins; houses on the Codeline net.
  Luchessa rides Time Coded, every other unit MQTT (AAR Tokens). Luchessa and Sargent host
  themselves; Watsonville, Caltrain, Interchange, Corporal, Christopher run on SPCoastApp.
- Caltrain: the Processor placeholder is Remote-IO-CMRInet 'Caltrain' (cpNode, UA 30) on
  CMRInet. Interchange: Remote-IO-JMRI 'JMRI' on JMRI_MQTT. Their Codeline ports now go to
  MQTT, not to the I/O transports. Watsonville's placeholder removed.
- South-cTc: SPCoastApp is a Processor-Virtual hosting the two I/O transports and five units;
  ten sheet pins with labels and wires; JohnCTC loses the node fields.
- Luchessa: 17 appliances' CP 'CP X' -> 'X', matching the panel columns' CP Name.
- GilroyCalTrain-Panel: a stray, unconnected AAR Tokens instance (Station Luchessa) removed.

Verified: gate passed on production/explicit-seams-before.net vs -after.net: every unit's
Codeline and Host net is exactly as expected, remote I/O and desk bus nets as expected,
connectivity away from the seams unchanged, no field changed except where the ruling says,
parts removed Proc1-3/HOST1/Encoding1 and added RIO1/RIO2/Proc6/Proc7. ERC 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
Parts:
- removed HOST1: SPCoastApp, symbol Railroad-Office:FieldUnit_Virtual
- added Proc7: SPCoastApp, symbol Railroad-HardwareIO:Processor-Virtual
- Encoding2001: Station ${SHEETNAME} -> (none)
Connections:
- net at Proc4.1 (Host): now also MACHINE2002.2 (Host); no longer MACHINE2002. (Host)
- net SPCoastApp: now reaches Transport2007.1 (Host), Transport2009.1 (Host)
- net SPCoastApp: now also Proc7.1 (Host)
Other:
- sheet Christopher ports: added Codeline, Host; removed none
- sheet Corporal ports: added Codeline, Host; removed none
- sheet Gilroy Caltrain ports: added CMRInet, Host; removed none
- sheet Gilroy Interchange ports: added Host, JMRI_MQTT; removed none
- sheet Sargent ports: added Codeline; removed none
- sheet Watsonville ports: added Host; removed none
