File: SPCoast/South-cTc.kicad_sch (KiCad schematic)
At the start: 10 parts

Commit message: refactor(kicad): head devices are DEVICE with Appliance head; the OfficeUnit's Role is OFFICE_UNIT; stale instance Roles follow the libraries
SPCoast/edits/2026-10-23-roles.py, ADR 0009 §3.10 as approved: CAST and MACHINE were implementation
words. The seven Device-Head-* symbols and their 57 placed instances carry Role DEVICE and Appliance head;
the OfficeUnit carries OFFICE_UNIT; the four transport instances still saying CODELINE_TRANSPORT say
TRANSPORT. Descriptions: Device-Switch loses "cast", the JMRI drivers say FieldUnit, the OfficeUnit says
what it is. Every cached definition that differed from its library copy refreshed.

Verified: netlist connectivity and parts identical; no field changed beyond Role, Appliance and
Description; no CAST, MACHINE or CODELINE_TRANSPORT remains on any instance; ERC 0.

Co-Authored-By: Claude Fable 5.1 <noreply@anthropic.com>
Parts:
- MACHINE2002: Role MACHINE -> OFFICE_UNIT
- Transport2005, Transport2006, Transport2007: Role CODELINE_TRANSPORT -> TRANSPORT
Changed lines of the file:
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@@
 			)
 		)
-		(property "Role" "CODELINE_TRANSPORT"
+		(property "Role" "TRANSPORT"
 			(at 167.64 74.93 0)
 			(hide yes)
@@
 			)
 		)
-		(property "Description" "One physical dispatcher cTc machine (protocol/vocabulary)."
+		(property "Description" "The OfficeUnit: the dispatcher's office logic and its desk; one per CTC machine. Its columns are its interlockings (ADR 0009)."
 			(at 192.405 56.515 0)
 			(hide yes)
@@
 			)
 		)
-		(property "Role" "MACHINE"
+		(property "Role" "OFFICE_UNIT"
 			(at 168.91 39.497 0)
 			(hide yes)
@@
 			)
 		)
-		(property "Role" "CODELINE_TRANSPORT"
+		(property "Role" "TRANSPORT"
 			(at 182.88 53.34 0)
 			(hide yes)
@@
 			)
 		)
-		(property "Role" "CODELINE_TRANSPORT"
+		(property "Role" "TRANSPORT"
 			(at 62.23 41.91 0)
 			(hide yes)

Commit message: chore(kicad): owner edits (2026-10-23): Address off Processor, Interlocking and Machine off PanelColumn, Railroad off Encoding-AAR, Broker default cleared; Host and Address off four instances; Sargent Cast4 Style back to the library's CL
Baseline before the scripted removal of the same fields from the remaining placed instances.

Verified: production/fields-after.net against roles-after.net: connectivity identical (820 nets, 1850 nodes,
743 parts); field delta is exactly Cast4 Style UQ->CL, Proc2 Address, Transport2005 Host, Transport2009 Host.
lint_symbol_fields: 96 symbols, 0 errors. ERC: two new lib_symbol_mismatch warnings on Transport-MQTT, the
cached copy still carrying the Broker default; nothing else.

Co-Authored-By: Claude Fable 5.1 <noreply@anthropic.com>
Parts:
- Proc2: Address Virtual -> (none)
Changed lines of the file:
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@@
-			)
-		)
-		(property "Address" "Virtual"
-			(at 77.47 41.91 0)
-			(hide yes)
-			(show_name no)
-			(do_not_autoplace no)
-			(effects
-				(font
-					(size 1.27 1.27)
-				)
 			)
 		)
@@
 			)
 		)
-		(property "Host" ""
-			(at 182.88 55.88 0)
-			(hide yes)
-			(show_name no)
-			(do_not_autoplace no)
-			(effects
-				(font
-					(size 1.27 1.27)
-				)
-			)
-		)

Commit message: refactor(kicad): model board lamps leave the columns; stale instance fields follow the libraries; PanelLamp-* retired
The owner's ruling (2026-10-23): the PanelColumn is the logical column, tied to a control point; the panel
I/O hardware is not. Every PanelLamp was a model board lamp except the maintainer-call lamp on the column's
pin 8. 34 lamps are now ModelLamp-<color> (no Column pin, Style board); 8 MC lamps are PanelMCall-Lamp.
Wires untouched: ~{LAMP} keeps its pin and the Column wire of a model lamp ends on nothing. Instance fields
the libraries dropped in c1d446b are gone from the sheets: Address on 7 processors, Interlocking and Machine
on 14 columns, Host on 2 transports. Railroad stays on the AAR encoding because its Topic template reads
${Railroad}; where Railroad lives is pending. Cached definitions refreshed for Processor, PanelColumn,
Transport-MQTT and Encoding-AAR. Scripted: SPCoast/edits/2026-10-23-model-lamps.py (edit, --check, --retire).

Verified: the script's gate on production/fields-after.net vs model-lamps-after.net: same 743 parts, lib ids
change only on the 42 lamps to the expected targets, fields change only as listed (Style indication->board
x34, the 37 drops), connectivity after == before minus the model lamps' pin 1, ERC 0 violations (the two
lib_symbol_mismatch warnings gone). lint_symbol_fields: 97 symbols, 0 errors (PanelLamp-BLUE, -GREEN, -RED, -YELLOW retired; there was no AMBER). Subdivision tests: 157 OK.

Co-Authored-By: Claude Fable 5.1 <noreply@anthropic.com>
Changed lines of the file:
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@@
-			)
-		)
-		(property "Host" ""
-			(at 161.29 78.74 0)
-			(hide yes)
-			(show_name no)
-			(do_not_autoplace no)
-			(effects
-				(font
-					(size 1.27 1.27)
-				)
 			)
 		)
@@
 		(property "Board" "cpNode-Xiao"
 			(at 179.07 40.64 0)
-			(hide yes)
-			(show_name no)
-			(do_not_autoplace no)
-			(effects
-				(font
-					(size 1.27 1.27)
-				)
-			)
-		)
-		(property "Address" ""
-			(at 177.8 44.45 0)
 			(hide yes)
 			(show_name no)
@@
 			(hide yes)
 			(show_name no)
-			(do_not_autoplace no)
-			(effects
-				(font
-					(size 1.27 1.27)
-				)
-			)
-		)
-		(property "Host" ""
-			(at 60.96 44.45 0)
-			(hide yes)
-			(show_name no)

Commit message: refactor(kicad): layout-wide facts on the Railroad symbol; the AAR Topic is the macro ctc/<STRUCTURE:RAILROAD:Name>/codeline/; Name on processors and transports
The owner's rulings (2026-10-23): a Railroad symbol on the root sheet (STRUCTURE/RAILROAD; Name, Railroad, Region,
Era, Rulebook) carries the layout-wide facts; a field may reference another symbol's field with <ROLE:KIND:Field>,
keyed by the fields the libraries key symbols by, resolved to the one instance in scope and expanded by the
compiler, never by KiCad (KIND empty for a Role without one); Name is the identity key everywhere, Value is never
read. The placed AAR encoding loses its Railroad field and its Topic becomes the macro; the library default follows.
The OfficeUnit instance loses Railroad and Era (off the library already). Processor and the four Transport-* gain
Name = ${Value}, library and 12 placed instances. Cached Encoding-AAR, OfficeUnit, Railroad, processors and
transports refreshed; no pin moved. Scripted: SPCoast/edits/2026-10-23-railroad.py (edit, --check).

Verified: the script's gate on production/model-lamps-after.net vs railroad-after.net: connectivity identical;
parts identical but for RAILROAD1; fields change only Topic (the macro, expanded against the one STRUCTURE/RAILROAD
symbol, equals the before value ctc/SPCoast/codeline/), Railroad x2 and Era x1 dropped, Name added on 12
processors and transports with Name == Value; ERC 0 violations. lint_symbol_fields: 98 symbols, 0 errors.

Co-Authored-By: Claude Fable 5.1 <noreply@anthropic.com>
Parts:
- Encoding2001: Railroad SPCoast -> (none); Topic ctc/${Railroad}/codeline/ -> ctc/<STRUCTURE:RAILROAD:Name>/codeline/
- MACHINE2002: Railroad SPCoast -> (none)
- Proc2, Proc4, Transport2005, Transport2006, Transport2007: Name (none) -> ${Value}
Changed lines of the file:
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@@
+			)
+		)
+		(property "Name" "${Value}"
+			(at 161.29 78.74 0)
+			(hide yes)
+			(show_name no)
+			(do_not_autoplace no)
+			(effects
+				(font
+					(size 1.27 1.27)
+				)
 			)
 		)
@@
 			)
 		)
+		(property "Name" "${Value}"
+			(at 179.07 40.64 0)
+			(hide yes)
+			(show_name no)
+			(do_not_autoplace no)
+			(effects
+				(font
+					(size 1.27 1.27)
+				)
+			)
+		)
 		(property "Kind" "PROCESSOR"
 			(at 188.976 48.641 0)
@@
 			)
 		)
-		(property "Era" ""
-			(at 165.227 41.275 0)
-			(hide yes)
-			(show_name yes)
-			(do_not_autoplace yes)
-			(effects
-				(font
-					(size 1.016 1.016)
-				)
-			)
-		)
 		(property "Role" "OFFICE_UNIT"
 			(at 168.91 39.497 0)
@@
 					(size 0.762 0.762)
 				)
-			)
-		)
-		(property "Railroad" "SPCoast"
-			(at 192.532 53.721 0)
-			(show_name no)
-			(do_not_autoplace yes)
-			(effects
-				(font
-					(size 0.762 0.762)
-				)
-				(justify left)
 			)
 		)
@@
 		(property "Role" "STRUCTURE"
 			(at 90.043 47.752 0)
+			(hide yes)
+			(show_name no)
+			(do_not_autoplace no)
+			(effects
+				(font
+					(size 1.27 1.27)
+				)
+			)
+		)
+		(property "Name" "${Value}"
+			(at 78.74 38.1 0)
 			(hide yes)
 			(show_name no)
@@
 			)
 		)
+		(property "Name" "${Value}"
+			(at 182.88 55.88 0)
+			(hide yes)
+			(show_name no)
+			(do_not_autoplace no)
+			(effects
+				(font
+					(size 1.27 1.27)
+				)
+			)
+		)
 		(property "Kind" "TIMECODE"
 			(at 185.42 57.785 0)
@@
 			)
 		)
-		(property "Topic" "ctc/${Railroad}/codeline/"
+		(property "Topic" "ctc/<STRUCTURE:RAILROAD:Name>/codeline/"
 			(at 179.07 93.98 0)
 			(show_name no)
@@
 				(font
 					(size 0.762 0.762)
-				)
-			)
-		)
-		(property "Railroad" "SPCoast"
-			(at 165.1 92.71 0)
-			(hide yes)
-			(show_name no)
-			(do_not_autoplace no)
-			(effects
-				(font
-					(size 1.27 1.27)
 				)
 			)
@@
 			)
 		)
+		(property "Name" "${Value}"
+			(at 60.96 44.45 0)
+			(hide yes)
+			(show_name no)
+			(do_not_autoplace no)
+			(effects
+				(font
+					(size 1.27 1.27)
+				)
+			)
+		)

Commit message: refactor(kicad): Name on every device, office unit and encoding; Kind on the JMRI drivers; Driver-JMRI-Light
The owner's rulings of 2026-10-24 on the review of ADR 0008 rev 4: Name = ${Value}
is the identity key everywhere, devices included; the OfficeUnit's Columns is
derived and struck; a JMRI driver carries no address and is keyed by its object
class and the device it serves, the class carried by Kind (TURNOUT, SENSOR,
SIGNALMAST, LIGHT); Driver-JMRI-Light (ADR 0005 §8: ON, INTENSITY) for a lamp
JMRI drives, and the two Gilroy Interchange maintainer-call lamps MC1 and MC2
become Lights (they were Sensors, which JMRI only displays).

Script: SPCoast/edits/2026-10-24-names-kind-light.py. Libraries: Name on 36
symbols (OfficeUnit, 5 encodings, 12 PANEL, 18 DEVICE), Columns off OfficeUnit,
Kind on 5 JMRI drivers, Driver-JMRI-Light added (the Sensor's pin positions,
INTENSITY as pin 3 below, no-connect on the two placed instances). Sheets: 359
Name instance fields, 16 Kind, 2 lib_id swaps, caches refreshed (no pin moved on
a refreshed symbol).

Verified: gate --check production/SPCoast.net production/names-after.net PASS:
same parts, same connectivity, Name == Value on all 273 named instances (47
heads with Value "~" resolve to an empty Name), Columns dropped once, Kind on 16
drivers, 2 Sensor -> Light with pin 1 reading ON; ERC 0 before and after.
Subdivision lint_symbol_fields: 99 symbols, 0 errors (Kind now allowed on
IODRIVER). production/SPCoast.net is the new export (production/ is untracked).

Co-Authored-By: Claude Fable 5.1 <noreply@anthropic.com>
Parts:
- Encoding2, Encoding2001, Encoding4: Name (none) -> ${Value}
- MACHINE2002: Columns 14 -> (none); Name (none) -> ${Value}
Changed lines of the file:
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@@
 			)
 		)
-		(property "Columns" "14"
-			(at 176.911 53.594 0)
-			(show_name no)
-			(do_not_autoplace yes)
-			(effects
-				(font
-					(size 0.762 0.762)
+		(property "Name" "${Value}"
+			(at 182.88 49.53 0)
+			(hide yes)
+			(show_name no)
+			(do_not_autoplace no)
+			(effects
+				(font
+					(size 1.27 1.27)
 				)
 			)
@@
 			)
 		)
+		(property "Name" "${Value}"
+			(at 165.1 72.39 0)
+			(hide yes)
+			(show_name no)
+			(do_not_autoplace no)
+			(effects
+				(font
+					(size 1.27 1.27)
+				)
+			)
+		)
 		(property "Kind" "USS506"
 			(at 175.895 81.915 0)
@@
 			)
 		)
+		(property "Name" "${Value}"
+			(at 64.77 58.42 0)
+			(hide yes)
+			(show_name no)
+			(do_not_autoplace no)
+			(effects
+				(font
+					(size 1.27 1.27)
+				)
+			)
+		)
 		(property "Kind" "CMRI"
 			(at 80.645 62.23 0)
@@
 			(hide yes)
 			(show_name no)
+			(do_not_autoplace no)
+			(effects
+				(font
+					(size 1.27 1.27)
+				)
+			)
+		)
+		(property "Name" "${Value}"
+			(at 165.1 92.71 0)
+			(hide yes)
+			(show_name no)

Commit message: fix(kicad): owner edit (2026-10-25): the CMRInet Node RIO1 carries IC CMRI, as its library and its bits do
The owner's ruling on ADR 0009 rev 3 decision 1: the token for CMRInet in every Kind and IC is CMRI; prose
and symbol names say CMRInet. RIO1 on the South-cTc sheet was the one instance with IC CMRInet.

Verified:
- Netlist exported by the owner 2026-10-25 22:30, newer than every sheet and library; the diff is the one
  IC field.

Co-Authored-By: Claude Opus 5.5 <noreply@anthropic.com>
Parts:
- RIO1: IC CMRInet -> CMRI
Changed lines of the file:
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@@
 			)
 		)
-		(property "IC" "CMRInet"
+		(property "IC" "CMRI"
 			(at 70.485 60.96 0)
 			(hide yes)
