File: SPCoast/Corporal-Panel.kicad_sch (KiCad schematic)
At the start: 16 parts, among them U12031 0x2A, U12032 0x2B

Commit message: chore(kicad): owner edits: Remote-IO node fields (Kind CMRI / MQTT-JMRI, bytes, UA), Interlocking Name, IOBus pins on remote drivers, sheet cleanup
Owner's edits of 2026-10-22, committed as they stand before the read-back.
Connections:
- net I2C renamed IOBus
Changed lines of the file:
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@@
 		(at 138.43 77.47)
 	)
-	(hierarchical_label "I2C"
+	(hierarchical_label "IOBus"
 		(shape bidirectional)
-		(at 160.02 111.76 0)
+		(at 162.56 111.76 0)
 		(effects
 			(font
@@
 		)
 	)
-	(hierarchical_label "I2C"
+	(hierarchical_label "IOBus"
 		(shape bidirectional)
-		(at 109.22 111.76 0)
+		(at 111.76 111.76 0)
 		(effects
 			(font
@@
 	(symbol
 		(lib_id "Railroad-HardwareIO:Driver-I2C-MAX7313-SPCoastcTc")
-		(at 99.06 72.39 0)
+		(at 100.33 72.39 0)
 		(unit 1)
 		(body_style 1)
@@
 		(dnp no)
 		(property "Reference" "U12031"
-			(at 91.44 22.86 0)
+			(at 92.71 22.86 0)
 			(hide yes)
 			(show_name no)
@@
 		)
 		(property "Value" "0x2A"
-			(at 103.505 22.86 0)
+			(at 104.775 22.86 0)
 			(show_name no)
 			(do_not_autoplace yes)
@@
 		)
 		(property "Footprint" ""
-			(at 99.06 72.39 0)
+			(at 100.33 72.39 0)
 			(hide yes)
 			(show_name no)
@@
 		)
 		(property "Datasheet" ""
-			(at 99.06 72.39 0)
+			(at 100.33 72.39 0)
 			(hide yes)
 			(show_name no)
@@
 		)
 		(property "Description" "One physical IO expander instance bound to a PanelColumn. Address is 0x10 to 0x4F"
-			(at 112.395 17.78 0)
+			(at 113.665 17.78 0)
 			(hide yes)
 			(show_name no)
@@
 		)
 		(property "Role" "IODRIVER"
-			(at 97.79 107.315 0)
+			(at 99.06 107.315 0)
 			(hide yes)
 			(show_name no)
@@
 		)
 		(property "Address" "0x2A"
-			(at 100.6281 112.3109 0)
+			(at 101.8981 112.3109 0)
 			(show_name no)
 			(do_not_autoplace no)
@@
 		)
 		(property "IC" "MAX7313"
-			(at 97.79 107.315 0)
+			(at 99.06 107.315 0)
 			(hide yes)
 			(show_name no)
@@
 		)
 		(property "Pin.A1" "binary"
-			(at 97.79 107.315 0)
+			(at 99.06 107.315 0)
 			(hide yes)
 			(show_name no)
@@
 		)
 		(property "Pin.A2" "binary"
-			(at 97.79 107.315 0)
+			(at 99.06 107.315 0)
 			(hide yes)
 			(show_name no)
@@
 		)
 		(property "Pin.A3" "binary"
-			(at 97.79 107.315 0)
+			(at 99.06 107.315 0)
 			(hide yes)
 			(show_name no)
@@
 		)
 		(property "Pin.A4" "binary"
-			(at 97.79 107.315 0)
+			(at 99.06 107.315 0)
 			(hide yes)
 			(show_name no)
@@
 		)
 		(property "Pin.A5" "binary"
-			(at 97.79 107.315 0)
+			(at 99.06 107.315 0)
 			(hide yes)
 			(show_name no)
@@
 		)
 		(property "Pin.A6" "binary"
-			(at 97.79 107.315 0)
+			(at 99.06 107.315 0)
 			(hide yes)
 			(show_name no)
@@
 		)
 		(property "Pin.A7" "binary"
-			(at 97.79 107.315 0)
+			(at 99.06 107.315 0)
 			(hide yes)
 			(show_name no)
@@
 		)
 		(property "Pin.A8" "binary"
-			(at 97.79 107.315 0)
+			(at 99.06 107.315 0)
 			(hide yes)
 			(show_name no)
@@
 		)
 		(property "Pin.B1" "binary"
-			(at 97.79 107.315 0)
+			(at 99.06 107.315 0)
 			(hide yes)
 			(show_name no)
@@
 		)
 		(property "Pin.B2" "binary"
-			(at 97.79 107.315 0)
+			(at 99.06 107.315 0)
 			(hide yes)
 			(show_name no)
@@
 		)
 		(property "Pin.B3" "binary"
-			(at 97.79 107.315 0)
+			(at 99.06 107.315 0)
 			(hide yes)
 			(show_name no)
@@
 		)
 		(property "Pin.B4" "binary"
-			(at 97.79 107.315 0)
+			(at 99.06 107.315 0)
 			(hide yes)
 			(show_name no)
@@
 		)
 		(property "Pin.B5" "binary"
-			(at 97.79 107.315 0)
+			(at 99.06 107.315 0)
 			(hide yes)
 			(show_name no)
@@
 		)
 		(property "Pin.B6" "binary"
-			(at 97.79 107.315 0)
+			(at 99.06 107.315 0)
 			(hide yes)
 			(show_name no)
@@
 		)
 		(property "Pin.B7" "binary"
-			(at 97.79 107.315 0)
+			(at 99.06 107.315 0)
 			(hide yes)
 			(show_name no)
@@
 		)
 		(property "Pin.B8" "binary"
-			(at 97.79 107.315 0)
+			(at 99.06 107.315 0)
 			(hide yes)
 			(show_name no)
@@
 	(symbol
 		(lib_id "Railroad-HardwareIO:Driver-I2C-MAX7313-SPCoastcTc")
-		(at 149.86 72.39 0)
+		(at 151.13 72.39 0)
 		(unit 1)
 		(body_style 1)
@@
 		(dnp no)
 		(property "Reference" "U12032"
-			(at 142.24 22.86 0)
+			(at 143.51 22.86 0)
 			(hide yes)
 			(show_name no)
@@
 		)
 		(property "Value" "0x2B"
-			(at 154.305 22.86 0)
+			(at 155.575 22.86 0)
 			(show_name no)
 			(do_not_autoplace yes)
@@
 		)
 		(property "Footprint" ""
-			(at 149.86 72.39 0)
+			(at 151.13 72.39 0)
 			(hide yes)
 			(show_name no)
@@
 		)
 		(property "Datasheet" ""
-			(at 149.86 72.39 0)
+			(at 151.13 72.39 0)
 			(hide yes)
 			(show_name no)
@@
 		)
 		(property "Description" "One physical IO expander instance bound to a PanelColumn. Address is 0x10 to 0x4F"
-			(at 163.195 17.78 0)
+			(at 164.465 17.78 0)
 			(hide yes)
 			(show_name no)
@@
 		)
 		(property "Role" "IODRIVER"
-			(at 148.59 107.315 0)
+			(at 149.86 107.315 0)
 			(hide yes)
 			(show_name no)
@@
 		)
 		(property "Address" "0x2B"
-			(at 151.4281 112.3109 0)
+			(at 152.6981 112.3109 0)
 			(show_name no)
 			(do_not_autoplace no)
@@
 		)
 		(property "IC" "MAX7313"
-			(at 148.59 107.315 0)
+			(at 149.86 107.315 0)
 			(hide yes)
 			(show_name no)
@@
 		)
 		(property "Pin.A1" "binary"
-			(at 148.59 107.315 0)
+			(at 149.86 107.315 0)
 			(hide yes)
 			(show_name no)
@@
 		)
 		(property "Pin.A2" "binary"
-			(at 148.59 107.315 0)
+			(at 149.86 107.315 0)
 			(hide yes)
 			(show_name no)
@@
 		)
 		(property "Pin.A3" "binary"
-			(at 148.59 107.315 0)
+			(at 149.86 107.315 0)
 			(hide yes)
 			(show_name no)
@@
 		)
 		(property "Pin.A4" "binary"
-			(at 148.59 107.315 0)
+			(at 149.86 107.315 0)
 			(hide yes)
 			(show_name no)
@@
 		)
 		(property "Pin.A5" "binary"
-			(at 148.59 107.315 0)
+			(at 149.86 107.315 0)
 			(hide yes)
 			(show_name no)
@@
 		)
 		(property "Pin.A6" "binary"
-			(at 148.59 107.315 0)
+			(at 149.86 107.315 0)
 			(hide yes)
 			(show_name no)
@@
 		)
 		(property "Pin.A7" "binary"
-			(at 148.59 107.315 0)
+			(at 149.86 107.315 0)
 			(hide yes)
 			(show_name no)
@@
 		)
 		(property "Pin.A8" "binary"
-			(at 148.59 107.315 0)
+			(at 149.86 107.315 0)
 			(hide yes)
 			(show_name no)
@@
 		)
 		(property "Pin.B1" "binary"
-			(at 148.59 107.315 0)
+			(at 149.86 107.315 0)
 			(hide yes)
 			(show_name no)
@@
 		)
 		(property "Pin.B2" "binary"
-			(at 148.59 107.315 0)
+			(at 149.86 107.315 0)
 			(hide yes)
 			(show_name no)
@@
 		)
 		(property "Pin.B3" "binary"
-			(at 148.59 107.315 0)
+			(at 149.86 107.315 0)
 			(hide yes)
 			(show_name no)
@@
 		)
 		(property "Pin.B4" "binary"
-			(at 148.59 107.315 0)
+			(at 149.86 107.315 0)
 			(hide yes)
 			(show_name no)
@@
 		)
 		(property "Pin.B5" "binary"
-			(at 148.59 107.315 0)
+			(at 149.86 107.315 0)
 			(hide yes)
 			(show_name no)
@@
 		)
 		(property "Pin.B6" "binary"
-			(at 148.59 107.315 0)
+			(at 149.86 107.315 0)
 			(hide yes)
 			(show_name no)
@@
 		)
 		(property "Pin.B7" "binary"
-			(at 148.59 107.315 0)
+			(at 149.86 107.315 0)
 			(hide yes)
 			(show_name no)
@@
 		)
 		(property "Pin.B8" "binary"
-			(at 148.59 107.315 0)
+			(at 149.86 107.315 0)
 			(hide yes)
 			(show_name no)
@@
 		(dnp no)
 		(property "Reference" "COL12031"
-			(at 80.01 133.985 0)
+			(at 74.93 120.65 0)
 			(hide yes)
 			(show_name no)
@@
 		(dnp no)
 		(property "Reference" "COL12032"
-			(at 130.81 133.985 0)
+			(at 125.73 120.65 0)
 			(hide yes)
 			(show_name no)
@@
 		(dnp no)
 		(property "Reference" "LKL12011"
-			(at 80.01 71.12 0)
+			(at 80.01 65.405 0)
 			(hide yes)
 			(show_name no)
@@
 		(dnp no)
 		(property "Reference" "LKL12011"
-			(at 80.01 71.12 0)
+			(at 80.01 65.405 0)
 			(hide yes)
 			(show_name no)
@@
 		(dnp no)
 		(property "Reference" "CDE12012"
-			(at 132.08 92.075 0)
+			(at 130.81 92.075 0)
 			(hide yes)
 			(show_name no)
