File: SPCoast/Luchessa-Panel.kicad_sch (KiCad schematic)
At the start: 16 parts, among them SW8784 783, SW8796 795, SW8800 799, U8004 0x24, U8005 0x25, U8006 0x26

Commit message: refactor(kicad): seam vocabulary after the naming audit: Processor, IOBus, PanelIOBus, House, Style, TimeCode, LocoNet, NodeType, MQTT-JMRI
SPCoast/edits/2026-10-22-vocabulary.py, the owner's rulings on
FieldUnit-Subdivision docs/review/naming-audit-2026-10-22.md:
- Host stays only on the transport symbols; the Interlocking, OfficeUnit and Processor pins, the unit
  sheets' port and labels are Processor.
- IOBus on the Processor pin; the office side is PanelIOBus on the unit ports, the Panel boxes' pins,
  the panel labels and the root sheet pins.
- MAIN HOUSE is House; its H pin is MC and hidden, as asked.
- OfficeUnit Type -> Style = US&S; TimeCode and LocoNet spellings, the LocoNet transport's pin is
  Transport; the one input Codeline sheet pin is bidirectional.
- The CMRInet node's Board -> NodeType (body text follows); JMRI drivers' IC = MQTT-JMRI.

Verified: --check on production/vocab-before.net vs vocab-after.net: identical connectivity under the
pin map, same parts (MAIN HOUSE -> House), only the ruled fields changed; field-io --check passes;
ERC 0 violations.

Co-Authored-By: Claude Fable 5.1 <noreply@anthropic.com>
Connections:
- net IOBus renamed PanelIOBus
Changed lines of the file:
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@@
 		(at 190.5 102.87)
 	)
-	(hierarchical_label "IOBus"
+	(hierarchical_label "PanelIOBus"
 		(shape bidirectional)
 		(at 214.63 139.7 0)
@@
 		)
 	)
-	(hierarchical_label "IOBus"
+	(hierarchical_label "PanelIOBus"
 		(shape bidirectional)
 		(at 163.83 139.7 0)
@@
 		)
 	)
-	(hierarchical_label "IOBus"
+	(hierarchical_label "PanelIOBus"
 		(shape bidirectional)
 		(at 113.03 139.7 0)
