File: SPCoast/Corporal.kicad_sch (KiCad schematic)
At the start: 61 parts, among them SW11829 829, SW11831 831, SW11900 829D, SW11901 1, SW11902 829

Commit message: chore(kicad): owner edits: CMRInet node on the transport net, sheet tidying (2026-10-23)
Changed lines of the file:
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@@
 		)
 	)
-	(hierarchical_label "PanelIOBus"
-		(shape bidirectional)
-		(at 104.14 25.4 0)
+	(label "IOBus"
+		(at 100.33 135.89 0)
 		(effects
 			(font
@@
 		)
 	)
-	(label "IOBus"
-		(at 100.33 135.89 0)
+	(hierarchical_label "PanelIOBus"
+		(shape bidirectional)
+		(at 104.14 25.4 0)
 		(effects
 			(font
@@
 		)
 		(property "Value" "Corporal"
-			(at 80.01 30.48 0)
+			(at 78.74 32.766 0)
 			(show_name no)
 			(do_not_autoplace yes)
@@
 					(size 1.27 1.27)
 				)
-				(justify left)
 			)
 		)
@@
 			(hide yes)
 			(show_name no)
+			(do_not_autoplace no)
+			(effects
+				(font
+					(size 1.27 1.27)
+				)
+			)
+		)
+		(property "Address" ""
+			(at 80.01 27.94 0)
+			(hide yes)
+			(show_name no)
