File: SPCoast/Corporal.kicad_sch (KiCad schematic)
At the start: 61 parts, among them SW11829 829, SW11831 831, SW11900 829D, SW11901 1, SW11902 829

Commit message: refactor(kicad): head devices are DEVICE with Appliance head; the OfficeUnit's Role is OFFICE_UNIT; stale instance Roles follow the libraries
SPCoast/edits/2026-10-23-roles.py, ADR 0009 §3.10 as approved: CAST and MACHINE were implementation
words. The seven Device-Head-* symbols and their 57 placed instances carry Role DEVICE and Appliance head;
the OfficeUnit carries OFFICE_UNIT; the four transport instances still saying CODELINE_TRANSPORT say
TRANSPORT. Descriptions: Device-Switch loses "cast", the JMRI drivers say FieldUnit, the OfficeUnit says
what it is. Every cached definition that differed from its library copy refreshed.

Verified: netlist connectivity and parts identical; no field changed beyond Role, Appliance and
Description; no CAST, MACHINE or CODELINE_TRANSPORT remains on any instance; ERC 0.

Co-Authored-By: Claude Fable 5.1 <noreply@anthropic.com>
Parts:
- Cast11001, Cast11002, Cast11003, Cast11004, Cast11005, Cast11006: Appliance (none) -> head; Role CAST -> DEVICE
Changed lines of the file:
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@@
 			)
 		)
-		(property "Role" "CAST"
+		(property "Role" "DEVICE"
 			(at 66.04 145.669 0)
 			(hide yes)
@@
 			)
 		)
+		(property "Appliance" "head"
+			(at 77.47 149.86 0)
+			(hide yes)
+			(show_name no)
+			(do_not_autoplace no)
+			(effects
+				(font
+					(size 1.27 1.27)
+				)
+			)
+		)
 		(property "Style" "CPL"
 			(at 66.04 144.907 0)
@@
 			)
 		)
-		(property "Role" "CAST"
+		(property "Role" "DEVICE"
 			(at 66.04 150.749 0)
 			(hide yes)
@@
 			)
 		)
+		(property "Appliance" "head"
+			(at 77.47 154.94 0)
+			(hide yes)
+			(show_name no)
+			(do_not_autoplace no)
+			(effects
+				(font
+					(size 1.27 1.27)
+				)
+			)
+		)
 		(property "Style" "CPL"
 			(at 66.04 149.987 0)
@@
 			)
 		)
-		(property "Role" "CAST"
+		(property "Role" "DEVICE"
 			(at 66.04 125.349 0)
 			(hide yes)
@@
 			)
 		)
+		(property "Appliance" "head"
+			(at 77.47 129.54 0)
+			(hide yes)
+			(show_name no)
+			(do_not_autoplace no)
+			(effects
+				(font
+					(size 1.27 1.27)
+				)
+			)
+		)
 		(property "Style" "CPL"
 			(at 66.04 124.587 0)
@@
 			)
 		)
-		(property "Role" "CAST"
+		(property "Role" "DEVICE"
 			(at 66.04 130.429 0)
 			(hide yes)
@@
 			)
 		)
+		(property "Appliance" "head"
+			(at 77.47 134.62 0)
+			(hide yes)
+			(show_name no)
+			(do_not_autoplace no)
+			(effects
+				(font
+					(size 1.27 1.27)
+				)
+			)
+		)
 		(property "Style" "CPL"
 			(at 66.04 129.667 0)
@@
 			)
 		)
-		(property "Role" "CAST"
+		(property "Role" "DEVICE"
 			(at 66.04 140.589 0)
 			(hide yes)
@@
 			)
 		)
+		(property "Appliance" "head"
+			(at 77.47 144.78 0)
+			(hide yes)
+			(show_name no)
+			(do_not_autoplace no)
+			(effects
+				(font
+					(size 1.27 1.27)
+				)
+			)
+		)
 		(property "Style" "CPL"
 			(at 66.04 139.827 0)
@@
 			)
 		)
-		(property "Role" "CAST"
+		(property "Role" "DEVICE"
 			(at 66.04 135.509 0)
 			(hide yes)
@@
 				)
 			)
+		)
+		(property "Appliance" "head"
+			(at 77.47 139.7 0)
+			(hide yes)
+			(show_name no)
+			(do_not_autoplace no)
+			(effects
+				(font
+					(size 1.27 1.27)
+				)
+			)

Commit message: refactor(kicad): model board lamps leave the columns; stale instance fields follow the libraries; PanelLamp-* retired
The owner's ruling (2026-10-23): the PanelColumn is the logical column, tied to a control point; the panel
I/O hardware is not. Every PanelLamp was a model board lamp except the maintainer-call lamp on the column's
pin 8. 34 lamps are now ModelLamp-<color> (no Column pin, Style board); 8 MC lamps are PanelMCall-Lamp.
Wires untouched: ~{LAMP} keeps its pin and the Column wire of a model lamp ends on nothing. Instance fields
the libraries dropped in c1d446b are gone from the sheets: Address on 7 processors, Interlocking and Machine
on 14 columns, Host on 2 transports. Railroad stays on the AAR encoding because its Topic template reads
${Railroad}; where Railroad lives is pending. Cached definitions refreshed for Processor, PanelColumn,
Transport-MQTT and Encoding-AAR. Scripted: SPCoast/edits/2026-10-23-model-lamps.py (edit, --check, --retire).

Verified: the script's gate on production/fields-after.net vs model-lamps-after.net: same 743 parts, lib ids
change only on the 42 lamps to the expected targets, fields change only as listed (Style indication->board
x34, the 37 drops), connectivity after == before minus the model lamps' pin 1, ERC 0 violations (the two
lib_symbol_mismatch warnings gone). lint_symbol_fields: 97 symbols, 0 errors (PanelLamp-BLUE, -GREEN, -RED, -YELLOW retired; there was no AMBER). Subdivision tests: 157 OK.

Co-Authored-By: Claude Fable 5.1 <noreply@anthropic.com>
Changed lines of the file:
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@@
-			)
-		)
-		(property "Address" ""
-			(at 80.01 27.94 0)
-			(hide yes)
-			(show_name no)
-			(do_not_autoplace no)
-			(effects
-				(font
-					(size 1.27 1.27)
-				)
 			)
 		)

Commit message: refactor(kicad): layout-wide facts on the Railroad symbol; the AAR Topic is the macro ctc/<STRUCTURE:RAILROAD:Name>/codeline/; Name on processors and transports
The owner's rulings (2026-10-23): a Railroad symbol on the root sheet (STRUCTURE/RAILROAD; Name, Railroad, Region,
Era, Rulebook) carries the layout-wide facts; a field may reference another symbol's field with <ROLE:KIND:Field>,
keyed by the fields the libraries key symbols by, resolved to the one instance in scope and expanded by the
compiler, never by KiCad (KIND empty for a Role without one); Name is the identity key everywhere, Value is never
read. The placed AAR encoding loses its Railroad field and its Topic becomes the macro; the library default follows.
The OfficeUnit instance loses Railroad and Era (off the library already). Processor and the four Transport-* gain
Name = ${Value}, library and 12 placed instances. Cached Encoding-AAR, OfficeUnit, Railroad, processors and
transports refreshed; no pin moved. Scripted: SPCoast/edits/2026-10-23-railroad.py (edit, --check).

Verified: the script's gate on production/model-lamps-after.net vs railroad-after.net: connectivity identical;
parts identical but for RAILROAD1; fields change only Topic (the macro, expanded against the one STRUCTURE/RAILROAD
symbol, equals the before value ctc/SPCoast/codeline/), Railroad x2 and Era x1 dropped, Name added on 12
processors and transports with Name == Value; ERC 0 violations. lint_symbol_fields: 98 symbols, 0 errors.

Co-Authored-By: Claude Fable 5.1 <noreply@anthropic.com>
Parts:
- Proc9: Name (none) -> ${Value}
Changed lines of the file:
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@@
+			)
+		)
+		(property "Name" "${Value}"
+			(at 78.74 31.75 0)
+			(hide yes)
+			(show_name no)
+			(do_not_autoplace no)
+			(effects
+				(font
+					(size 1.27 1.27)
+				)
 			)
 		)

Commit message: refactor(kicad): Name on every device, office unit and encoding; Kind on the JMRI drivers; Driver-JMRI-Light
The owner's rulings of 2026-10-24 on the review of ADR 0008 rev 4: Name = ${Value}
is the identity key everywhere, devices included; the OfficeUnit's Columns is
derived and struck; a JMRI driver carries no address and is keyed by its object
class and the device it serves, the class carried by Kind (TURNOUT, SENSOR,
SIGNALMAST, LIGHT); Driver-JMRI-Light (ADR 0005 §8: ON, INTENSITY) for a lamp
JMRI drives, and the two Gilroy Interchange maintainer-call lamps MC1 and MC2
become Lights (they were Sensors, which JMRI only displays).

Script: SPCoast/edits/2026-10-24-names-kind-light.py. Libraries: Name on 36
symbols (OfficeUnit, 5 encodings, 12 PANEL, 18 DEVICE), Columns off OfficeUnit,
Kind on 5 JMRI drivers, Driver-JMRI-Light added (the Sensor's pin positions,
INTENSITY as pin 3 below, no-connect on the two placed instances). Sheets: 359
Name instance fields, 16 Kind, 2 lib_id swaps, caches refreshed (no pin moved on
a refreshed symbol).

Verified: gate --check production/SPCoast.net production/names-after.net PASS:
same parts, same connectivity, Name == Value on all 273 named instances (47
heads with Value "~" resolve to an empty Name), Columns dropped once, Kind on 16
drivers, 2 Sensor -> Light with pin 1 reading ON; ERC 0 before and after.
Subdivision lint_symbol_fields: 99 symbols, 0 errors (Kind now allowed on
IODRIVER). production/SPCoast.net is the new export (production/ is untracked).

Co-Authored-By: Claude Fable 5.1 <noreply@anthropic.com>
Parts:
- Cast11001, Cast11002, Cast11003, Cast11004, Cast11005, Cast11006, DevLamp11001, DevMast11001, DevMast11002, DevMast11003, DevMast11004, DevSW11001, DevSW11002, DevSW11003, DevTC11001, DevTC11002, DevTC11003, DevTC11004, DevTC11005, LK11001, SW11902: Name (none) -> ${Value}

Commit message: refactor(kicad): Name = ${Value} on every Trackplan appliance, so no key is read from Value
The owner (2026-10-24), on review finding 4: no exception for appliance names
read from Value. Data model keys are functional descriptions of their content
and the symbol attribute names reflect that choice; Value is generic. Every
Railroad-Trackplan APPLIANCE symbol (switches, derails, masts, heads, track
circuits, maintainer calls, auxiliaries) gains Name = ${Value}: the appliance's
own name, a head's letter. The compiler reads Name, never Value.

Script: SPCoast/edits/2026-10-24-trackplan-names.py (library symbols, placed
instances, caches refreshed; no pin moved).

Verified: gate --check production/SPCoast.net production/trackplan-names-after.net
PASS: same parts, lib ids, Values and connectivity; the only field change is Name
added on every Trackplan appliance with Name == Value; ERC 0 before and after.
Subdivision lint_symbol_fields: 99 symbols, 0 errors. production/SPCoast.net is
the new export.

Co-Authored-By: Claude Fable 5.1 <noreply@anthropic.com>
Parts:
- H11001, H11002, H11003, H11004, H11005, H11006, MC11001, S11001, S11002, S11003, S11004, SW11829, SW11831, SW11900, SW11901, TC11001, TC11002, TC11003, TC11004, TC11005: Name (none) -> ${Value}
Changed lines of the file:
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@@
 			)
 		)
+		(property "Name" "${Value}"
+			(at 139.7 64.77 0)
+			(hide yes)
+			(show_name no)
+			(do_not_autoplace no)
+			(effects
+				(font
+					(size 1.27 1.27)
+				)
+			)
+		)
 		(property "Appliance" "head"
 			(at 139.7 64.77 0)
@@
 			)
 		)
+		(property "Name" "${Value}"
+			(at 123.19 68.58 0)
+			(hide yes)
+			(show_name no)
+			(do_not_autoplace no)
+			(effects
+				(font
+					(size 1.27 1.27)
+				)
+			)
+		)
 		(property "IndicationCeiling" "STOP/RESTRICTING"
 			(at 121.92 67.945 0)
@@
 			)
 		)
+		(property "Name" "${Value}"
+			(at 154.94 81.28 0)
+			(hide yes)
+			(show_name no)
+			(do_not_autoplace no)
+			(effects
+				(font
+					(size 1.27 1.27)
+				)
+			)
+		)
 		(property "Appliance" "head"
 			(at 154.94 81.28 0)
@@
 			)
 		)
+		(property "Name" "${Value}"
+			(at 152.4 81.28 0)
+			(hide yes)
+			(show_name no)
+			(do_not_autoplace no)
+			(effects
+				(font
+					(size 1.27 1.27)
+				)
+			)
+		)
 		(property "Appliance" "head"
 			(at 152.4 81.28 0)
@@
 			)
 		)
+		(property "Name" "${Value}"
+			(at 99.06 85.09 0)
+			(hide yes)
+			(show_name no)
+			(do_not_autoplace no)
+			(effects
+				(font
+					(size 1.27 1.27)
+				)
+			)
+		)
 		(property "IndicationCeiling" ""
 			(at 112.395 84.455 0)
@@
 			)
 		)
+		(property "Name" "${Value}"
+			(at 156.21 81.28 0)
+			(hide yes)
+			(show_name no)
+			(do_not_autoplace no)
+			(effects
+				(font
+					(size 1.27 1.27)
+				)
+			)
+		)
 		(property "Appliance" "mast"
 			(at 156.21 81.28 0)
@@
 			)
 		)
+		(property "Name" "${Value}"
+			(at 82.55 105.41 0)
+			(hide yes)
+			(show_name no)
+			(do_not_autoplace no)
+			(effects
+				(font
+					(size 1.27 1.27)
+				)
+			)
+		)
 		(property "Appliance" "head"
 			(at 82.55 105.41 0)
@@
 			)
 		)
+		(property "Name" "${Value}"
+			(at 170.18 68.58 0)
+			(hide yes)
+			(show_name no)
+			(do_not_autoplace no)
+			(effects
+				(font
+					(size 1.27 1.27)
+				)
+			)
+		)
 		(property "IndicationCeiling" "RESTRICTING/RESTRICTING"
 			(at 181.61 67.945 0)
@@
 			)
 		)
+		(property "Name" "${Value}"
+			(at 194.31 85.09 0)
+			(hide yes)
+			(show_name no)
+			(do_not_autoplace no)
+			(effects
+				(font
+					(size 1.27 1.27)
+				)
+			)
+		)
 		(property "Appliance" "track_circuit"
 			(at 194.31 85.09 0)
@@
 			)
 		)
+		(property "Name" "${Value}"
+			(at 147.32 68.58 0)
+			(hide yes)
+			(show_name no)
+			(do_not_autoplace no)
+			(effects
+				(font
+					(size 1.27 1.27)
+				)
+			)
+		)
 		(property "Appliance" "track_circuit"
 			(at 147.32 68.58 0)
@@
 			)
 		)
+		(property "Name" "${Value}"
+			(at 85.09 88.9 0)
+			(hide yes)
+			(show_name no)
+			(do_not_autoplace no)
+			(effects
+				(font
+					(size 1.27 1.27)
+				)
+			)
+		)
 		(property "Appliance" "head"
 			(at 85.09 88.9 0)
@@
 			)
 		)
+		(property "Name" "${Value}"
+			(at 73.66 85.09 0)
+			(hide yes)
+			(show_name no)
+			(do_not_autoplace no)
+			(effects
+				(font
+					(size 1.27 1.27)
+				)
+			)
+		)
 		(property "Appliance" "track_circuit"
 			(at 73.66 85.09 0)
@@
 			)
 		)
+		(property "Name" "${Value}"
+			(at 85.09 105.41 0)
+			(hide yes)
+			(show_name no)
+			(do_not_autoplace no)
+			(effects
+				(font
+					(size 1.27 1.27)
+				)
+			)
+		)
 		(property "Appliance" "head"
 			(at 85.09 105.41 0)
@@
 			)
 		)
+		(property "Name" "${Value}"
+			(at 81.28 105.41 0)
+			(hide yes)
+			(show_name no)
+			(do_not_autoplace no)
+			(effects
+				(font
+					(size 1.27 1.27)
+				)
+			)
+		)
 		(property "Appliance" "mast"
 			(at 81.28 105.41 0)
@@
 			)
 		)
+		(property "Name" "${Value}"
+			(at 81.28 88.9 0)
+			(hide yes)
+			(show_name no)
+			(do_not_autoplace no)
+			(effects
+				(font
+					(size 1.27 1.27)
+				)
+			)
+		)
 		(property "Appliance" "mast"
 			(at 81.28 88.9 0)
@@
 			)
 		)
+		(property "Name" "${Value}"
+			(at 137.16 85.09 0)
+			(hide yes)
+			(show_name no)
+			(do_not_autoplace no)
+			(effects
+				(font
+					(size 1.27 1.27)
+				)
+			)
+		)
 		(property "IndicationCeiling" ""
 			(at 123.825 85.725 0)
@@
 			)
 		)
+		(property "Name" "${Value}"
+			(at 99.06 49.53 0)
+			(hide yes)
+			(show_name no)
+			(do_not_autoplace no)
+			(effects
+				(font
+					(size 1.27 1.27)
+				)
+			)
+		)
 		(property "Appliance" "lamp"
 			(at 95.25 44.45 0)
@@
 			)
 		)
+		(property "Name" "${Value}"
+			(at 138.43 64.77 0)
+			(hide yes)
+			(show_name no)
+			(do_not_autoplace no)
+			(effects
+				(font
+					(size 1.27 1.27)
+				)
+			)
+		)
 		(property "Appliance" "mast"
 			(at 138.43 64.77 0)
@@
 			)
 		)
+		(property "Name" "${Value}"
+			(at 170.18 85.09 0)
+			(hide yes)
+			(show_name no)
+			(do_not_autoplace no)
+			(effects
+				(font
+					(size 1.27 1.27)
+				)
+			)
+		)
 		(property "Appliance" "track_circuit"
 			(at 170.18 85.09 0)
@@
 			(at 73.66 101.6 0)
 			(hide yes)
+			(show_name no)
+			(do_not_autoplace no)
+			(effects
+				(font
+					(size 1.27 1.27)
+				)
+			)
+		)
+		(property "Name" "${Value}"
+			(at 73.66 101.6 0)
+			(hide yes)

Commit message: feat(kicad): owner edit (2026-10-24): Industry symbol (TRACK, Kind INDUSTRY) replaces the dark stubs at Sargent, Corporal and Luchessa
Railroad-Trackplan gains Industry: Role TRACK, Kind INDUSTRY, one pin EoT at
(1.27, 0), description "Track exists past this point, but is not drawn". It is
visually distinct from Bumper and carries its own Kind, so a reader can tell
"track ends" from "track continues, not drawn" (ADR 0009 §3.10 amended in
FieldUnit-Subdivision).

Sargent B8, B9 and Corporal B6, B7 sit directly on the N and R ports of the
hand-thrown switch beyond END CTC; the wires drawn into dark track are gone.
Luchessa's industry spur: the Bumper B7007 and the wire into dark track are
gone; B7010 becomes Industry, and a new IRJ-END_CTC B11008 stands beside it.

The other sheets change only in their embedded library cache. On
GilroyInterchange KiCad renamed the cached Driver-JMRI-Light's second Kind
property to Kind_1: the library itself still carries two Kind properties on
that symbol (LIGHT and SENSOR, from 6882aa6), to be fixed separately. No placed
symbol is affected.

Verified:
- kicad-cli ERC: 0 violations
- lint_symbol_fields.py: 100 symbols, 0 errors, 0 warnings
- component field diff, previous netlist vs fresh export: only the five added
  Industry symbols, the added END CTC, the removed Bumper and B7010's Kind
- compile_layout.py output unchanged except provenance
- no lock files; owner reports KiCad project closed and files saved

Co-Authored-By: Claude Fable 5.1 <noreply@anthropic.com>
Parts:
- added B6, B7: (no value), symbol Railroad-Trackplan:Industry
Connections:
- net at SW11901.2 (N): now also B7.2 (EoT)
- net at SW11901.3 (R): now also B6.2 (EoT)
- no-connect marks 16 -> 12
Changed lines of the file:
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@@
 	)
 	(no_connect
-		(at 207.01 68.58)
-	)
-	(no_connect
 		(at 209.55 148.59)
 	)
@@
 	)
 	(no_connect
-		(at 207.01 52.07)
-	)
-	(no_connect
 		(at 77.47 166.37)
 	)
@@
 	)
 	(no_connect
-		(at 187.96 52.07)
-	)
-	(no_connect
-		(at 187.96 68.58)
-	)
-	(no_connect
 		(at 209.55 166.37)
 	)
@@
 	(wire
 		(pts
-			(xy 187.96 68.58) (xy 207.01 68.58)
-		)
-		(stroke
-			(width 0.4064)
-			(type dash)
-			(color 72 72 72 1)
-		)
-	)
-	(wire
-		(pts
 			(xy 104.14 33.02) (xy 97.79 33.02)
 		)
@@
 	(wire
 		(pts
-			(xy 187.96 52.07) (xy 207.01 52.07)
-		)
-		(stroke
-			(width 0.4064)
-			(type dash)
-			(color 72 72 72 1)
-		)
-	)
-	(wire
-		(pts
 			(xy 104.14 38.1) (xy 99.06 38.1)
 		)
@@
 	)
 	(symbol
+		(lib_id "Railroad-Trackplan:Industry")
+		(at 189.23 52.07 180)
+		(unit 1)
+		(body_style 1)
+		(exclude_from_sim no)
+		(in_bom yes)
+		(on_board yes)
+		(in_pos_files yes)
+		(dnp no)
+		(fields_autoplaced yes)
+		(property "Reference" "B6"
+			(at 189.23 49.53 0)
+			(hide yes)
+			(show_name no)
+			(do_not_autoplace no)
+			(effects
+				(font
+					(size 1.27 1.27)
+				)
+			)
+		)
+		(property "Value" ""
+			(at 189.23 52.07 0)
+			(hide yes)
+			(show_name no)
+			(do_not_autoplace no)
+			(effects
+				(font
+					(size 1.27 1.27)
+				)
+			)
+		)
+		(property "Footprint" ""
+			(at 189.23 52.07 0)
+			(hide yes)
+			(show_name no)
+			(do_not_autoplace no)
+			(effects
+				(font
+					(size 1.27 1.27)
+				)
+			)
+		)
+		(property "Datasheet" ""
+			(at 189.23 52.07 0)
+			(hide yes)
+			(show_name no)
+			(do_not_autoplace no)
+			(effects
+				(font
+					(size 1.27 1.27)
+				)
+			)
+		)
+		(property "Description" "Track exists past this point, but is not drawn"
+			(at 189.23 46.99 0)
+			(hide yes)
+			(show_name no)
+			(do_not_autoplace no)
+			(effects
+				(font
+					(size 1.27 1.27)
+				)
+			)
+		)
+		(property "Role" "TRACK"
+			(at 189.23 46.99 0)
+			(hide yes)
+			(show_name no)
+			(do_not_autoplace no)
+			(effects
+				(font
+					(size 1.27 1.27)
+				)
+			)
+		)
+		(property "Kind" "INDUSTRY"
+			(at 189.23 46.99 0)
+			(hide yes)
+			(show_name no)
+			(do_not_autoplace no)
+			(effects
+				(font
+					(size 1.27 1.27)
+				)
+			)
+		)
+		(pin "2"
+		)
+		(instances
+			(project "SPCoast"
+				(path "/528348b2-add8-5367-a5f7-439c76f0ca33/2ed995e3-3819-55cd-b8d9-5c2af048ccb4/152658f8-a042-4e04-bedb-bf34ee4ce875"
+					(reference "B6")
+					(unit 1)
+				)
+			)
+		)
+	)
+	(symbol
 		(lib_id "Railroad-Field:Device-TrackCircuit-Optical")
 		(at 129.54 166.37 0)
@@
 					(unit 1)
 				)
+			)
+		)
+	)
+	(symbol
+		(lib_id "Railroad-Trackplan:Industry")
+		(at 189.23 68.58 180)
+		(unit 1)
+		(body_style 1)
+		(exclude_from_sim no)
+		(in_bom yes)
+		(on_board yes)
+		(in_pos_files yes)
+		(dnp no)
+		(fields_autoplaced yes)
+		(property "Reference" "B7"
+			(at 189.23 66.04 0)
+			(hide yes)
+			(show_name no)
+			(do_not_autoplace no)
+			(effects
+				(font
+					(size 1.27 1.27)
+				)
+			)
+		)
+		(property "Value" ""
+			(at 189.23 68.58 0)
+			(hide yes)
+			(show_name no)
+			(do_not_autoplace no)
+			(effects
+				(font
+					(size 1.27 1.27)
+				)
+			)
+		)
+		(property "Footprint" ""
+			(at 189.23 68.58 0)
+			(hide yes)
+			(show_name no)
+			(do_not_autoplace no)
+			(effects
+				(font
+					(size 1.27 1.27)
+				)
+			)
+		)
+		(property "Datasheet" ""
+			(at 189.23 68.58 0)
+			(hide yes)
+			(show_name no)
+			(do_not_autoplace no)
+			(effects
+				(font
+					(size 1.27 1.27)
+				)
+			)
+		)
+		(property "Description" "Track exists past this point, but is not drawn"
+			(at 189.23 63.5 0)
+			(hide yes)
+			(show_name no)
+			(do_not_autoplace no)
+			(effects
+				(font
+					(size 1.27 1.27)
+				)
+			)
+		)
+		(property "Role" "TRACK"
+			(at 189.23 63.5 0)
+			(hide yes)
+			(show_name no)
+			(do_not_autoplace no)
+			(effects
+				(font
+					(size 1.27 1.27)
+				)
+			)
+		)
+		(property "Kind" "INDUSTRY"
+			(at 189.23 63.5 0)
+			(hide yes)
+			(show_name no)
+			(do_not_autoplace no)
+			(effects
+				(font
+					(size 1.27 1.27)
+				)
+			)
+		)
+		(pin "2"
+		)
+		(instances
+			(project "SPCoast"
+				(path "/528348b2-add8-5367-a5f7-439c76f0ca33/2ed995e3-3819-55cd-b8d9-5c2af048ccb4/152658f8-a042-4e04-bedb-bf34ee4ce875"
+					(reference "B7")
+					(unit 1)
+				)
