File: SPCoast/Corporal.kicad_sch (KiCad schematic)
At the start: 63 parts, among them SW11829 829, SW11831 831, SW11900 829D, SW11901 1, SW11902 829

Commit message: feat(kicad): owner edit (2026-10-26): NextCP carries Interlocking; Industry carries Name; HBA leaves the track
The owner's edits after the trackplan review:
- NextCP gains Interlocking = ${Value}, a key the compiler reads for the destination; every instance takes it.
  Christopher's two NextCPs toward Corporal now say Corporal (both said Sargent).
- Industry gains Name = ${VALUE}. The five Industries are named: Gilroy Industry at Luchessa, Beet Loader 1
  and 2 at Corporal and at Sargent.
- Sargent's HBA (hot box alarm) is moved off 1SAT's net; its MC pin is unconnected and it carries Milepost 83.4.
- Watsonville: one Rule 93 (YARD) symbol is moved to the yard side of its joint.
Panels/ is left untracked.

Verified:
- Netlist exported by the owner 2026-10-26 12:37, newer than every sheet and the library.
- lint_symbol_fields: 100 symbols, 0 errors, 0 warnings.

Co-Authored-By: Claude Opus 5.5 <noreply@anthropic.com>
Parts:
- B6: value (none) -> Beet Loader 1; Name (none) -> ${VALUE}
- B7: value (none) -> Beet Loader 2; Name (none) -> ${VALUE}
- CP11001, CP11002, CP11003: Interlocking (none) -> ${Value}
Connections:
- net at SW11900.1 (C): now also B11004.1 (A), DOT11006.1 (To); no longer SW11829.3 (R)
- new net: SW11829.3 (R), SW11900.2 (R)
Changed lines of the file:
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@@
 		)
 		(property "Value" "Christopher"
-			(at 61.595 101.6 0)
+			(at 66.04 110.49 0)
+			(hide yes)
 			(show_name no)
-			(do_not_autoplace no)
+			(do_not_autoplace yes)
 			(effects
 				(font
@@
 			)
 		)
+		(property "Interlocking" "${Value}"
+			(at 66.04 110.49 0)
+			(hide yes)
+			(show_name no)
+			(do_not_autoplace no)
+			(effects
+				(font
+					(size 1.27 1.27)
+				)
+			)
+		)
 		(pin "1"
 		)
@@
 		(lib_id "Railroad-Trackplan:Derail")
 		(at 123.19 68.58 0)
+		(mirror y)
 		(unit 1)
 		(body_style 1)
@@
 		(dnp no)
 		(property "Reference" "SW11900"
-			(at 120.65 71.12 0)
+			(at 125.73 71.12 0)
 			(hide yes)
 			(show_name no)
@@
 		)
 		(property "TC" ""
-			(at 130.81 66.04 0)
+			(at 115.57 66.04 0)
 			(show_name no)
 			(do_not_autoplace no)
@@
 		)
 		(property "IndicationCeiling" "STOP/RESTRICTING"
-			(at 121.92 67.945 0)
+			(at 124.46 67.945 0)
 			(show_name no)
 			(do_not_autoplace yes)
@@
 			)
 		)
-		(property "Value" ""
+		(property "Value" "Beet Loader 1"
 			(at 189.23 52.07 0)
 			(hide yes)
@@
 			)
 		)
+		(property "Name" "${VALUE}"
+			(at 189.23 52.07 0)
+			(hide yes)
+			(show_name no)
+			(do_not_autoplace no)
+			(effects
+				(font
+					(size 1.27 1.27)
+				)
+			)
+		)
 		(pin "2"
 		)
@@
 			)
 		)
-		(property "Value" ""
+		(property "Value" "Beet Loader 2"
 			(at 189.23 68.58 0)
 			(hide yes)
@@
 			)
 		)
+		(property "Name" "${VALUE}"
+			(at 189.23 68.58 0)
+			(hide yes)
+			(show_name no)
+			(do_not_autoplace no)
+			(effects
+				(font
+					(size 1.27 1.27)
+				)
+			)
+		)
 		(pin "2"
 		)
@@
 		)
 		(property "Value" "Sargent"
-			(at 205.105 85.09 0)
+			(at 209.55 93.98 0)
+			(hide yes)
 			(show_name no)
-			(do_not_autoplace no)
+			(do_not_autoplace yes)
 			(effects
 				(font
@@
 			)
 		)
+		(property "Interlocking" "${Value}"
+			(at 209.55 93.98 0)
+			(hide yes)
+			(show_name no)
+			(do_not_autoplace no)
+			(effects
+				(font
+					(size 1.27 1.27)
+				)
+			)
+		)
 		(pin "1"
 		)
@@
 		)
 		(property "Value" "Christopher"
-			(at 61.595 85.09 0)
+			(at 66.04 93.98 0)
+			(hide yes)
 			(show_name no)
-			(do_not_autoplace no)
+			(do_not_autoplace yes)
 			(effects
 				(font
@@
 			(hide yes)
 			(show_name no)
+			(do_not_autoplace no)
+			(effects
+				(font
+					(size 1.27 1.27)
+				)
+			)
+		)
+		(property "Interlocking" "${Value}"
+			(at 66.04 93.98 0)
+			(hide yes)
+			(show_name no)
