File: SPCoast/Watsonville.kicad_sch (KiCad schematic)
At the start: 201 parts, among them SW15003 3, SW15005 5, SW15007 7, SW15009 9, SW15011 11, SW15013 13, SW15015 15, SW15017 17, SW15019 19, SW15021 21, SW15023 23, SW15025 25, SW15837 837

Commit message: chore(kicad): owner edits: CMRInet node on the transport net, sheet tidying (2026-10-23)
Changed lines of the file:
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@@
 		)
 	)
-	(hierarchical_label "Codeline"
-		(shape bidirectional)
-		(at 64.77 30.48 0)
+	(label "IOBus"
+		(at 81.28 114.3 0)
 		(effects
 			(font
@@
 	)
 	(label "IOBus"
-		(at 81.28 114.3 0)
+		(at 218.44 124.46 0)
 		(effects
 			(font
@@
 	)
 	(label "IOBus"
-		(at 218.44 124.46 0)
+		(at 64.77 25.4 0)
 		(effects
 			(font
@@
 	)
 	(label "IOBus"
-		(at 64.77 25.4 0)
+		(at 172.72 124.46 0)
 		(effects
 			(font
@@
 	)
 	(label "IOBus"
-		(at 172.72 124.46 0)
+		(at 265.43 124.46 180)
 		(effects
 			(font
 				(size 1.27 1.27)
 			)
-			(justify left)
+			(justify right)
 		)
 	)
-	(hierarchical_label "PanelIOBus"
+	(hierarchical_label "Codeline"
 		(shape bidirectional)
-		(at 64.77 17.78 0)
+		(at 64.77 30.48 0)
 		(effects
 			(font
@@
 		)
 	)
-	(label "IOBus"
-		(at 265.43 124.46 180)
+	(hierarchical_label "PanelIOBus"
+		(shape bidirectional)
+		(at 64.77 17.78 0)
 		(effects
 			(font
 				(size 1.27 1.27)
 			)
-			(justify right)
+			(justify left)
 		)
 	)
@@
 		)
 		(property "Value" "Watsonville"
-			(at 36.83 22.86 0)
+			(at 35.56 25.146 0)
 			(show_name no)
 			(do_not_autoplace yes)
@@
 					(size 1.27 1.27)
 				)
-				(justify left)
 			)
 		)
@@
 			(hide yes)
 			(show_name no)
+			(do_not_autoplace no)
+			(effects
+				(font
+					(size 1.27 1.27)
+				)
+			)
+		)
+		(property "Address" ""
+			(at 36.83 20.32 0)
+			(hide yes)
+			(show_name no)
