File: SPCoast/Watsonville.kicad_sch (KiCad schematic)
At the start: 201 parts, among them SW15003 3, SW15005 5, SW15007 7, SW15009 9, SW15011 11, SW15013 13, SW15015 15, SW15017 17, SW15019 19, SW15021 21, SW15023 23, SW15025 25, SW15837 837

Commit message: refactor(kicad): head devices are DEVICE with Appliance head; the OfficeUnit's Role is OFFICE_UNIT; stale instance Roles follow the libraries
SPCoast/edits/2026-10-23-roles.py, ADR 0009 §3.10 as approved: CAST and MACHINE were implementation
words. The seven Device-Head-* symbols and their 57 placed instances carry Role DEVICE and Appliance head;
the OfficeUnit carries OFFICE_UNIT; the four transport instances still saying CODELINE_TRANSPORT say
TRANSPORT. Descriptions: Device-Switch loses "cast", the JMRI drivers say FieldUnit, the OfficeUnit says
what it is. Every cached definition that differed from its library copy refreshed.

Verified: netlist connectivity and parts identical; no field changed beyond Role, Appliance and
Description; no CAST, MACHINE or CODELINE_TRANSPORT remains on any instance; ERC 0.

Co-Authored-By: Claude Fable 5.1 <noreply@anthropic.com>
Parts:
- Cast15001, Cast15002, Cast15003, Cast15004, Cast15005, Cast15006, Cast15007, Cast15008, Cast15009, Cast15010: Appliance (none) -> head; Role CAST -> DEVICE
Changed lines of the file:
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@@
 			)
 		)
-		(property "Role" "CAST"
+		(property "Role" "DEVICE"
 			(at 46.99 118.999 0)
 			(hide yes)
@@
 			)
 		)
+		(property "Appliance" "head"
+			(at 58.42 123.19 0)
+			(hide yes)
+			(show_name no)
+			(do_not_autoplace no)
+			(effects
+				(font
+					(size 1.27 1.27)
+				)
+			)
+		)
 		(property "Style" "CPL"
 			(at 46.99 118.237 0)
@@
 			)
 		)
-		(property "Role" "CAST"
+		(property "Role" "DEVICE"
 			(at 46.99 134.239 0)
 			(hide yes)
@@
 			)
 		)
+		(property "Appliance" "head"
+			(at 58.42 138.43 0)
+			(hide yes)
+			(show_name no)
+			(do_not_autoplace no)
+			(effects
+				(font
+					(size 1.27 1.27)
+				)
+			)
+		)
 		(property "Style" "CPL"
 			(at 46.99 133.477 0)
@@
 			)
 		)
-		(property "Role" "CAST"
+		(property "Role" "DEVICE"
 			(at 46.99 108.839 0)
 			(hide yes)
@@
 			)
 		)
+		(property "Appliance" "head"
+			(at 58.42 113.03 0)
+			(hide yes)
+			(show_name no)
+			(do_not_autoplace no)
+			(effects
+				(font
+					(size 1.27 1.27)
+				)
+			)
+		)
 		(property "Style" "CPL"
 			(at 46.99 108.077 0)
@@
 			)
 		)
-		(property "Role" "CAST"
+		(property "Role" "DEVICE"
 			(at 46.99 146.939 0)
 			(hide yes)
@@
 			)
 		)
+		(property "Appliance" "head"
+			(at 58.42 151.13 0)
+			(hide yes)
+			(show_name no)
+			(do_not_autoplace no)
+			(effects
+				(font
+					(size 1.27 1.27)
+				)
+			)
+		)
 		(property "Style" "CPL"
 			(at 46.99 146.177 0)
@@
 			)
 		)
-		(property "Role" "CAST"
+		(property "Role" "DEVICE"
 			(at 46.99 113.919 0)
 			(hide yes)
@@
 			)
 		)
+		(property "Appliance" "head"
+			(at 58.42 118.11 0)
+			(hide yes)
+			(show_name no)
+			(do_not_autoplace no)
+			(effects
+				(font
+					(size 1.27 1.27)
+				)
+			)
+		)
 		(property "Style" "CPL"
 			(at 46.99 113.157 0)
@@
 			)
 		)
-		(property "Role" "CAST"
+		(property "Role" "DEVICE"
 			(at 46.99 129.159 0)
 			(hide yes)
@@
 			)
 		)
+		(property "Appliance" "head"
+			(at 58.42 133.35 0)
+			(hide yes)
+			(show_name no)
+			(do_not_autoplace no)
+			(effects
+				(font
+					(size 1.27 1.27)
+				)
+			)
+		)
 		(property "Style" "CPL"
 			(at 46.99 128.397 0)
@@
 			)
 		)
-		(property "Role" "CAST"
+		(property "Role" "DEVICE"
 			(at 46.99 139.319 0)
 			(hide yes)
@@
 			)
 		)
+		(property "Appliance" "head"
+			(at 58.42 143.51 0)
+			(hide yes)
+			(show_name no)
+			(do_not_autoplace no)
+			(effects
+				(font
+					(size 1.27 1.27)
+				)
+			)
+		)
 		(property "Style" "CPL"
 			(at 46.99 138.557 0)
@@
 			)
 		)
-		(property "Role" "CAST"
+		(property "Role" "DEVICE"
 			(at 46.99 152.019 0)
 			(hide yes)
@@
 			)
 		)
+		(property "Appliance" "head"
+			(at 58.42 156.21 0)
+			(hide yes)
+			(show_name no)
+			(do_not_autoplace no)
+			(effects
+				(font
+					(size 1.27 1.27)
+				)
+			)
+		)
 		(property "Style" "CPL"
 			(at 46.99 151.257 0)
@@
 			)
 		)
-		(property "Role" "CAST"
+		(property "Role" "DEVICE"
 			(at 46.99 124.079 0)
 			(hide yes)
@@
 			)
 		)
+		(property "Appliance" "head"
+			(at 58.42 128.27 0)
+			(hide yes)
+			(show_name no)
+			(do_not_autoplace no)
+			(effects
+				(font
+					(size 1.27 1.27)
+				)
+			)
+		)
 		(property "Style" "CPL"
 			(at 46.99 123.317 0)
@@
 			)
 		)
-		(property "Role" "CAST"
+		(property "Role" "DEVICE"
 			(at 46.99 103.759 0)
 			(hide yes)
@@
 				)
 			)
+		)
+		(property "Appliance" "head"
+			(at 58.42 107.95 0)
+			(hide yes)
+			(show_name no)
+			(do_not_autoplace no)
+			(effects
+				(font
+					(size 1.27 1.27)
+				)
+			)

Commit message: refactor(kicad): model board lamps leave the columns; stale instance fields follow the libraries; PanelLamp-* retired
The owner's ruling (2026-10-23): the PanelColumn is the logical column, tied to a control point; the panel
I/O hardware is not. Every PanelLamp was a model board lamp except the maintainer-call lamp on the column's
pin 8. 34 lamps are now ModelLamp-<color> (no Column pin, Style board); 8 MC lamps are PanelMCall-Lamp.
Wires untouched: ~{LAMP} keeps its pin and the Column wire of a model lamp ends on nothing. Instance fields
the libraries dropped in c1d446b are gone from the sheets: Address on 7 processors, Interlocking and Machine
on 14 columns, Host on 2 transports. Railroad stays on the AAR encoding because its Topic template reads
${Railroad}; where Railroad lives is pending. Cached definitions refreshed for Processor, PanelColumn,
Transport-MQTT and Encoding-AAR. Scripted: SPCoast/edits/2026-10-23-model-lamps.py (edit, --check, --retire).

Verified: the script's gate on production/fields-after.net vs model-lamps-after.net: same 743 parts, lib ids
change only on the 42 lamps to the expected targets, fields change only as listed (Style indication->board
x34, the 37 drops), connectivity after == before minus the model lamps' pin 1, ERC 0 violations (the two
lib_symbol_mismatch warnings gone). lint_symbol_fields: 97 symbols, 0 errors (PanelLamp-BLUE, -GREEN, -RED, -YELLOW retired; there was no AMBER). Subdivision tests: 157 OK.

Co-Authored-By: Claude Fable 5.1 <noreply@anthropic.com>
Changed lines of the file:
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@@
-			)
-		)
-		(property "Address" ""
-			(at 36.83 20.32 0)
-			(hide yes)
-			(show_name no)
-			(do_not_autoplace no)
-			(effects
-				(font
-					(size 1.27 1.27)
-				)
 			)
 		)

Commit message: refactor(kicad): layout-wide facts on the Railroad symbol; the AAR Topic is the macro ctc/<STRUCTURE:RAILROAD:Name>/codeline/; Name on processors and transports
The owner's rulings (2026-10-23): a Railroad symbol on the root sheet (STRUCTURE/RAILROAD; Name, Railroad, Region,
Era, Rulebook) carries the layout-wide facts; a field may reference another symbol's field with <ROLE:KIND:Field>,
keyed by the fields the libraries key symbols by, resolved to the one instance in scope and expanded by the
compiler, never by KiCad (KIND empty for a Role without one); Name is the identity key everywhere, Value is never
read. The placed AAR encoding loses its Railroad field and its Topic becomes the macro; the library default follows.
The OfficeUnit instance loses Railroad and Era (off the library already). Processor and the four Transport-* gain
Name = ${Value}, library and 12 placed instances. Cached Encoding-AAR, OfficeUnit, Railroad, processors and
transports refreshed; no pin moved. Scripted: SPCoast/edits/2026-10-23-railroad.py (edit, --check).

Verified: the script's gate on production/model-lamps-after.net vs railroad-after.net: connectivity identical;
parts identical but for RAILROAD1; fields change only Topic (the macro, expanded against the one STRUCTURE/RAILROAD
symbol, equals the before value ctc/SPCoast/codeline/), Railroad x2 and Era x1 dropped, Name added on 12
processors and transports with Name == Value; ERC 0 violations. lint_symbol_fields: 98 symbols, 0 errors.

Co-Authored-By: Claude Fable 5.1 <noreply@anthropic.com>
Parts:
- Proc8: Name (none) -> ${Value}
Changed lines of the file:
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@@
+			)
+		)
+		(property "Name" "${Value}"
+			(at 35.56 24.13 0)
+			(hide yes)
+			(show_name no)
+			(do_not_autoplace no)
+			(effects
+				(font
+					(size 1.27 1.27)
+				)
 			)
 		)

Commit message: refactor(kicad): Name on every device, office unit and encoding; Kind on the JMRI drivers; Driver-JMRI-Light
The owner's rulings of 2026-10-24 on the review of ADR 0008 rev 4: Name = ${Value}
is the identity key everywhere, devices included; the OfficeUnit's Columns is
derived and struck; a JMRI driver carries no address and is keyed by its object
class and the device it serves, the class carried by Kind (TURNOUT, SENSOR,
SIGNALMAST, LIGHT); Driver-JMRI-Light (ADR 0005 §8: ON, INTENSITY) for a lamp
JMRI drives, and the two Gilroy Interchange maintainer-call lamps MC1 and MC2
become Lights (they were Sensors, which JMRI only displays).

Script: SPCoast/edits/2026-10-24-names-kind-light.py. Libraries: Name on 36
symbols (OfficeUnit, 5 encodings, 12 PANEL, 18 DEVICE), Columns off OfficeUnit,
Kind on 5 JMRI drivers, Driver-JMRI-Light added (the Sensor's pin positions,
INTENSITY as pin 3 below, no-connect on the two placed instances). Sheets: 359
Name instance fields, 16 Kind, 2 lib_id swaps, caches refreshed (no pin moved on
a refreshed symbol).

Verified: gate --check production/SPCoast.net production/names-after.net PASS:
same parts, same connectivity, Name == Value on all 273 named instances (47
heads with Value "~" resolve to an empty Name), Columns dropped once, Kind on 16
drivers, 2 Sensor -> Light with pin 1 reading ON; ERC 0 before and after.
Subdivision lint_symbol_fields: 99 symbols, 0 errors (Kind now allowed on
IODRIVER). production/SPCoast.net is the new export (production/ is untracked).

Co-Authored-By: Claude Fable 5.1 <noreply@anthropic.com>
Parts:
- Cast15001, Cast15002, Cast15003, Cast15004, Cast15005, Cast15006, Cast15007, Cast15008, Cast15009, Cast15010, DevMast15001, DevMast15002, DevMast15003, DevMast15004, DevMast15005, DevMast15006, DevMast15007, DevMast15008, DevMast15009, DevSW15001, DevSW15002, DevSW15003, DevSW15004, DevSW15005, DevSW15006, DevSW15007, DevSW15008, DevSW15009, DevSW15010, DevSW15011, DevSW15012, DevSW15013, DevTC15001, DevTC15002, DevTC15003, DevTC15004, DevTC15005, DevTC15006, DevTC15007, DevTC15008, DevTC15009, DevTC15010, DevTC15011, DevTC15012, DevTC15013, DevTC15014, DevTC15015, DevTC15016, DevTC15017, DevTC15018, DevTC15019, DevTC15020, DevTC15021, DevTC15022, DevTC15023, DevTC15024, DevTC15025, DevTC15026, DevTC15027, DevTC15028, DevTC15029, DevTC15030, DevTC15031, DevTC15032: Name (none) -> ${Value}

Commit message: refactor(kicad): Name = ${Value} on every Trackplan appliance, so no key is read from Value
The owner (2026-10-24), on review finding 4: no exception for appliance names
read from Value. Data model keys are functional descriptions of their content
and the symbol attribute names reflect that choice; Value is generic. Every
Railroad-Trackplan APPLIANCE symbol (switches, derails, masts, heads, track
circuits, maintainer calls, auxiliaries) gains Name = ${Value}: the appliance's
own name, a head's letter. The compiler reads Name, never Value.

Script: SPCoast/edits/2026-10-24-trackplan-names.py (library symbols, placed
instances, caches refreshed; no pin moved).

Verified: gate --check production/SPCoast.net production/trackplan-names-after.net
PASS: same parts, lib ids, Values and connectivity; the only field change is Name
added on every Trackplan appliance with Name == Value; ERC 0 before and after.
Subdivision lint_symbol_fields: 99 symbols, 0 errors. production/SPCoast.net is
the new export.

Co-Authored-By: Claude Fable 5.1 <noreply@anthropic.com>
Parts:
- FLK15003, FLK15004, H15001, H15002, H15003, H15004, H15005, H15006, H15007, H15008, H15009, H15010, H15011, H15012, S15001, S15002, S15003, S15004, S15005, S15006, S15007, S15008, S15009, S15010, SW15003, SW15005, SW15007, SW15009, SW15011, SW15013, SW15015, SW15017, SW15019, SW15021, SW15023, SW15025, SW15837, TC15001, TC15002, TC15003, TC15004, TC15005, TC15006, TC15007, TC15008, TC15009, TC15010, TC15011, TC15012, TC15013, TC15014, TC15015, TC15016, TC15017, TC15018, TC15019, TC15020, TC15021, TC15022, TC15023, TC15024, TC15025, TC15026, TC15027, TC15028, TC15029, TC15030, TC15031, TC15032, TC15033, TC15034: Name (none) -> ${Value}

Commit message: fix(kicad): owner edit (2026-10-25): Watsonville's second 838N mast is 838NCD with heads C and D
Signal 838N has two double masts, on 837's N and R legs; both were named 838NAB with heads A and B, a
duplicate name the layout compiler's trackplan piece reports as an error (ADR 0003 D8; head letters unique
across one signal's masts, rule 6). The owner renamed the second mast and relettered its heads. The
project file's change is KiCad's reordering of used_designators on save.

Verified:
- Netlist exported by the owner 2026-10-25 22:25, newer than every sheet and library; the diff is the
  three Value fields and the designator list only.

Co-Authored-By: Claude Opus 5.5 <noreply@anthropic.com>
Parts:
- H15001: value A -> C
- H15002: value B -> D
- S15001: value 838NAB -> 838NCD
Changed lines of the file:
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@@
 			)
 		)
-		(property "Value" "A"
+		(property "Value" "C"
 			(at 38.1 63.5 90)
 			(show_name no)
@@
 			)
 		)
-		(property "Value" "B"
+		(property "Value" "D"
 			(at 40.64 63.5 90)
 			(show_name no)
@@
 			)
 		)
-		(property "Value" "838NAB"
+		(property "Value" "838NCD"
 			(at 46.355 60.833 0)
 			(show_name no)
