File: SPCoast/Watsonville-Panel.kicad_sch (KiCad schematic)
At the start: 8 parts, among them U16034 0x2D

Commit message: refactor(kicad): seam vocabulary after the naming audit: Processor, IOBus, PanelIOBus, House, Style, TimeCode, LocoNet, NodeType, MQTT-JMRI
SPCoast/edits/2026-10-22-vocabulary.py, the owner's rulings on
FieldUnit-Subdivision docs/review/naming-audit-2026-10-22.md:
- Host stays only on the transport symbols; the Interlocking, OfficeUnit and Processor pins, the unit
  sheets' port and labels are Processor.
- IOBus on the Processor pin; the office side is PanelIOBus on the unit ports, the Panel boxes' pins,
  the panel labels and the root sheet pins.
- MAIN HOUSE is House; its H pin is MC and hidden, as asked.
- OfficeUnit Type -> Style = US&S; TimeCode and LocoNet spellings, the LocoNet transport's pin is
  Transport; the one input Codeline sheet pin is bidirectional.
- The CMRInet node's Board -> NodeType (body text follows); JMRI drivers' IC = MQTT-JMRI.

Verified: --check on production/vocab-before.net vs vocab-after.net: identical connectivity under the
pin map, same parts (MAIN HOUSE -> House), only the ruled fields changed; field-io --check passes;
ERC 0 violations.

Co-Authored-By: Claude Fable 5.1 <noreply@anthropic.com>
Connections:
- net IOBus renamed PanelIOBus
Changed lines of the file:
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@@
 		(at 87.63 104.14)
 	)
-	(hierarchical_label "IOBus"
+	(hierarchical_label "PanelIOBus"
 		(shape bidirectional)
 		(at 111.76 111.76 0)

Commit message: refactor(kicad): model board lamps leave the columns; stale instance fields follow the libraries; PanelLamp-* retired
The owner's ruling (2026-10-23): the PanelColumn is the logical column, tied to a control point; the panel
I/O hardware is not. Every PanelLamp was a model board lamp except the maintainer-call lamp on the column's
pin 8. 34 lamps are now ModelLamp-<color> (no Column pin, Style board); 8 MC lamps are PanelMCall-Lamp.
Wires untouched: ~{LAMP} keeps its pin and the Column wire of a model lamp ends on nothing. Instance fields
the libraries dropped in c1d446b are gone from the sheets: Address on 7 processors, Interlocking and Machine
on 14 columns, Host on 2 transports. Railroad stays on the AAR encoding because its Topic template reads
${Railroad}; where Railroad lives is pending. Cached definitions refreshed for Processor, PanelColumn,
Transport-MQTT and Encoding-AAR. Scripted: SPCoast/edits/2026-10-23-model-lamps.py (edit, --check, --retire).

Verified: the script's gate on production/fields-after.net vs model-lamps-after.net: same 743 parts, lib ids
change only on the 42 lamps to the expected targets, fields change only as listed (Style indication->board
x34, the 37 drops), connectivity after == before minus the model lamps' pin 1, ERC 0 violations (the two
lib_symbol_mismatch warnings gone). lint_symbol_fields: 97 symbols, 0 errors (PanelLamp-BLUE, -GREEN, -RED, -YELLOW retired; there was no AMBER). Subdivision tests: 157 OK.

Co-Authored-By: Claude Fable 5.1 <noreply@anthropic.com>
Parts:
- COL16034: Interlocking Watsonville -> (none); Machine SPCoast South -> (none)
- LMP16141, LMP16142, LMP16143: symbol Railroad-Office:PanelLamp-YELLOW -> Railroad-Office:ModelLamp-YELLOW; Style indication -> board
Connections:
- net at COL16034.1 (Column): no longer LMP16141.1 (Column)
- net at COL16034.3 (Column): no longer LMP16143.1 (Column)
- net at COL16034.2 (Column): no longer LMP16142.1 (Column)
Changed lines of the file:
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@@
 	)
 	(symbol
-		(lib_id "Railroad-Office:PanelLamp-YELLOW")
+		(lib_id "Railroad-Office:ModelLamp-YELLOW")
 		(at 80.01 26.67 0)
 		(unit 1)
@@
 			)
 		)
-		(property "Description" "One physical model board lamp. Value is a free descriptive label (e.g. OS, TRACK, MC) and is not used elsewhere. IndicationToken is a comma-separated list of indication names (track circuits such as 795T1,2NAA,799T1, or tokens such as MC1K) OR'd to drive this one lamp. All listed indications are still individually on the CodeLine wire"
+		(property "Description" "One physical model board lamp. Value is a free descriptive label (e.g. OS, TRACK ...) and is not used elsewhere. IndicationToken is a comma-separated list of indication names (tokens from the CodeLine) OR'd to drive this one lamp."
 			(at 80.01 34.29 0)
 			(hide yes)
@@
 			)
 		)
-		(property "Style" "indication"
+		(property "Style" "board"
 			(at 80.01 24.13 0)
 			(hide yes)
@@
 				)
 			)
-		)
-		(pin "1"
 		)
 		(pin "2"
@@
 	)
 	(symbol
-		(lib_id "Railroad-Office:PanelLamp-YELLOW")
+		(lib_id "Railroad-Office:ModelLamp-YELLOW")
 		(at 80.01 36.83 0)
 		(unit 1)
@@
 			)
 		)
-		(property "Description" "One physical model board lamp. Value is a free descriptive label (e.g. OS, TRACK, MC) and is not used elsewhere. IndicationToken is a comma-separated list of indication names (track circuits such as 795T1,2NAA,799T1, or tokens such as MC1K) OR'd to drive this one lamp. All listed indications are still individually on the CodeLine wire"
+		(property "Description" "One physical model board lamp. Value is a free descriptive label (e.g. OS, TRACK ...) and is not used elsewhere. IndicationToken is a comma-separated list of indication names (tokens from the CodeLine) OR'd to drive this one lamp."
 			(at 80.01 44.45 0)
 			(hide yes)
@@
 			)
 		)
-		(property "Style" "indication"
+		(property "Style" "board"
 			(at 80.01 34.29 0)
 			(hide yes)
@@
 				)
 			)
-		)
-		(pin "1"
 		)
 		(pin "2"
@@
 			)
 		)
-		(property "Interlocking" "Watsonville"
-			(at 80.01 129.54 0)
-			(show_name yes)
-			(do_not_autoplace yes)
-			(effects
-				(font
-					(size 1.27 1.27)
-				)
-			)
-		)
-		(property "Machine" "SPCoast South"
-			(at 80.645 125.73 0)
-			(show_name no)
-			(do_not_autoplace yes)
-			(effects
-				(font
-					(size 1.905 1.905)
-				)
-			)
-		)
 		(property "Role" "COLUMN"
 			(at 80.645 122.555 0)
@@
 	)
 	(symbol
-		(lib_id "Railroad-Office:PanelLamp-YELLOW")
+		(lib_id "Railroad-Office:ModelLamp-YELLOW")
 		(at 80.01 31.75 0)
 		(unit 1)
@@
 			)
 		)
-		(property "Description" "One physical model board lamp. Value is a free descriptive label (e.g. OS, TRACK, MC) and is not used elsewhere. IndicationToken is a comma-separated list of indication names (track circuits such as 795T1,2NAA,799T1, or tokens such as MC1K) OR'd to drive this one lamp. All listed indications are still individually on the CodeLine wire"
+		(property "Description" "One physical model board lamp. Value is a free descriptive label (e.g. OS, TRACK ...) and is not used elsewhere. IndicationToken is a comma-separated list of indication names (tokens from the CodeLine) OR'd to drive this one lamp."
 			(at 80.01 39.37 0)
 			(hide yes)
@@
 			)
 		)
-		(property "Style" "indication"
+		(property "Style" "board"
 			(at 80.01 29.21 0)
 			(hide yes)
@@
 			)
 		)
-		(pin "1"
-		)
 		(pin "2"

Commit message: refactor(kicad): Name on every device, office unit and encoding; Kind on the JMRI drivers; Driver-JMRI-Light
The owner's rulings of 2026-10-24 on the review of ADR 0008 rev 4: Name = ${Value}
is the identity key everywhere, devices included; the OfficeUnit's Columns is
derived and struck; a JMRI driver carries no address and is keyed by its object
class and the device it serves, the class carried by Kind (TURNOUT, SENSOR,
SIGNALMAST, LIGHT); Driver-JMRI-Light (ADR 0005 §8: ON, INTENSITY) for a lamp
JMRI drives, and the two Gilroy Interchange maintainer-call lamps MC1 and MC2
become Lights (they were Sensors, which JMRI only displays).

Script: SPCoast/edits/2026-10-24-names-kind-light.py. Libraries: Name on 36
symbols (OfficeUnit, 5 encodings, 12 PANEL, 18 DEVICE), Columns off OfficeUnit,
Kind on 5 JMRI drivers, Driver-JMRI-Light added (the Sensor's pin positions,
INTENSITY as pin 3 below, no-connect on the two placed instances). Sheets: 359
Name instance fields, 16 Kind, 2 lib_id swaps, caches refreshed (no pin moved on
a refreshed symbol).

Verified: gate --check production/SPCoast.net production/names-after.net PASS:
same parts, same connectivity, Name == Value on all 273 named instances (47
heads with Value "~" resolve to an empty Name), Columns dropped once, Kind on 16
drivers, 2 Sensor -> Light with pin 1 reading ON; ERC 0 before and after.
Subdivision lint_symbol_fields: 99 symbols, 0 errors (Kind now allowed on
IODRIVER). production/SPCoast.net is the new export (production/ is untracked).

Co-Authored-By: Claude Fable 5.1 <noreply@anthropic.com>
Parts:
- CDE16014, LMP16141, LMP16142, LMP16143, SGL16014, SWL16014: Name (none) -> ${Value}
Changed lines of the file:
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@@
+			)
+		)
+		(property "Name" "${Value}"
+			(at 80.01 63.5 0)
+			(hide yes)
+			(show_name no)
+			(do_not_autoplace no)
+			(effects
+				(font
+					(size 1.27 1.27)
+				)
 			)
 		)
@@
 			)
 		)
+		(property "Name" "${Value}"
+			(at 80.01 83.82 0)
+			(hide yes)
+			(show_name no)
+			(do_not_autoplace no)
+			(effects
+				(font
+					(size 1.27 1.27)
+				)
+			)
+		)
 		(property "Appliance" "lever"
 			(at 80.01 92.71 0)
@@
 			)
 		)
+		(property "Name" "${Value}"
+			(at 80.01 26.67 0)
+			(hide yes)
+			(show_name no)
+			(do_not_autoplace no)
+			(effects
+				(font
+					(size 1.27 1.27)
+				)
+			)
+		)
 		(property "Appliance" "lamp"
 			(at 80.01 24.13 0)
@@
 			)
 		)
+		(property "Name" "${Value}"
+			(at 80.01 36.83 0)
+			(hide yes)
+			(show_name no)
+			(do_not_autoplace no)
+			(effects
+				(font
+					(size 1.27 1.27)
+				)
+			)
+		)
 		(property "Appliance" "lamp"
 			(at 80.01 34.29 0)
@@
 			)
 		)
+		(property "Name" "${Value}"
+			(at 80.01 97.79 0)
+			(hide yes)
+			(show_name no)
+			(do_not_autoplace no)
+			(effects
+				(font
+					(size 1.27 1.27)
+				)
+			)
+		)
 		(property "Appliance" "lever"
 			(at 80.01 90.17 0)
@@
 			)
 		)
+		(property "Name" "${Value}"
+			(at 80.01 63.5 0)
+			(hide yes)
+			(show_name no)
+			(do_not_autoplace no)
+			(effects
+				(font
+					(size 1.27 1.27)
+				)
+			)
+		)
 		(property "Appliance" "lever"
 			(at 80.645 76.2 0)
@@
 			)
 		)
+		(property "Name" "${Value}"
+			(at 80.01 83.82 0)
+			(hide yes)
+			(show_name no)
+			(do_not_autoplace no)
+			(effects
+				(font
+					(size 1.27 1.27)
+				)
+			)
+		)
 		(property "Appliance" "lever"
 			(at 80.01 92.71 0)
@@
 			(hide yes)
 			(show_name no)
+			(do_not_autoplace no)
+			(effects
+				(font
+					(size 1.27 1.27)
+				)
+			)
+		)
+		(property "Name" "${Value}"
+			(at 80.01 31.75 0)
+			(hide yes)
+			(show_name no)

Commit message: feat(spcoast): every desk column names its CP Name
The owner's edit in KiCad: each PanelColumn carries a CP Name. On an
AAR codeline it may name the interlocking (Christopher, Gilroy
Interchange); on the 506 it names the house.

Verified: a fresh kicad-cli netlist compiles with no column.cp_name
diagnostics; the three column.house errors (columns 3, 4, 9) are
resolved by the importer rule, not the drawing.

Co-Authored-By: Claude Opus 5.5 <noreply@anthropic.com>
Parts:
- COL16034: CP Name (none) -> Watsonville
Changed lines of the file:
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@@
 			)
 		)
-		(property "CP Name" ""
+		(property "CP Name" "Watsonville"
 			(at 80.645 132.08 0)
 			(show_name yes)

Commit message: feat(spcoast): per-pin token fields on the panels, lamp Indication expressions, maintainer calls named 1MC
Applies the symbol rulings of 2026-10-28 to every sheet: the lib_symbols
caches of the changed symbols are the library's copies (this also clears
the stale PanelMCall and MaintainerCall caches), and every placed
instance gets the new hidden Control.*/Indication.* fields, loses
PanelLock Invert, and PanelMCall's whole-symbol Control and Indication
(Pin.MCK binary). Model lamps' IndicationToken becomes Indication: each
comma-separated circuit gets its K, qualifiers kept, joined with " | "
(795T1,01T,799T1 -> 795T1K | 01TK | 799T1K).

Maintainer calls in Christopher (1, 2), Corporal, Luchessa and Sargent
follow Gilroy Interchange (5dad54f): Value MC<n> -> <n>, Name ${Value}MC,
and the separate PanelMCall-Lamp is replaced by unit 2 of the same
PanelMCall at the old lamp's position, so its MCK pin sits where the
LAMP pin was. The old lamps' Column pin touched PanelColumn pin 8
directly (no wire); that pin is now unconnected, as on Gilroy
Interchange. Gilroy Interchange's local MaintainerCall_1 cache and its
two trackplan calls lose Indication.

Verified: fresh netlist before/after: components 752 -> 747 (the five
lamps), nets 1028 -> 1028; each old LAMP-pin net now holds the lever's
unit-2 MCK pin (pin 3) on the same expander pin (B1, pin 9); the levers'
nets are renamed only (~{S} -> ~{MCS}, unit suffix A); no other net
changed. Every field difference is an intended one. ERC 18 -> 1
violations (lib_symbol_mismatch 17 -> 0; pre-existing Sargent AUX1
pin_not_connected remains).

Co-Authored-By: Claude Opus 5.5 <noreply@anthropic.com>
Parts:
- LMP16141: Indication (none) -> 0101TK; IndicationToken 0101T -> (none)
- LMP16142: Indication (none) -> 0100TK; IndicationToken 0100T -> (none)
- LMP16143: Indication (none) -> 01TK; IndicationToken 01T -> (none)
- SGL16014: Control.HS (none) -> ${Value}HS; Control.NGS (none) -> ${Value}NGS; Control.SGS (none) -> ${Value}SGS; Indication.NGK (none) -> ${Value}NGK; Indication.SGK (none) -> ${Value}SGK; Indication.TEK (none) -> ${Value}TEK
- SWL16014: Control.NWS (none) -> ${Value}NWS; Control.RWS (none) -> ${Value}RWS; Indication.NWK (none) -> ${Value}NWK; Indication.RWK (none) -> ${Value}RWK
Changed lines of the file:
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@@
+			)
+		)
+		(property "Control.NWS" "${Value}NWS"
+			(at 80.645 76.2 0)
+			(hide yes)
+			(show_name no)
+			(do_not_autoplace no)
+			(effects
+				(font
+					(size 1.27 1.27)
+				)
+			)
+		)
+		(property "Control.RWS" "${Value}RWS"
+			(at 80.645 76.2 0)
+			(hide yes)
+			(show_name no)
+			(do_not_autoplace no)
+			(effects
+				(font
+					(size 1.27 1.27)
+				)
+			)
+		)
+		(property "Indication.NWK" "${Value}NWK"
+			(at 80.645 76.2 0)
+			(hide yes)
+			(show_name no)
+			(do_not_autoplace no)
+			(effects
+				(font
+					(size 1.27 1.27)
+				)
+			)
+		)
+		(property "Indication.RWK" "${Value}RWK"
+			(at 80.645 76.2 0)
+			(hide yes)
+			(show_name no)
+			(do_not_autoplace no)
+			(effects
+				(font
+					(size 1.27 1.27)
+				)
 			)
 		)
@@
 			)
 		)
+		(property "Control.NGS" "${Value}NGS"
+			(at 80.01 92.71 0)
+			(hide yes)
+			(show_name no)
+			(do_not_autoplace no)
+			(effects
+				(font
+					(size 1.27 1.27)
+				)
+			)
+		)
+		(property "Control.HS" "${Value}HS"
+			(at 80.01 92.71 0)
+			(hide yes)
+			(show_name no)
+			(do_not_autoplace no)
+			(effects
+				(font
+					(size 1.27 1.27)
+				)
+			)
+		)
+		(property "Control.SGS" "${Value}SGS"
+			(at 80.01 92.71 0)
+			(hide yes)
+			(show_name no)
+			(do_not_autoplace no)
+			(effects
+				(font
+					(size 1.27 1.27)
+				)
+			)
+		)
+		(property "Indication.NGK" "${Value}NGK"
+			(at 80.01 92.71 0)
+			(hide yes)
+			(show_name no)
+			(do_not_autoplace no)
+			(effects
+				(font
+					(size 1.27 1.27)
+				)
+			)
+		)
+		(property "Indication.SGK" "${Value}SGK"
+			(at 80.01 92.71 0)
+			(hide yes)
+			(show_name no)
+			(do_not_autoplace no)
+			(effects
+				(font
+					(size 1.27 1.27)
+				)
+			)
+		)
+		(property "Indication.TEK" "${Value}TEK"
+			(at 80.01 92.71 0)
+			(hide yes)
+			(show_name no)
+			(do_not_autoplace no)
+			(effects
+				(font
+					(size 1.27 1.27)
+				)
+			)
+		)
 		(pin "1"
 		)
@@
 			)
 		)
-		(property "IndicationToken" "0101T"
+		(property "Indication" "0101TK"
 			(at 78.105 26.67 0)
 			(show_name no)
@@
 			)
 		)
-		(property "IndicationToken" "01T"
+		(property "Indication" "01TK"
 			(at 78.105 36.83 0)
 			(show_name no)
@@
 			)
 		)
+		(property "Control.CODE" ""
+			(at 80.01 90.17 0)
+			(hide yes)
+			(show_name no)
+			(do_not_autoplace no)
+			(effects
+				(font
+					(size 1.27 1.27)
+				)
+			)
+		)
 		(pin "1"
 		)
@@
 			)
 		)
+		(property "Control.NWS" "${Value}NWS"
+			(at 80.645 76.2 0)
+			(hide yes)
+			(show_name no)
+			(do_not_autoplace no)
+			(effects
+				(font
+					(size 1.27 1.27)
+				)
+			)
+		)
+		(property "Control.RWS" "${Value}RWS"
+			(at 80.645 76.2 0)
+			(hide yes)
+			(show_name no)
+			(do_not_autoplace no)
+			(effects
+				(font
+					(size 1.27 1.27)
+				)
+			)
+		)
+		(property "Indication.NWK" "${Value}NWK"
+			(at 80.645 76.2 0)
+			(hide yes)
+			(show_name no)
+			(do_not_autoplace no)
+			(effects
+				(font
+					(size 1.27 1.27)
+				)
+			)
+		)
+		(property "Indication.RWK" "${Value}RWK"
+			(at 80.645 76.2 0)
+			(hide yes)
+			(show_name no)
+			(do_not_autoplace no)
+			(effects
+				(font
+					(size 1.27 1.27)
+				)
+			)
+		)
 		(pin "1"
 		)
@@
 			)
 		)
+		(property "Control.NGS" "${Value}NGS"
+			(at 80.01 92.71 0)
+			(hide yes)
+			(show_name no)
+			(do_not_autoplace no)
+			(effects
+				(font
+					(size 1.27 1.27)
+				)
+			)
+		)
+		(property "Control.HS" "${Value}HS"
+			(at 80.01 92.71 0)
+			(hide yes)
+			(show_name no)
+			(do_not_autoplace no)
+			(effects
+				(font
+					(size 1.27 1.27)
+				)
+			)
+		)
+		(property "Control.SGS" "${Value}SGS"
+			(at 80.01 92.71 0)
+			(hide yes)
+			(show_name no)
+			(do_not_autoplace no)
+			(effects
+				(font
+					(size 1.27 1.27)
+				)
+			)
+		)
+		(property "Indication.NGK" "${Value}NGK"
+			(at 80.01 92.71 0)
+			(hide yes)
+			(show_name no)
+			(do_not_autoplace no)
+			(effects
+				(font
+					(size 1.27 1.27)
+				)
+			)
+		)
+		(property "Indication.SGK" "${Value}SGK"
+			(at 80.01 92.71 0)
+			(hide yes)
+			(show_name no)
+			(do_not_autoplace no)
+			(effects
+				(font
+					(size 1.27 1.27)
+				)
+			)
+		)
+		(property "Indication.TEK" "${Value}TEK"
+			(at 80.01 92.71 0)
+			(hide yes)
+			(show_name no)
+			(do_not_autoplace no)
+			(effects
+				(font
+					(size 1.27 1.27)
+				)
+			)
+		)
 		(pin "5"
 		)
@@
 			)
 		)
-		(property "IndicationToken" "0100T"
+		(property "Indication" "0100TK"
 			(at 78.105 31.75 0)
 			(show_name no)
