File: SPCoast/Luchessa.kicad_sch (KiCad schematic)
At the start: 79 parts, among them SW7783 783, SW7795 795, SW7799 799, SW7900 795

Commit message: refactor(kicad): Name = ${Value} on every Trackplan appliance, so no key is read from Value
The owner (2026-10-24), on review finding 4: no exception for appliance names
read from Value. Data model keys are functional descriptions of their content
and the symbol attribute names reflect that choice; Value is generic. Every
Railroad-Trackplan APPLIANCE symbol (switches, derails, masts, heads, track
circuits, maintainer calls, auxiliaries) gains Name = ${Value}: the appliance's
own name, a head's letter. The compiler reads Name, never Value.

Script: SPCoast/edits/2026-10-24-trackplan-names.py (library symbols, placed
instances, caches refreshed; no pin moved).

Verified: gate --check production/SPCoast.net production/trackplan-names-after.net
PASS: same parts, lib ids, Values and connectivity; the only field change is Name
added on every Trackplan appliance with Name == Value; ERC 0 before and after.
Subdivision lint_symbol_fields: 99 symbols, 0 errors. production/SPCoast.net is
the new export.

Co-Authored-By: Claude Fable 5.1 <noreply@anthropic.com>
Parts:
- DERAIL7795, FLK7001, FLK7002, H7001, H7002, H7003, H7004, H7006, H7007, H7008, MC7001, S784E1, S784E2, S784W1, S784W2, S784W3, SW7783, SW7795, SW7799, TC7001, TC7002, TC7003, TC7004, TC7005, TC7006: Name (none) -> ${Value}

Commit message: feat(kicad): owner edit (2026-10-24): Industry symbol (TRACK, Kind INDUSTRY) replaces the dark stubs at Sargent, Corporal and Luchessa
Railroad-Trackplan gains Industry: Role TRACK, Kind INDUSTRY, one pin EoT at
(1.27, 0), description "Track exists past this point, but is not drawn". It is
visually distinct from Bumper and carries its own Kind, so a reader can tell
"track ends" from "track continues, not drawn" (ADR 0009 §3.10 amended in
FieldUnit-Subdivision).

Sargent B8, B9 and Corporal B6, B7 sit directly on the N and R ports of the
hand-thrown switch beyond END CTC; the wires drawn into dark track are gone.
Luchessa's industry spur: the Bumper B7007 and the wire into dark track are
gone; B7010 becomes Industry, and a new IRJ-END_CTC B11008 stands beside it.

The other sheets change only in their embedded library cache. On
GilroyInterchange KiCad renamed the cached Driver-JMRI-Light's second Kind
property to Kind_1: the library itself still carries two Kind properties on
that symbol (LIGHT and SENSOR, from 6882aa6), to be fixed separately. No placed
symbol is affected.

Verified:
- kicad-cli ERC: 0 violations
- lint_symbol_fields.py: 100 symbols, 0 errors, 0 warnings
- component field diff, previous netlist vs fresh export: only the five added
  Industry symbols, the added END CTC, the removed Bumper and B7010's Kind
- compile_layout.py output unchanged except provenance
- no lock files; owner reports KiCad project closed and files saved

Co-Authored-By: Claude Fable 5.1 <noreply@anthropic.com>
Parts:
- removed B7007: (no value), symbol Railroad-Trackplan:Bumper
- removed B7010: (no value), symbol Railroad-Trackplan:IRJ
- added B11008: END CTC, symbol Railroad-Trackplan:IRJ-END_CTC
- added B7010: (no value), symbol Railroad-Trackplan:Industry
Connections:
- net at B7004.2 (B), DOT7006.1 (To), TC7005.1 (TC): now also B11008.1 (CTC)
- new net: B11008.2 (DARK), B7010.2 (EoT)
Changed lines of the file:
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@@
 	(text "Industry"
 		(exclude_from_sim no)
-		(at 50.8 67.564 0)
+		(at 43.942 69.85 0)
 		(effects
 			(font
@@
 	(wire
 		(pts
-			(xy 38.1 69.85) (xy 59.69 69.85)
-		)
-		(stroke
-			(width 0.254)
-			(type dash)
-			(color 72 72 72 1)
-		)
-	)
-	(wire
-		(pts
 			(xy 123.19 102.87) (xy 214.63 102.87)
 		)
@@
 	)
 	(symbol
-		(lib_id "Railroad-Trackplan:Bumper")
-		(at 36.83 69.85 0)
-		(unit 1)
-		(body_style 1)
-		(exclude_from_sim no)
-		(in_bom yes)
-		(on_board yes)
-		(in_pos_files yes)
-		(dnp no)
-		(fields_autoplaced yes)
-		(property "Reference" "B7007"
-			(at 36.83 72.39 0)
-			(hide yes)
-			(show_name no)
-			(do_not_autoplace no)
-			(effects
-				(font
-					(size 1.27 1.27)
-				)
-			)
-		)
-		(property "Value" ""
-			(at 36.83 69.85 0)
-			(hide yes)
-			(show_name no)
-			(do_not_autoplace no)
-			(effects
-				(font
-					(size 1.27 1.27)
-				)
-			)
-		)
-		(property "Footprint" ""
-			(at 36.83 69.85 0)
-			(hide yes)
-			(show_name no)
-			(do_not_autoplace no)
-			(effects
-				(font
-					(size 1.27 1.27)
-				)
-			)
-		)
-		(property "Datasheet" ""
-			(at 36.83 69.85 0)
-			(hide yes)
-			(show_name no)
-			(do_not_autoplace no)
-			(effects
-				(font
-					(size 1.27 1.27)
-				)
-			)
-		)
-		(property "Description" "End of Track Bumper/Stop"
-			(at 36.83 69.85 0)
-			(hide yes)
-			(show_name no)
-			(do_not_autoplace no)
-			(effects
-				(font
-					(size 1.27 1.27)
-				)
-			)
-		)
-		(property "Role" "TRACK"
-			(at 36.83 69.85 0)
-			(hide yes)
-			(show_name no)
-			(do_not_autoplace no)
-			(effects
-				(font
-					(size 1.27 1.27)
-				)
-			)
-		)
-		(property "Kind" "BUMPER"
-			(at 36.83 69.85 0)
-			(hide yes)
-			(show_name no)
-			(do_not_autoplace no)
-			(effects
-				(font
-					(size 1.27 1.27)
-				)
-			)
-		)
-		(pin "2"
-		)
-		(instances
-			(project "SPCoast"
-				(path "/528348b2-add8-5367-a5f7-439c76f0ca33/2ed995e3-3819-55cd-b8d9-5c2af048ccb4/b4829d91-9b5a-495f-b7c8-ba6a6006660d"
-					(reference "B7007")
-					(unit 1)
-				)
-			)
-		)
-	)
-	(symbol
 		(lib_id "Railroad-Trackplan:Signal Head - CPL")
 		(at 200.66 66.04 0)
@@
 	)
 	(symbol
+		(lib_id "Railroad-Trackplan:Industry")
+		(at 58.42 69.85 0)
+		(unit 1)
+		(body_style 1)
+		(exclude_from_sim no)
+		(in_bom yes)
+		(on_board yes)
+		(in_pos_files yes)
+		(dnp no)
+		(fields_autoplaced yes)
+		(property "Reference" "B7010"
+			(at 58.42 72.39 0)
+			(hide yes)
+			(show_name no)
+			(do_not_autoplace no)
+			(effects
+				(font
+					(size 1.27 1.27)
+				)
+			)
+		)
+		(property "Value" ""
+			(at 58.42 69.85 0)
+			(hide yes)
+			(show_name no)
+			(do_not_autoplace no)
+			(effects
+				(font
+					(size 1.27 1.27)
+				)
+			)
+		)
+		(property "Footprint" ""
+			(at 58.42 69.85 0)
+			(hide yes)
+			(show_name no)
+			(do_not_autoplace no)
+			(effects
+				(font
+					(size 1.27 1.27)
+				)
+			)
+		)
+		(property "Datasheet" ""
+			(at 58.42 69.85 0)
+			(hide yes)
+			(show_name no)
+			(do_not_autoplace no)
+			(effects
+				(font
+					(size 1.27 1.27)
+				)
+			)
+		)
+		(property "Description" "Insulated Rail Joint"
+			(at 58.42 74.93 0)
+			(hide yes)
+			(show_name no)
+			(do_not_autoplace no)
+			(effects
+				(font
+					(size 1.27 1.27)
+				)
+			)
+		)
+		(property "Role" "TRACK"
+			(at 58.42 74.93 0)
+			(hide yes)
+			(show_name no)
+			(do_not_autoplace no)
+			(effects
+				(font
+					(size 1.27 1.27)
+				)
+			)
+		)
+		(property "Kind" "INDUSTRY"
+			(at 58.42 74.93 0)
+			(hide yes)
+			(show_name no)
+			(do_not_autoplace no)
+			(effects
+				(font
+					(size 1.27 1.27)
+				)
+			)
+		)
+		(pin "2"
+		)
+		(instances
+			(project "SPCoast"
+				(path "/528348b2-add8-5367-a5f7-439c76f0ca33/2ed995e3-3819-55cd-b8d9-5c2af048ccb4/b4829d91-9b5a-495f-b7c8-ba6a6006660d"
+					(reference "B7010")
+					(unit 1)
+				)
+			)
+		)
+	)
+	(symbol
 		(lib_id "Railroad-Trackplan:Switch_Powered")
 		(at 71.12 86.36 0)
@@
 	)
 	(symbol
+		(lib_id "Railroad-Trackplan:IRJ-END_CTC")
+		(at 60.96 69.85 0)
+		(unit 1)
+		(body_style 1)
+		(exclude_from_sim no)
+		(in_bom yes)
+		(on_board yes)
+		(in_pos_files yes)
+		(dnp no)
+		(fields_autoplaced yes)
+		(property "Reference" "B11008"
+			(at 60.96 76.835 0)
+			(hide yes)
+			(show_name no)
+			(do_not_autoplace no)
+			(effects
+				(font
+					(size 1.27 1.27)
+				)
+			)
+		)
+		(property "Value" "END CTC"
+			(at 61.2775 63.5 0)
+			(show_name no)
+			(do_not_autoplace no)
+			(effects
+				(font
+					(size 1.27 1.27)
+				)
+			)
+		)
+		(property "Footprint" ""
+			(at 60.96 69.85 0)
+			(hide yes)
+			(show_name no)
+			(do_not_autoplace no)
+			(effects
+				(font
+					(size 1.27 1.27)
+				)
+			)
+		)
+		(property "Datasheet" ""
+			(at 60.96 69.85 0)
+			(hide yes)
+			(show_name no)
+			(do_not_autoplace no)
+			(effects
+				(font
+					(size 1.27 1.27)
+				)
+			)
+		)
+		(property "Description" ""
+			(at 60.96 69.85 0)
+			(hide yes)
+			(show_name no)
+			(do_not_autoplace no)
+			(effects
+				(font
+					(size 1.27 1.27)
+				)
+			)
+		)
+		(property "Kind" "END_CTC"
+			(at 60.96 80.645 0)
+			(hide yes)
+			(show_name no)
+			(do_not_autoplace no)
+			(effects
+				(font
+					(size 1.27 1.27)
+				)
+			)
+		)
+		(property "Role" "TRACK"
+			(at 60.96 78.74 0)
+			(hide yes)
+			(show_name no)
+			(do_not_autoplace no)
+			(effects
+				(font
+					(size 1.27 1.27)
+				)
+			)
+		)
+		(pin "2"
+		)
+		(pin "1"
+		)
+		(instances
+			(project "SPCoast"
+				(path "/528348b2-add8-5367-a5f7-439c76f0ca33/2ed995e3-3819-55cd-b8d9-5c2af048ccb4/b4829d91-9b5a-495f-b7c8-ba6a6006660d"
+					(reference "B11008")
+					(unit 1)
+				)
+			)
+		)
+	)
+	(symbol
 		(lib_id "Railroad-Trackplan:Rule261-DoT-BiDirectional")
 		(at 36.83 83.82 0)
@@
 		)
 		(property "Value" "Gilroy Interchange"
-			(at 26.035 86.36 0)
+			(at 44.958 89.662 0)
 			(show_name no)
 			(do_not_autoplace no)
@@
 					(unit 1)
 				)
-			)
-		)
-	)
-	(symbol
-		(lib_id "Railroad-Trackplan:IRJ")
-		(at 60.96 69.85 0)
-		(unit 1)
-		(body_style 1)
-		(exclude_from_sim no)
-		(in_bom yes)
-		(on_board yes)
-		(in_pos_files yes)
-		(dnp no)
-		(fields_autoplaced yes)
-		(property "Reference" "B7010"
-			(at 60.96 72.39 0)
-			(hide yes)
-			(show_name no)
-			(do_not_autoplace no)
-			(effects
-				(font
-					(size 1.27 1.27)
-				)
-			)
-		)
-		(property "Value" ""
-			(at 60.96 69.85 0)
-			(hide yes)
-			(show_name no)
-			(do_not_autoplace no)
-			(effects
-				(font
-					(size 1.27 1.27)
-				)
-			)
-		)
-		(property "Footprint" ""
-			(at 60.96 69.85 0)
-			(hide yes)
-			(show_name no)
-			(do_not_autoplace no)
-			(effects
-				(font
-					(size 1.27 1.27)
-				)
-			)
-		)
-		(property "Datasheet" ""
-			(at 60.96 69.85 0)
-			(hide yes)
-			(show_name no)
-			(do_not_autoplace no)
-			(effects
-				(font
-					(size 1.27 1.27)
-				)
-			)
-		)
-		(property "Description" "Insulated Rail Joint"
-			(at 60.96 69.85 0)
-			(hide yes)
-			(show_name no)
-			(do_not_autoplace no)
-			(effects
-				(font
-					(size 1.27 1.27)
-				)
-			)
-		)
-		(property "Role" "TRACK"
-			(at 60.96 69.85 0)
-			(hide yes)
-			(show_name no)
-			(do_not_autoplace no)
-			(effects
-				(font
-					(size 1.27 1.27)
-				)
-			)
-		)
-		(property "Kind" "IRJ"
-			(at 60.96 69.85 0)
-			(hide yes)
-			(show_name no)
-			(do_not_autoplace no)
-			(effects
-				(font
-					(size 1.27 1.27)
-				)
-			)
-		)
-		(pin "1"
-		)
-		(pin "2"
-		)
-		(instances
-			(project "SPCoast"
-				(path "/528348b2-add8-5367-a5f7-439c76f0ca33/2ed995e3-3819-55cd-b8d9-5c2af048ccb4/b4829d91-9b5a-495f-b7c8-ba6a6006660d"
-					(reference "B7010")
-					(unit 1)
-				)

Commit message: feat(kicad): owner edit (2026-10-25): Milepost carries Name = ${Value}; mileposts ground the region at Lick
The Milepost symbol gains Name = ${Value} like every other keyed symbol, so the
compiler reads no Value for it. The two Luchessa mileposts take the field, and
three new mileposts are placed: 55.3 (Lick) and 77.1 at Gilroy Caltrain, 77.0 at
Gilroy Interchange. Panels/ is left untracked.

Verified: lint_symbol_fields 100 symbols, 0 errors, 0 warnings; the diff is
additions only, no instance field reset; FieldUnit-Subdivision 201 tests against
a fresh export; compile_layout.py --geometry writes mileposts 55.3, 77.1, 77.0,
78.3, 79.3 with no geometry info.

Co-Authored-By: Claude Fable 5.1 <noreply@anthropic.com>
Parts:
- MP7001, MP7002: Name (none) -> ${Value}
Changed lines of the file:
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@@
 			)
 		)
+		(property "Name" "${Value}"
+			(at 58.42 55.88 0)
+			(hide yes)
+			(show_name no)
+			(do_not_autoplace no)
+			(effects
+				(font
+					(size 1.27 1.27)
+				)
+			)
+		)
 		(instances
 			(project "SPCoast"
@@
 			(at 160.02 55.88 0)
 			(hide yes)
+			(show_name no)
+			(do_not_autoplace no)
+			(effects
+				(font
+					(size 1.27 1.27)
+				)
+			)
+		)
+		(property "Name" "${Value}"
+			(at 160.02 55.88 0)
+			(hide yes)

Commit message: feat(kicad): owner edit (2026-10-26): NextCP carries Interlocking; Industry carries Name; HBA leaves the track
The owner's edits after the trackplan review:
- NextCP gains Interlocking = ${Value}, a key the compiler reads for the destination; every instance takes it.
  Christopher's two NextCPs toward Corporal now say Corporal (both said Sargent).
- Industry gains Name = ${VALUE}. The five Industries are named: Gilroy Industry at Luchessa, Beet Loader 1
  and 2 at Corporal and at Sargent.
- Sargent's HBA (hot box alarm) is moved off 1SAT's net; its MC pin is unconnected and it carries Milepost 83.4.
- Watsonville: one Rule 93 (YARD) symbol is moved to the yard side of its joint.
Panels/ is left untracked.

Verified:
- Netlist exported by the owner 2026-10-26 12:37, newer than every sheet and the library.
- lint_symbol_fields: 100 symbols, 0 errors, 0 warnings.

Co-Authored-By: Claude Opus 5.5 <noreply@anthropic.com>
Parts:
- B7010: value (none) -> Gilroy Industry; Name (none) -> ${VALUE}
- CP7001, CP7002, CP7003, CP7004: Interlocking (none) -> ${Value}
Other:
- note removed: "Industry"
Changed lines of the file:
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@@
 		(comment 9 "active")
 	)
-	(text "Industry"
-		(exclude_from_sim no)
-		(at 43.942 69.85 0)
-		(effects
-			(font
-				(size 2.54 2.54)
-				(thickness 0.254)
-				(bold yes)
-			)
-		)
-	)
 	(text "Rule 261 (Track Signaled in Both Directions): \nGoverns bi-directional signal territory (often controlled by \nCentralized Traffic Control, or CTC).  Under Rule 261, block signal \nindications supersede train superiority for both opposing and\nfollowing movements on the same track, allowing the dispatcher to\ndynamically change the direction of traffic by clearing signals."
 		(exclude_from_sim no)
@@
 	(symbol
 		(lib_id "Railroad-Trackplan:NextCP")
-		(at 245.11 102.87 180)
+		(at 245.11 102.87 0)
 		(unit 1)
 		(body_style 1)
@@
 		(dnp no)
 		(property "Reference" "CP7004"
-			(at 241.935 100.965 0)
+			(at 248.285 104.775 0)
 			(hide yes)
 			(show_name no)
@@
 		)
 		(property "Value" "Christopher"
-			(at 247.015 102.87 0)
+			(at 247.65 111.76 0)
+			(hide yes)
 			(show_name no)
-			(do_not_autoplace no)
+			(do_not_autoplace yes)
 			(effects
 				(font
@@
 		)
 		(property "Footprint" ""
-			(at 248.92 102.87 0)
+			(at 241.3 102.87 0)
 			(hide yes)
 			(show_name no)
@@
 		)
 		(property "Datasheet" ""
-			(at 248.92 102.87 0)
+			(at 241.3 102.87 0)
 			(hide yes)
 			(show_name no)
@@
 		)
 		(property "Description" "Identifies the next control point on this track"
-			(at 248.285 95.885 0)
+			(at 241.935 109.855 0)
 			(hide yes)
 			(show_name no)
@@
 			)
 		)
+		(property "Interlocking" "${Value}"
+			(at 247.65 111.76 0)
+			(hide yes)
+			(show_name no)
+			(do_not_autoplace no)
+			(effects
+				(font
+					(size 1.27 1.27)
+				)
+			)
+		)
 		(pin "1"
 		)
@@
 		(in_pos_files yes)
 		(dnp no)
-		(fields_autoplaced yes)
 		(property "Reference" "B7010"
 			(at 58.42 72.39 0)
@@
 			)
 		)
-		(property "Value" ""
+		(property "Value" "Gilroy Industry"
 			(at 58.42 69.85 0)
 			(hide yes)
@@
 			)
 		)
-		(property "Description" "Insulated Rail Joint"
+		(property "Description" "Track exists past this point, but is not drawn"
 			(at 58.42 74.93 0)
 			(hide yes)
@@
 			)
 		)
+		(property "Name" "${VALUE}"
+			(at 58.42 69.85 0)
+			(hide yes)
+			(show_name no)
+			(do_not_autoplace no)
+			(effects
+				(font
+					(size 1.27 1.27)
+				)
+			)
+		)
 		(pin "2"
 		)
@@
 	(symbol
 		(lib_id "Railroad-Trackplan:NextCP")
-		(at 245.11 86.36 180)
+		(at 245.11 86.36 0)
 		(unit 1)
 		(body_style 1)
@@
 		(dnp no)
 		(property "Reference" "CP7003"
-			(at 241.935 84.455 0)
+			(at 248.285 88.265 0)
 			(hide yes)
 			(show_name no)
@@
 		)
 		(property "Value" "Christopher"
-			(at 247.015 86.36 0)
+			(at 247.65 95.25 0)
+			(hide yes)
 			(show_name no)
-			(do_not_autoplace no)
+			(do_not_autoplace yes)
 			(effects
 				(font
@@
 		)
 		(property "Footprint" ""
-			(at 248.92 86.36 0)
+			(at 241.3 86.36 0)
 			(hide yes)
 			(show_name no)
@@
 		)
 		(property "Datasheet" ""
-			(at 248.92 86.36 0)
+			(at 241.3 86.36 0)
 			(hide yes)
 			(show_name no)
@@
 		)
 		(property "Description" "Identifies the next control point on this track"
-			(at 248.285 79.375 0)
+			(at 241.935 93.345 0)
 			(hide yes)
 			(show_name no)
@@
 			)
 		)
+		(property "Interlocking" "${Value}"
+			(at 247.65 95.25 0)
+			(hide yes)
+			(show_name no)
+			(do_not_autoplace no)
+			(effects
+				(font
+					(size 1.27 1.27)
+				)
+			)
+		)
 		(pin "1"
 		)
@@
 	(symbol
 		(lib_id "Railroad-Trackplan:NextCP")
-		(at 245.11 69.85 180)
+		(at 245.11 69.85 0)
 		(unit 1)
 		(body_style 1)
@@
 		(dnp no)
 		(property "Reference" "CP7002"
-			(at 241.935 67.945 0)
+			(at 248.285 71.755 0)
 			(hide yes)
 			(show_name no)
@@
 		)
 		(property "Value" "Hollister"
-			(at 247.015 69.85 0)
+			(at 247.65 78.74 0)
+			(hide yes)
 			(show_name no)
-			(do_not_autoplace no)
+			(do_not_autoplace yes)
 			(effects
 				(font
@@
 		)
 		(property "Footprint" ""
-			(at 248.92 69.85 0)
+			(at 241.3 69.85 0)
 			(hide yes)
 			(show_name no)
@@
 		)
 		(property "Datasheet" ""
-			(at 248.92 69.85 0)
+			(at 241.3 69.85 0)
 			(hide yes)
 			(show_name no)
@@
 		)
 		(property "Description" "Identifies the next control point on this track"
-			(at 248.285 62.865 0)
+			(at 241.935 76.835 0)
 			(hide yes)
 			(show_name no)
@@
 			)
 		)
+		(property "Interlocking" "${Value}"
+			(at 247.65 78.74 0)
+			(hide yes)
+			(show_name no)
+			(do_not_autoplace no)
+			(effects
+				(font
+					(size 1.27 1.27)
+				)
+			)
+		)
 		(pin "1"
 		)
@@
 		)
 		(property "Value" "Gilroy Interchange"
-			(at 44.958 89.662 0)
+			(at 30.48 95.25 0)
+			(hide yes)
 			(show_name no)
-			(do_not_autoplace no)
+			(do_not_autoplace yes)
 			(effects
 				(font
@@
 			(hide yes)
 			(show_name no)
+			(do_not_autoplace no)
+			(effects
+				(font
+					(size 1.27 1.27)
+				)
+			)
+		)
+		(property "Interlocking" "${Value}"
+			(at 30.48 95.25 0)
+			(hide yes)
+			(show_name no)

Commit message: refactor(symbols): the CP field is CP Name on every trackplan symbol
One fact, which house an appliance or circuit stands in, had two field
names: CP Name on the House and PanelColumn, CP on 17 trackplan
symbols. Every CP is now CP Name, in the library and in each placed
symbol, by a text rename of the field name only (KiCad's update
symbols was not used; it resets per-instance fields).

Verified: fresh kicad-cli netlists before and after: 754 components on
both, 136 had CP, every field identical once CP is read as CP Name, no
CP left. lint_symbol_fields: 100 symbols, 0 errors, 0 warnings.

Co-Authored-By: Claude Opus 5.5 <noreply@anthropic.com>
Parts:
- B7001, FLK7001, FLK7002, SW7783, TC7006: CP Luchessa -> (none); CP Name (none) -> Luchessa
- B7003, B7004, DERAIL7795, SW7795, TC7004, TC7005: CP Gilroy -> (none); CP Name (none) -> Gilroy
- B7008, B7009, SW7799, TC7001, TC7002, TC7003: CP Carnadero -> (none); CP Name (none) -> Carnadero
Changed lines of the file:
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@@
 			)
 		)
-		(property "CP" "Gilroy"
+		(property "CP Name" "Gilroy"
 			(at 77.47 67.31 0)
 			(show_name no)
@@
 			)
 		)
-		(property "CP" "Carnadero"
+		(property "CP Name" "Carnadero"
 			(at 214.63 88.265 0)
 			(show_name no)
@@
 			)
 		)
-		(property "CP" "Luchessa"
+		(property "CP Name" "Luchessa"
 			(at 220.98 45.72 0)
 			(show_name no)
@@
 			)
 		)
-		(property "CP" "Carnadero"
+		(property "CP Name" "Carnadero"
 			(at 214.63 104.775 0)
 			(show_name no)
@@
 			)
 		)
-		(property "CP" "Gilroy"
+		(property "CP Name" "Gilroy"
 			(at 66.04 71.755 0)
 			(show_name no)
@@
 			)
 		)
-		(property "CP" "Carnadero"
+		(property "CP Name" "Carnadero"
 			(at 172.72 90.805 0)
 			(show_name no)
@@
 			)
 		)
-		(property "CP" "Gilroy"
+		(property "CP Name" "Gilroy"
 			(at 137.16 88.265 0)
 			(show_name no)
@@
 			)
 		)
-		(property "CP" "Gilroy"
+		(property "CP Name" "Gilroy"
 			(at 109.22 90.805 0)
 			(show_name no)
@@
 			)
 		)
-		(property "CP" "Luchessa"
+		(property "CP Name" "Luchessa"
 			(at 214.63 45.72 0)
 			(show_name no)
@@
 			)
 		)
-		(property "CP" "Luchessa"
+		(property "CP Name" "Luchessa"
 			(at 71.12 81.915 0)
 			(show_name no)
@@
 			)
 		)
-		(property "CP" "Carnadero"
+		(property "CP Name" "Carnadero"
 			(at 214.63 71.755 0)
 			(show_name no)
@@
 			)
 		)
-		(property "CP" "Luchessa"
+		(property "CP Name" "Luchessa"
 			(at 50.8 88.265 0)
 			(show_name no)
@@
 			)
 		)
-		(property "CP" "Carnadero"
+		(property "CP Name" "Carnadero"
 			(at 204.47 88.9 0)
 			(show_name no)
@@
 			)
 		)
-		(property "CP" "Carnadero"
+		(property "CP Name" "Carnadero"
 			(at 204.47 72.39 0)
 			(show_name no)
@@
 			)
 		)
-		(property "CP" "Luchessa"
+		(property "CP Name" "Luchessa"
 			(at 58.42 83.82 0)
 			(show_name no)
@@
 			)
 		)
-		(property "CP" "Gilroy"
+		(property "CP Name" "Gilroy"
 			(at 121.92 105.41 0)
 			(show_name no)
@@
 			)
 		)
-		(property "CP" "Gilroy"
+		(property "CP Name" "Gilroy"
 			(at 85.09 74.295 0)
 			(show_name no)
